File: HARDWARE/FOC_CONTROLLER/FOC_CONTROLLER_V1/U.kicad_sch (KiCad schematic)
At the start: 17 parts

Commit message: up
Parts:
- Q1: renamed from Q; footprint DMT6018LDR7 -> samacsys:DMT6018LDR7
- renumbered D to D2
Connections:
- net GND: now also C15.1
Changed lines of the file:
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@@
 		(dnp no)
 		(fields_autoplaced yes)
-		(property "Reference" "D"
+		(property "Reference" "D2"
 			(at 109.22 33.02 0)
 			(effects
@@
 					(unit 1)
 				)
+				(path "/21624bb8-7220-4725-ab4f-34c4768aac8d/f72fcd55-797d-4de7-b16c-a295f170430e"
+					(reference "D2")
+					(unit 1)
+				)
 				(path "/21624bb8-7220-4725-ab4f-34c4768aac8d/fc458950-2711-4a11-802f-b3226dc264b9"
 					(reference "D6")
@@
 	)
 	(symbol
+		(lib_id "power:GND")
+		(at 180.34 138.43 0)
+		(unit 1)
+		(exclude_from_sim no)
+		(in_bom yes)
+		(on_board yes)
+		(dnp no)
+		(fields_autoplaced yes)
+		(property "Reference" "#PWR034"
+			(at 180.34 144.78 0)
+			(effects
+				(font
+					(size 1.27 1.27)
+				)
+				(hide yes)
+			)
+		)
+		(property "Value" "GND"
+			(at 180.34 143.51 0)
+			(effects
+				(font
+					(size 1.27 1.27)
+				)
+			)
+		)
+		(property "Footprint" ""
+			(at 180.34 138.43 0)
+			(effects
+				(font
+					(size 1.27 1.27)
+				)
+				(hide yes)
+			)
+		)
+		(property "Datasheet" ""
+			(at 180.34 138.43 0)
+			(effects
+				(font
+					(size 1.27 1.27)
+				)
+				(hide yes)
+			)
+		)
+		(property "Description" "Power symbol creates a global label with name \"GND\" , ground"
+			(at 180.34 138.43 0)
+			(effects
+				(font
+					(size 1.27 1.27)
+				)
+				(hide yes)
+			)
+		)
+		(pin "1"
+		)
+		(instances
+			(project "FOC_CONTROLLER_V1"
+				(path "/21624bb8-7220-4725-ab4f-34c4768aac8d/c3cbd430-6fb2-4bfe-86b9-0dcdbd0b95f5"
+					(reference "#PWR035")
+					(unit 1)
+				)
+				(path "/21624bb8-7220-4725-ab4f-34c4768aac8d/f72fcd55-797d-4de7-b16c-a295f170430e"
+					(reference "#PWR034")
+					(unit 1)
+				)
+				(path "/21624bb8-7220-4725-ab4f-34c4768aac8d/fc458950-2711-4a11-802f-b3226dc264b9"
+					(reference "#PWR036")
+					(unit 1)
+				)
+			)
+		)
+	)
+	(symbol
 		(lib_id "Diode:1N4148WT")
 		(at 109.22 59.69 0)
@@
 		(dnp no)
 		(fields_autoplaced yes)
-		(property "Reference" "Q"
+		(property "Reference" "Q1"
 			(at 157.48 33.02 0)
 			(effects
@@
 			)
 		)
-		(property "Footprint" "DMT6018LDR7"
+		(property "Footprint" "samacsys:DMT6018LDR7"
 			(at 165.1 144.45 0)
 			(effects
@@
 					(unit 1)
 				)
+				(path "/21624bb8-7220-4725-ab4f-34c4768aac8d/f72fcd55-797d-4de7-b16c-a295f170430e"
+					(reference "Q1")
+					(unit 1)
+				)
 				(path "/21624bb8-7220-4725-ab4f-34c4768aac8d/fc458950-2711-4a11-802f-b3226dc264b9"
 					(reference "Q3")
@@
 		(dnp no)
 		(fields_autoplaced yes)
-		(property "Reference" "#PWR"
+		(property "Reference" "#PWR0101"
 			(at 104.14 132.08 0)
 			(effects
@@
 					(unit 1)
 				)
+				(path "/21624bb8-7220-4725-ab4f-34c4768aac8d/f72fcd55-797d-4de7-b16c-a295f170430e"
+					(reference "#PWR0101")
+					(unit 1)
+				)

Commit message: update
Parts:
- added R43: 3k, Resistor_SMD:R_0201_0603Metric_Pad0.64x0.40mm_HandSolder, symbol Device:R_Small
Connections:
- net SHUNT+: now also R43.1
- new net SHUNTAFTER+: R43.2
Changed lines of the file:
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@@
+	)
+	(junction
+		(at 168.91 68.58)
+		(diameter 0)
+		(color 0 0 0 0)
 	)
 	(junction
@@
 	(wire
 		(pts
-			(xy 168.91 63.5) (xy 168.91 76.2)
+			(xy 168.91 63.5) (xy 168.91 68.58)
 		)
 		(stroke
@@
 	(wire
 		(pts
+			(xy 168.91 68.58) (xy 168.91 76.2)
+		)
+		(stroke
+			(width 0)
+			(type default)
+		)
+	)
+	(wire
+		(pts
 			(xy 180.34 130.81) (xy 185.42 130.81)
 		)
@@
 		(pts
 			(xy 135.89 127) (xy 140.97 127)
+		)
+		(stroke
+			(width 0)
+			(type default)
+		)
+	)
+	(wire
+		(pts
+			(xy 168.91 68.58) (xy 170.18 68.58)
 		)
 		(stroke
@@
 		(shape input)
 		(at 140.97 134.62 0)
+		(effects
+			(font
+				(size 1.27 1.27)
+			)
+			(justify left)
+		)
+	)
+	(hierarchical_label "SHUNTAFTER+"
+		(shape input)
+		(at 175.26 68.58 0)
 		(effects
 			(font
@@
 					(unit 1)
 				)
+			)
+		)
+	)
+	(symbol
+		(lib_id "Device:R_Small")
+		(at 172.72 68.58 90)
+		(unit 1)
+		(exclude_from_sim no)
+		(in_bom yes)
+		(on_board yes)
+		(dnp no)
+		(fields_autoplaced yes)
+		(property "Reference" "R43"
+			(at 172.72 63.5 90)
+			(effects
+				(font
+					(size 1.016 1.016)
+				)
+			)
+		)
+		(property "Value" "3k"
+			(at 172.72 66.04 90)
+			(effects
+				(font
+					(size 1.27 1.27)
+				)
+			)
+		)
+		(property "Footprint" "Resistor_SMD:R_0201_0603Metric_Pad0.64x0.40mm_HandSolder"
+			(at 172.72 68.58 0)
+			(effects
+				(font
+					(size 1.27 1.27)
+				)
+				(hide yes)
+			)
+		)
+		(property "Datasheet" "~"
+			(at 172.72 68.58 0)
+			(effects
+				(font
+					(size 1.27 1.27)
+				)
+				(hide yes)
+			)
+		)
+		(property "Description" "Resistor, small symbol"
+			(at 172.72 68.58 0)
+			(effects
+				(font
+					(size 1.27 1.27)
+				)
+				(hide yes)
+			)
+		)
+		(pin "1"
+		)
+		(pin "2"
+		)
+		(instances
+			(project "FOC_CONTROLLER_V1"
+				(path "/21624bb8-7220-4725-ab4f-34c4768aac8d/c3cbd430-6fb2-4bfe-86b9-0dcdbd0b95f5"
+					(reference "R44")
+					(unit 1)
+				)
+				(path "/21624bb8-7220-4725-ab4f-34c4768aac8d/f72fcd55-797d-4de7-b16c-a295f170430e"
+					(reference "R43")
+					(unit 1)
+				)
+				(path "/21624bb8-7220-4725-ab4f-34c4768aac8d/fc458950-2711-4a11-802f-b3226dc264b9"
+					(reference "R45")
+					(unit 1)
+				)

Commit message: update foc
Parts:
- removed R8: 10mR, Resistor_SMD:R_0201_0603Metric_Pad0.64x0.40mm_HandSolder, symbol Device:R_Small
- added R48: R_Shunt, samacsys:4wire_0603, symbol Device:R_Shunt
- C13: Manufacturer_Part_Number (none) -> GCM188M8EH105KE8D; Mouser Part Number (none) -> 81-GCM188M8EH105KE8D
Connections:
- net GND: now also R48.4; no longer R9.1
- net SHUNT+: now also R48.2; no longer Q1.3 (S2), R10.1
- new net: Q1.3 (S2), R48.1
- new net INPUTAOP+: R10.1
- new net INPUTAOP-: R9.1
- new net SHUNT-: R48.3
Other:
- note removed: "GCM188D71H105KE35"
- note removed: "WURTH 580060716002"
- moved on the sheet: R43
Changed lines of the file:
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@@
 	(generator_version "9.0")
 	(paper "A4")
-	(text "GCM188D71H105KE35"
-		(exclude_from_sim no)
-		(at 149.86 70.358 0)
-		(effects
-			(font
-				(size 1.27 1.27)
-			)
-		)
-	)
-	(text "50V\n"
+	(text "50V"
 		(exclude_from_sim no)
 		(at 188.722 35.56 0)
@@
 		)
 	)
-	(text "WURTH 580060716002"
-		(exclude_from_sim no)
-		(at 191.516 80.01 0)
-		(effects
-			(font
-				(size 1.27 1.27)
-			)
-		)
-	)
 	(junction
 		(at 125.73 59.69)
@@
 	)
 	(junction
-		(at 168.91 68.58)
-		(diameter 0)
-		(color 0 0 0 0)
-	)
-	(junction
 		(at 104.14 134.62)
 		(diameter 0)
@@
 	(wire
 		(pts
+			(xy 173.99 69.85) (xy 173.99 73.66)
+		)
+		(stroke
+			(width 0)
+			(type default)
+		)
+	)
+	(wire
+		(pts
 			(xy 101.6 59.69) (xy 101.6 63.5)
 		)
@@
 	(wire
 		(pts
-			(xy 118.11 127) (xy 124.46 127)
-		)
-		(stroke
-			(width 0)
-			(type default)
-		)
-	)
-	(wire
-		(pts
 			(xy 90.17 63.5) (xy 101.6 63.5)
 		)
@@
 	(wire
 		(pts
+			(xy 119.38 127) (xy 124.46 127)
+		)
+		(stroke
+			(width 0)
+			(type default)
+		)
+	)
+	(wire
+		(pts
 			(xy 111.76 48.26) (xy 101.6 48.26)
 		)
@@
 	(wire
 		(pts
-			(xy 168.91 63.5) (xy 168.91 68.58)
+			(xy 168.91 63.5) (xy 168.91 71.12)
 		)
 		(stroke
@@
 	(wire
 		(pts
-			(xy 168.91 68.58) (xy 168.91 76.2)
+			(xy 172.72 73.66) (xy 173.99 73.66)
 		)
 		(stroke
@@
 	(wire
 		(pts
-			(xy 168.91 68.58) (xy 170.18 68.58)
-		)
-		(stroke
-			(width 0)
-			(type default)
-		)
-	)
-	(wire
-		(pts
 			(xy 129.54 127) (xy 135.89 127)
 		)
@@
 	(wire
 		(pts
+			(xy 173.99 78.74) (xy 172.72 78.74)
+		)
+		(stroke
+			(width 0)
+			(type default)
+		)
+	)
+	(wire
+		(pts
 			(xy 116.84 48.26) (xy 125.73 48.26)
 		)
@@
 			(width 0)
 			(type default)
-		)
-	)
-	(label "SHUNT-"
-		(at 168.91 85.09 0)
-		(effects
-			(font
-				(size 1.27 1.27)
-			)
-			(justify left bottom)
-		)
-	)
-	(label "SHUNT-"
-		(at 118.11 127 180)
-		(effects
-			(font
-				(size 1.27 1.27)
-			)
-			(justify right bottom)
-		)
-	)
-	(label "SHUNT+"
-		(at 92.71 134.62 180)
-		(effects
-			(font
-				(size 1.27 1.27)
-			)
-			(justify right bottom)
-		)
-	)
-	(label "SHUNT+"
-		(at 168.91 74.93 0)
-		(effects
-			(font
-				(size 1.27 1.27)
-			)
-			(justify left bottom)
 		)
 	)
@@
 		)
 	)
+	(hierarchical_label "INPUTAOP-"
+		(shape input)
+		(at 119.38 127 180)
+		(effects
+			(font
+				(size 1.27 1.27)
+			)
+			(justify right)
+		)
+	)
 	(hierarchical_label "OPO"
 		(shape input)
@@
 		)
 	)
+	(hierarchical_label "SHUNT+"
+		(shape input)
+		(at 173.99 73.66 0)
+		(effects
+			(font
+				(size 1.27 1.27)
+			)
+			(justify left)
+		)
+	)
 	(hierarchical_label "OPP"
 		(shape input)
@@
 	(hierarchical_label "SHUNTAFTER+"
 		(shape input)
-		(at 175.26 68.58 0)
+		(at 179.07 69.85 0)
 		(effects
 			(font
@@
 		)
 	)
+	(hierarchical_label "INPUTAOP+"
+		(shape input)
+		(at 92.71 134.62 180)
+		(effects
+			(font
+				(size 1.27 1.27)
+			)
+			(justify right)
+		)
+	)
 	(hierarchical_label "HS"
 		(shape input)
@@
 		(shape input)
 		(at 185.42 52.07 0)
+		(effects
+			(font
+				(size 1.27 1.27)
+			)
+			(justify left)
+		)
+	)
+	(hierarchical_label "SHUNT-"
+		(shape input)
+		(at 173.99 78.74 0)
 		(effects
 			(font
@@
 	(symbol
 		(lib_id "Device:R_Small")
-		(at 172.72 68.58 90)
+		(at 176.53 69.85 90)
 		(unit 1)
 		(exclude_from_sim no)
@@
 		(fields_autoplaced yes)
 		(property "Reference" "R43"
-			(at 172.72 63.5 90)
+			(at 176.53 64.77 90)
 			(effects
 				(font
@@
 		)
 		(property "Value" "3k"
-			(at 172.72 66.04 90)
+			(at 176.53 67.31 90)
 			(effects
 				(font
@@
 		)
 		(property "Footprint" "Resistor_SMD:R_0201_0603Metric_Pad0.64x0.40mm_HandSolder"
-			(at 172.72 68.58 0)
+			(at 176.53 69.85 0)
 			(effects
 				(font
@@
 		)
 		(property "Datasheet" "~"
-			(at 172.72 68.58 0)
+			(at 176.53 69.85 0)
 			(effects
 				(font
@@
 		)
 		(property "Description" "Resistor, small symbol"
-			(at 172.72 68.58 0)
+			(at 176.53 69.85 0)
 			(effects
 				(font
@@
 	(symbol
 		(lib_id "Device:R_Small")
-		(at 168.91 78.74 180)
-		(unit 1)
-		(exclude_from_sim no)
-		(in_bom yes)
-		(on_board yes)
-		(dnp no)
-		(fields_autoplaced yes)
-		(property "Reference" "R8"
-			(at 171.45 77.4699 0)
-			(effects
-				(font
-					(size 1.016 1.016)
-				)
-				(justify right)
-			)
-		)
-		(property "Value" "10mR"
-			(at 171.45 80.0099 0)
-			(effects
-				(font
-					(size 1.27 1.27)
-				)
-				(justify right)
-			)
-		)
-		(property "Footprint" "Resistor_SMD:R_0201_0603Metric_Pad0.64x0.40mm_HandSolder"
-			(at 168.91 78.74 0)
-			(effects
-				(font
-					(size 1.27 1.27)
-				)
-				(hide yes)
-			)
-		)
-		(property "Datasheet" "~"
-			(at 168.91 78.74 0)
-			(effects
-				(font
-					(size 1.27 1.27)
-				)
-				(hide yes)
-			)
-		)
-		(property "Description" "580060716002"
-			(at 168.91 78.74 0)
-			(effects
-				(font
-					(size 1.27 1.27)
-				)
-				(hide yes)
-			)
-		)
-		(pin "1"
-		)
-		(pin "2"
-		)
-		(instances
-			(project "FOC_CONTROLLER_V1"
-				(path "/21624bb8-7220-4725-ab4f-34c4768aac8d/c3cbd430-6fb2-4bfe-86b9-0dcdbd0b95f5"
-					(reference "R24")
-					(unit 1)
-				)
-				(path "/21624bb8-7220-4725-ab4f-34c4768aac8d/f72fcd55-797d-4de7-b16c-a295f170430e"
-					(reference "R8")
-					(unit 1)
-				)
-				(path "/21624bb8-7220-4725-ab4f-34c4768aac8d/fc458950-2711-4a11-802f-b3226dc264b9"
-					(reference "R35")
-					(unit 1)
-				)
-			)
-		)
-	)
-	(symbol
-		(lib_id "Device:R_Small")
 		(at 99.06 134.62 90)
 		(unit 1)
@@
 		(on_board yes)
 		(dnp no)
-		(fields_autoplaced yes)
 		(property "Reference" "C13"
 			(at 180.34 34.2835 0)
@@
 				)
 				(hide yes)
+			)
+		)
+		(property "Manufacturer_Part_Number" "GCM188M8EH105KE8D"
+			(at 177.8 35.56 0)
+			(effects
+				(font
+					(size 1.27 1.27)
+				)
+				(hide yes)
+			)
+		)
+		(property "Mouser Part Number" "81-GCM188M8EH105KE8D"
+			(at 193.802 40.64 0)
+			(effects
+				(font
+					(size 1.27 1.27)
+				)
 			)
 		)
@@
 					(unit 1)
 				)
+			)
+		)
+	)
+	(symbol
+		(lib_id "Device:R_Shunt")
+		(at 168.91 76.2 0)
+		(unit 1)
+		(exclude_from_sim no)
+		(in_bom yes)
+		(on_board yes)
+		(dnp no)
+		(property "Reference" "R48"
+			(at 166.37 74.9299 0)
+			(effects
+				(font
+					(size 1.27 1.27)
+				)
+				(justify right)
+			)
+		)
+		(property "Value" "R_Shunt"
+			(at 166.37 77.4699 0)
+			(effects
+				(font
+					(size 1.27 1.27)
+				)
+				(justify right)
+			)
+		)
+		(property "Footprint" "samacsys:4wire_0603"
+			(at 167.132 76.2 90)
+			(effects
+				(font
+					(size 1.27 1.27)
+				)
+				(hide yes)
+			)
+		)
+		(property "Datasheet" "~"
+			(at 168.91 76.2 0)
+			(effects
+				(font
+					(size 1.27 1.27)
+				)
+				(hide yes)
+			)
+		)
+		(property "Description" "Shunt resistor"
+			(at 168.91 76.2 0)
+			(effects
+				(font
+					(size 1.27 1.27)
+				)
+				(hide yes)
+			)
+		)
+		(property "Manufacturer_Part_Number" "580060716002"
+			(at 168.91 76.2 0)
+			(effects
+				(font
+					(size 1.27 1.27)
+				)
+				(hide yes)
+			)
+		)
+		(property "Mouser Part Number" "710-580060716002"
+			(at 147.066 75.946 0)
+			(effects
+				(font
+					(size 1.27 1.27)
+				)
+			)
+		)
+		(pin "2"
+		)
+		(pin "1"
+		)
+		(pin "4"
+		)
+		(pin "3"
+		)
+		(instances
+			(project ""
+				(path "/21624bb8-7220-4725-ab4f-34c4768aac8d/c3cbd430-6fb2-4bfe-86b9-0dcdbd0b95f5"
+					(reference "R49")
+					(unit 1)
+				)
+				(path "/21624bb8-7220-4725-ab4f-34c4768aac8d/f72fcd55-797d-4de7-b16c-a295f170430e"
+					(reference "R48")
+					(unit 1)
+				)
+				(path "/21624bb8-7220-4725-ab4f-34c4768aac8d/fc458950-2711-4a11-802f-b3226dc264b9"
+					(reference "R50")
+					(unit 1)
+				)
