File: HARDWARE/FOC_CONTROLLER/FOC_CONTROLLER_V1/FOC_CONTROLLER_V1.kicad_sch (KiCad schematic)
At the start: 18 parts, among them IC1 STSPIN32G0A2

Commit message: update
Parts:
- added C24, C25, C26, C27: 47u, Capacitor_SMD:C_0805_2012Metric, symbol Device:C_Small
- added C28, C29: 100n, Capacitor_SMD:C_0201_0603Metric_Pad0.64x0.40mm_HandSolder, symbol Device:C_Small
- added C30: 1nF, Capacitor_SMD:C_0201_0603Metric_Pad0.64x0.40mm_HandSolder, symbol Device:C_Small
- added J1: SM04B-GHS-TB_LF__SN_, samacsys:SM04B-GHS-TB, symbol samacsys:SM04B-GHS-TB_LF__SN_
- added J2: SM06B-GHS-TB_LF__SN_, samacsys:SM06B-GHS-TB, symbol samacsys:SM06B-GHS-TB_LF__SN_
- added R40: 10k, Resistor_SMD:R_0201_0603Metric_Pad0.64x0.40mm_HandSolder, symbol Device:R_Small
- added R41: 100k, Resistor_SMD:R_0201_0603Metric_Pad0.64x0.40mm_HandSolder, symbol Device:R_Small
- added R42: 15k, Resistor_SMD:R_0201_0603Metric_Pad0.64x0.40mm_HandSolder, symbol Device:R_Small
- added R46: 18k, Resistor_SMD:R_0201_0603Metric_Pad0.64x0.40mm_HandSolder, symbol Device:R_Small
- added TP1, TP2, TP3, TP4: TestPoint, MountingHole:MountingHole_2.2mm_M2_Pad_Via, symbol Connector:TestPoint
Connections:
- net HALL2 is gone; now on net UART_TX: IC1.13 (PA1)
- net HALL3 is gone; now on net UART_RX: IC1.14 (PA2)
- net +3.3V: now also R40.1, R41.1, R46.1
- net GND: now also C24.2, C25.2, C26.2, C27.2, C28.2, C29.2, C30.2, J1.3, J2.1, J2.2, R42.2, TP1.1, TP2.1, TP3.1, TP4.1
- net SWCLK: now also J1.2
- net SWDIO: now also J1.1
- net UART_RX: now also J2.3; no longer IC1.45 (PB7)
- net UART_TX: now also J2.4; no longer IC1.43 (PB6)
- net VBAT+: now also C24.1, C25.1, C26.1, C27.1, J2.5, J2.6
- net MGL: now reaches IC1.15 (PA3)
- net MGH: now reaches IC1.16 (PA4)
- net at IC1.17 (PA5): now also C29.1, R41.2, R42.1
- net SHUNT+AFTER: now reaches IC1.25 (OCCOMP)
- net SHUNT+AFTER: now also C30.1, R46.2
- net BTN: now reaches IC1.39 (PA12_[PA10])
- net BTN: now also C28.1, J1.4, R40.2
- net SPI2_CS: now reaches IC1.42 (PA15)
- net HALL1 renamed SPI2_SCK
- new net SPI2_MISO: IC1.43 (PB6)
- new net SPI2_MOSI: IC1.45 (PB7)
- no-connect marks 4 -> 2
Other:
- sheet HALL ports: added MGH, MGL, SPI_CS, SPI_MISO, SPI_MOSI, SPI_SCK; removed CSQ, DATA, HALLA, HALLB, HALLC, SCK
- sheet U ports: added SHUNTAFTER+; removed none
- sheet V ports: added SHUNTAFTER+; removed none
- sheet W ports: added SHUNTAFTER+; removed none
- note added: "A TROUVER"
- note added: "MAIN_CONNECTOR"
- note added: "NTCSC0201E3104FXHT 1% 4311K 0201"
- note added: "SWD"
- moved on the sheet: C1, C10, C11, C12, C2, C3, C4, C5, C6, C7, C8, C9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

Commit message: update
Parts:
- added D8: LED, LED_SMD:LED_0402_1005Metric, symbol Device:LED
- added R47: 1k, Resistor_SMD:R_0201_0603Metric_Pad0.64x0.40mm_HandSolder, symbol Device:R_Small
Connections:
- net GND: now also J2.5, J2.6, R47.1; no longer J2.1, J2.2
- net SWCLK: now also J1.1; no longer J1.2
- net SWDIO: now also J1.2; no longer J1.1
- net VBAT+: now also J2.1, J2.2; no longer J2.5, J2.6
- net at IC1.10 (PF0-OSC_IN): now also D8.2 (A)
- new net: D8.1 (K), R47.2
- no-connect marks 2 -> 1

Commit message: up
Connections:
- net MGH: now also IC1.13 (PA1); no longer IC1.16 (PA4)
- net MGL: now also IC1.16 (PA4); no longer IC1.15 (PA3)
- net UART_RX: now also IC1.15 (PA3); no longer IC1.14 (PA2)
- net UART_TX: now also IC1.14 (PA2); no longer IC1.13 (PA1)
Changed lines of the file:
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@@
-	(wire
-		(pts
-			(xy 326.39 132.08) (xy 326.39 130.81)
-		)
-		(stroke
-			(width 0)
-			(type default)
-		)
-	)
 	(wire
 		(pts
@@
 	(wire
 		(pts
+			(xy 334.01 137.16) (xy 334.01 130.81)
+		)
+		(stroke
+			(width 0)
+			(type default)
+		)
+	)
+	(wire
+		(pts
 			(xy 248.92 111.76) (xy 252.73 111.76)
 		)
@@
 	(wire
 		(pts
-			(xy 331.47 130.81) (xy 331.47 135.89)
-		)
-		(stroke
-			(width 0)
-			(type default)
-		)
-	)
-	(wire
-		(pts
 			(xy 353.06 158.75) (xy 353.06 160.02)
 		)
@@
 	(wire
 		(pts
-			(xy 328.93 132.08) (xy 328.93 130.81)
-		)
-		(stroke
-			(width 0)
-			(type default)
-		)
-	)
-	(wire
-		(pts
 			(xy 382.27 85.09) (xy 386.08 85.09)
 		)
@@
 	(wire
 		(pts
+			(xy 331.47 133.35) (xy 331.47 130.81)
+		)
+		(stroke
+			(width 0)
+			(type default)
+		)
+	)
+	(wire
+		(pts
 			(xy 302.26 105.41) (xy 318.77 105.41)
 		)
@@
 	(wire
 		(pts
-			(xy 334.01 130.81) (xy 334.01 135.89)
-		)
-		(stroke
-			(width 0)
-			(type default)
-		)
-	)
-	(wire
-		(pts
 			(xy 356.87 50.8) (xy 356.87 57.15)
 		)
@@
 	(wire
 		(pts
+			(xy 326.39 137.16) (xy 326.39 130.81)
+		)
+		(stroke
+			(width 0)
+			(type default)
+		)
+	)
+	(wire
+		(pts
 			(xy 374.65 110.49) (xy 374.65 132.08)
 		)
@@
 		(pts
 			(xy 367.03 43.18) (xy 367.03 45.72)
+		)
+		(stroke
+			(width 0)
+			(type default)
+		)
+	)
+	(wire
+		(pts
+			(xy 328.93 133.35) (xy 328.93 130.81)
 		)
 		(stroke
@@
 	)
 	(label "UART_TX"
-		(at 326.39 132.08 270)
+		(at 328.93 133.35 270)
 		(effects
 			(font
@@
 	)
 	(label "MGL"
-		(at 331.47 135.89 270)
+		(at 334.01 137.16 270)
 		(effects
 			(font
@@
 	)
 	(label "MGH"
-		(at 334.01 135.89 270)
+		(at 326.39 137.16 270)
 		(effects
 			(font
@@
 	)
 	(label "UART_RX"
-		(at 328.93 132.08 270)
-		(effects
-			(font
+		(at 331.47 133.35 270)
+		(effects
+			(font

Commit message: update foc
Parts:
- removed J1: SM04B-GHS-TB_LF__SN_, samacsys:SM04B-GHS-TB, symbol samacsys:SM04B-GHS-TB_LF__SN_
- added C23, C31, C33, C34, C35, C36: 22u, Capacitor_SMD:C_0805_2012Metric, symbol Device:C_Small
- added J1: SM06B-GHS-TB_LF__SN_, samacsys:SM06B-GHS-TB, symbol samacsys:SM06B-GHS-TB_LF__SN_
- added TP10, TP11, TP12, TP13, TP15, TP8, TP9: TestPoint, samacsys:pad_0.7mm, symbol Connector:TestPoint
- added TP5, TP6, TP7: TestPoint, samacsys:hole_1.5mm, symbol Connector:TestPoint
- C10: Manufacturer_Part_Number (none) -> GRM188R71E224KA88; Mouser Part Number (none) -> 81-GRM188R71E224KA88
- C11: Manufacturer_Part_Number (none) -> GRM188R61E106MA3D; Mouser Part Number (none) -> 81-GRM188R61E106MA3D
- C2, C3, C4: Manufacturer_Part_Number (none) -> GCM188M8EH105KE8D; Mouser Part Number (none) -> 81-GCM188M8EH105KE8D
- C24, C25, C26, C27: value 47u -> 22u; Manufacturer_Part_Number (none) -> GRM21BR61E226ME4L; Mouser Part Number (none) -> 81-GRM21BR61E226ME4L
- C7: Manufacturer_Part_Number (none) -> GRM21BR61A476ME5L; Mouser Part Number (none) -> 81-GRM21BR61A476ME5L
- C8: value 100n -> 10n
- IC1: Mouser Part Number (none) -> 511-STSPIN32G0A2
- R41: Manufacturer_Part_Number (none) -> NTCSC0201E3104FX; Mouser Part Number (none) -> 594-NTCSC0201E3104FX
- TP1, TP2, TP3, TP4: now not fitted
Connections:
- net +3.3V: now also J1.4
- net BTN: now also J1.6
- net GND: now also J2.7, J2.8, C23.2, C31.2, C33.2, C34.2, C35.2, C36.2, J1.5, J1.7, J1.8, TP15.1
- net ISNSU: now also IC1.20 (PA7); no longer IC1.18 (PA6)
- net ISNSV: now also IC1.18 (PA6); no longer IC1.20 (PA7)
- net MGH: now also TP12.1
- net MGL: now also TP11.1
- net OP2N: now also TP9.1
- net OP2O: now also TP8.1
- net OP2P: now also TP10.1
- net OUTU: now also TP5.1
- net OUTV: now also TP6.1
- net OUTW: now also TP7.1
- net SPI2_MOSI: now also TP13.1
- net SWCLK: now also J1.2
- net SWDIO: now also J1.3
- net VBAT+: now also C23.1, C31.1, C33.1, C34.1, C35.1, C36.1
- net NRST: now reaches C9.1, R3.2, S1.1 (NO_1), S1.2 (NO_2)
- net NRST: now also J1.1
Other:
- sheet U ports: added INPUTAOP+, INPUTAOP-, SHUNT+, SHUNT-; removed none
- sheet V ports: added INPUTAOP+, INPUTAOP-, SHUNT+, SHUNT-; removed none
- sheet W ports: added INPUTAOP+, INPUTAOP-, SHUNT+, SHUNT-; removed none
- note added: "1% 4311K 0201"
- note removed: "A TROUVER"
- note removed: "NTCSC0201E3104FXHT 1% 4311K 0201"
- moved on the sheet: C24, C25, C26, C27

Commit message: jgfffn
Parts:
- TP1, TP2, TP3, TP4: footprint MountingHole:MountingHole_2.2mm_M2_Pad_Via -> samacsys:m3test
Other:
- note added: "m3"
Changed lines of the file:
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@@
 		)
 	)
+	(text "m3\n"
+		(exclude_from_sim no)
+		(at 110.236 89.916 0)
+		(effects
+			(font
+				(size 1.27 1.27)
+			)
+		)
+	)
 	(text "MAIN_CONNECTOR"
 		(exclude_from_sim no)
@@
 	)
 	(junction
-		(at 129.54 85.09)
-		(diameter 0)
-		(color 0 0 0 0)
-	)
-	(junction
 		(at 252.73 111.76)
 		(diameter 0)
@@
 	)
 	(junction
+		(at 132.08 85.09)
+		(diameter 0)
+		(color 0 0 0 0)
+	)
+	(junction
 		(at 382.27 85.09)
 		(diameter 0)
@@
 	)
 	(junction
+		(at 123.19 85.09)
+		(diameter 0)
+		(color 0 0 0 0)
+	)
+	(junction
 		(at 234.95 127)
 		(diameter 0)
@@
 	)
 	(junction
-		(at 123.19 85.09)
-		(diameter 0)
-		(color 0 0 0 0)
-	)
-	(junction
 		(at 129.54 208.28)
 		(diameter 0)
@@
 	(wire
 		(pts
+			(xy 132.08 85.09) (xy 146.05 85.09)
+		)
+		(stroke
+			(width 0)
+			(type default)
+		)
+	)
+	(wire
+		(pts
 			(xy 353.06 158.75) (xy 353.06 160.02)
 		)
@@
 	(wire
 		(pts
+			(xy 123.19 85.09) (xy 132.08 85.09)
+		)
+		(stroke
+			(width 0)
+			(type default)
+		)
+	)
+	(wire
+		(pts
 			(xy 64.77 90.17) (xy 62.23 90.17)
 		)
@@
 	(wire
 		(pts
-			(xy 123.19 85.09) (xy 129.54 85.09)
-		)
-		(stroke
-			(width 0)
-			(type default)
-		)
-	)
-	(wire
-		(pts
 			(xy 128.27 242.57) (xy 143.51 242.57)
 		)
@@
 	(wire
 		(pts
-			(xy 129.54 85.09) (xy 142.24 85.09)
-		)
-		(stroke
-			(width 0)
-			(type default)
-		)
-	)
-	(wire
-		(pts
 			(xy 234.95 127) (xy 252.73 127)
 		)
@@
 			)
 		)
-		(property "Footprint" "MountingHole:MountingHole_2.2mm_M2_Pad_Via"
+		(property "Footprint" "samacsys:m3test"
 			(at 121.92 85.09 0)
 			(effects
@@
 	)
 	(symbol
+		(lib_id "Connector:TestPoint")
+		(at 132.08 85.09 0)
+		(unit 1)
+		(exclude_from_sim no)
+		(in_bom yes)
+		(on_board yes)
+		(dnp yes)
+		(fields_autoplaced yes)
+		(property "Reference" "TP3"
+			(at 134.62 80.5179 0)
+			(effects
+				(font
+					(size 1.27 1.27)
+				)
+				(justify left)
+			)
+		)
+		(property "Value" "TestPoint"
+			(at 134.62 83.0579 0)
+			(effects
+				(font
+					(size 1.27 1.27)
+				)
+				(justify left)
+			)
+		)
+		(property "Footprint" "samacsys:m3test"
+			(at 137.16 85.09 0)
+			(effects
+				(font
+					(size 1.27 1.27)
+				)
+				(hide yes)
+			)
+		)
+		(property "Datasheet" "~"
+			(at 137.16 85.09 0)
+			(effects
+				(font
+					(size 1.27 1.27)
+				)
+				(hide yes)
+			)
+		)
+		(property "Description" "test point"
+			(at 132.08 85.09 0)
+			(effects
+				(font
+					(size 1.27 1.27)
+				)
+				(hide yes)
+			)
+		)
+		(pin "1"
+		)
+		(instances
+			(project "FOC_CONTROLLER_V1"
+				(path "/21624bb8-7220-4725-ab4f-34c4768aac8d"
+					(reference "TP3")
+					(unit 1)
+				)
+			)
+		)
+	)
+	(symbol
 		(lib_id "power:GND")
 		(at 222.25 217.17 90)
@@
 	)
 	(symbol
-		(lib_id "Connector:TestPoint")
-		(at 142.24 85.09 0)
-		(unit 1)
-		(exclude_from_sim no)
-		(in_bom yes)
-		(on_board yes)
-		(dnp yes)
-		(fields_autoplaced yes)
-		(property "Reference" "TP4"
-			(at 144.78 80.5179 0)
-			(effects
-				(font
-					(size 1.27 1.27)
-				)
-				(justify left)
-			)
-		)
-		(property "Value" "TestPoint"
-			(at 144.78 83.0579 0)
-			(effects
-				(font
-					(size 1.27 1.27)
-				)
-				(justify left)
-			)
-		)
-		(property "Footprint" "MountingHole:MountingHole_2.2mm_M2_Pad_Via"
-			(at 147.32 85.09 0)
-			(effects
-				(font
-					(size 1.27 1.27)
-				)
-				(hide yes)
-			)
-		)
-		(property "Datasheet" "~"
-			(at 147.32 85.09 0)
-			(effects
-				(font
-					(size 1.27 1.27)
-				)
-				(hide yes)
-			)
-		)
-		(property "Description" "test point"
-			(at 142.24 85.09 0)
-			(effects
-				(font
-					(size 1.27 1.27)
-				)
-				(hide yes)
-			)
-		)
-		(pin "1"
-		)
-		(instances
-			(project "FOC_CONTROLLER_V1"
-				(path "/21624bb8-7220-4725-ab4f-34c4768aac8d"
-					(reference "TP4")
-					(unit 1)
-				)
-			)
-		)
-	)
-	(symbol
 		(lib_id "power:+3.3V")
 		(at 367.03 132.08 90)
@@
 	)
 	(symbol
-		(lib_id "Connector:TestPoint")
-		(at 129.54 85.09 0)
-		(unit 1)
-		(exclude_from_sim no)
-		(in_bom yes)
-		(on_board yes)
-		(dnp yes)
-		(fields_autoplaced yes)
-		(property "Reference" "TP3"
-			(at 132.08 80.5179 0)
-			(effects
-				(font
-					(size 1.27 1.27)
-				)
-				(justify left)
-			)
-		)
-		(property "Value" "TestPoint"
-			(at 132.08 83.0579 0)
-			(effects
-				(font
-					(size 1.27 1.27)
-				)
-				(justify left)
-			)
-		)
-		(property "Footprint" "MountingHole:MountingHole_2.2mm_M2_Pad_Via"
-			(at 134.62 85.09 0)
-			(effects
-				(font
-					(size 1.27 1.27)
-				)
-				(hide yes)
-			)
-		)
-		(property "Datasheet" "~"
-			(at 134.62 85.09 0)
-			(effects
-				(font
-					(size 1.27 1.27)
-				)
-				(hide yes)
-			)
-		)
-		(property "Description" "test point"
-			(at 129.54 85.09 0)
-			(effects
-				(font
-					(size 1.27 1.27)
-				)
-				(hide yes)
-			)
-		)
-		(pin "1"
-		)
-		(instances
-			(project "FOC_CONTROLLER_V1"
-				(path "/21624bb8-7220-4725-ab4f-34c4768aac8d"
-					(reference "TP3")
-					(unit 1)
-				)
-			)
-		)
-	)
-	(symbol
 		(lib_id "power:GND")
 		(at 304.8 166.37 0)
@@
 			)
 		)
-		(property "Footprint" "MountingHole:MountingHole_2.2mm_M2_Pad_Via"
+		(property "Footprint" "samacsys:m3test"
 			(at 107.95 85.09 0)
 			(effects
@@
 					(unit 1)
 				)
+			)
+		)
+	)
+	(symbol
+		(lib_id "Connector:TestPoint")
+		(at 146.05 85.09 0)
+		(unit 1)
+		(exclude_from_sim no)
+		(in_bom yes)
+		(on_board yes)
+		(dnp yes)
+		(fields_autoplaced yes)
+		(property "Reference" "TP4"
+			(at 148.59 80.5179 0)
+			(effects
+				(font
+					(size 1.27 1.27)
+				)
+				(justify left)
+			)
+		)
+		(property "Value" "TestPoint"
+			(at 148.59 83.0579 0)
+			(effects
+				(font
+					(size 1.27 1.27)
+				)
+				(justify left)
+			)
+		)
+		(property "Footprint" "samacsys:m3test"
+			(at 151.13 85.09 0)
+			(effects
+				(font
+					(size 1.27 1.27)
+				)
+				(hide yes)
+			)
+		)
+		(property "Datasheet" "~"
+			(at 151.13 85.09 0)
+			(effects
+				(font
+					(size 1.27 1.27)
+				)
+				(hide yes)
+			)
+		)
+		(property "Description" "test point"
+			(at 146.05 85.09 0)
+			(effects
+				(font
+					(size 1.27 1.27)
+				)
+				(hide yes)
+			)
+		)
+		(pin "1"
+		)
+		(instances
+			(project "FOC_CONTROLLER_V1"
+				(path "/21624bb8-7220-4725-ab4f-34c4768aac8d"
+					(reference "TP4")
+					(unit 1)
+				)
