File: HARDWARE/PCB_PAPI/connector.kicad_sch (KiCad schematic)
At the start: 20 parts, among them J1 USB4110-GF-A, J3 SM03B-GHS-TB_LF__SN_, J4 XT30AW-M, J7 Conn_01x03_Pin, J8 Conn_01x03_Pin, J9 SM05B-GHS-TB_LF__SN_

Commit message: update
Parts:
- removed CAN1, CAN2: SM04B-GHE-TB, Connector_JST:JST_GH_SM04B-GHS-TB_1x04-1MP_P1.25mm_Horizontal, symbol fc_h7:jst_4_pin
- removed J3: SM03B-GHS-TB_LF__SN_, SM03BGHSTBLFSN, symbol SamacSys_Parts:SM03B-GHS-TB_LF__SN_
- removed J4: XT30AW-M, XT30AWM, symbol SamacSys_Parts:XT30AW-M
- removed J7, J8: Conn_01x03_Pin, symbol Connector:Conn_01x03_Pin
- removed J9: SM05B-GHS-TB_LF__SN_, SM05B-GHS-TB, symbol SamacSys_Parts:SM05B-GHS-TB_LF__SN_
- added ACCESSORIES1: SM10B-SRSS-TB_LF__SN_, samacsys:SM10B-SRSS-TB, symbol samacsys:SM10B-SRSS-TB_LF__SN_
- added J3: XT30PW-M, samacsys:XT30PWM, symbol samacsys:XT30PW-M
- added SWD1: SM04B-GHE-TB, Connector_JST:JST_GH_SM04B-GHS-TB_1x04-1MP_P1.25mm_Horizontal, symbol fc_h7:jst_4_pin
- added USBJUMP1: Conn_01x08_Pin, Connector_PinHeader_1.00mm:PinHeader_2x04_P1.00mm_Vertical_SMD, symbol Connector:Conn_01x08_Pin
- renumbered CAN4 to LIDAR1, CAN3 to TOF1, CAN6 to TOF2, CAN5 to TOF3
Connections:
- net +5V: no longer LIDAR1.4, TOF1.1, TOF2.1, TOF3.1
- net GND: now also ACCESSORIES1.MP, J3.2, J3.3, J3.4, SWD1.MP; no longer ESC1.6, ESC1.7, ESC1.8, ESC2.6, ESC2.7, ESC2.8, ESC3.6, ESC3.7, ESC3.8, LIDAR1.2, TOF1.4, TOF2.4, TOF3.4
- net GPIO_Mot1: no longer ESC1.3
- net GPIO_Mot2: no longer ESC2.3
- net GPIO_Mot3: no longer ESC3.3
- net PWM_LiDAR: no longer LIDAR1.1
- net RX_LiDAR: no longer LIDAR1.3
- net RX_Mot1: no longer ESC1.1
- net RX_Mot2: no longer ESC2.1
- net RX_Mot3: no longer ESC3.1
- net SCL_TOF1: no longer TOF1.2
- net SCL_TOF2: no longer TOF2.2
- net SCL_TOF3: no longer TOF3.2
- net SDA_TOF1: no longer TOF1.3
- net SDA_TOF2: no longer TOF2.3
- net SDA_TOF3: no longer TOF3.3
- net TX_Mot1: no longer ESC1.2
- net TX_Mot2: no longer ESC2.2
- net TX_Mot3: no longer ESC3.2
- net VBAT+: no longer ESC1.4, ESC1.5, ESC2.4, ESC2.5, ESC3.4, ESC3.5
- net DATA-OUT: now reaches R9.2
- net DATA+OUT: now reaches R10.2
- new net BAT+: J3.1
Other:
- note added: "ACCESSORIES"
- note added: "checker"
- note removed: "ARGB LED Conn"
- note removed: "OLED 1"
- note removed: "OLED2"
- moved on the sheet: ESC3, LIDAR1

Commit message: up
Parts:
- added H1, H2, H3: MountingHole_Pad, MountingHole:MountingHole_2.5mm_Pad_Via, symbol Mechanical:MountingHole_Pad
Connections:
- net D+: now also J1.A6 (D+), J1.B6 (D+), R10.1
- net D-: now also J1.A7 (D-), J1.B7 (D-), R9.1
- net GND: now also ESC1.1, ESC1.2, ESC1.3, ESC2.1, ESC2.2, ESC2.3, ESC3.1, ESC3.2, ESC3.3, H1.1, H2.1, H3.1
- net GPIO_Mot1: now also ESC1.4
- net GPIO_Mot2: now also ESC2.4
- net GPIO_Mot3: now also ESC3.4
- net HP+: now also ACCESSORIES1.1
- net HP-: now also ACCESSORIES1.2
- net RX_Mot1: now also ESC1.6
- net RX_Mot2: now also ESC2.6
- net RX_Mot3: now also ESC3.6
- net TX_Mot1: now also ESC1.5
- net TX_Mot2: now also ESC2.5
- net TX_Mot3: now also ESC3.5
- net VBAT+: now also ESC1.7, ESC1.8, ESC2.7, ESC2.8, ESC3.7, ESC3.8

Commit message: updfate
Parts:
- removed ACCESSORIES1: SM10B-SRSS-TB_LF__SN_, samacsys:SM10B-SRSS-TB, symbol samacsys:SM10B-SRSS-TB_LF__SN_
- added J4: SM02B-GHS-TB_LF__SN_, SM02BGHSTBLFSN, symbol samacsys:SM02B-GHS-TB_LF__SN_
- added J5: SM12B-SRSS-TB_LF__SN_, SM12BSRSSTBLFSN, symbol samacsys:SM12B-SRSS-TB_LF__SN_
- LIDAR1, TOF1, TOF2, TOF3: footprint Connector_JST:JST_GH_SM04B-GHS-TB_1x04-1MP_P1.25mm_Horizontal -> Connector_JST:JST_GH_BM04B-GHS-TBT_1x04-1MP_P1.25mm_Vertical
Connections:
- net +3.3V: now also TOF1.1, TOF2.1, TOF3.1, J5.11
- net +5V: now also LIDAR1.4, J5.7
- net ARGB Din: now also J5.5
- net D+: now also D1.1 (I/O_1); no longer D1.3 (I/O_2)
- net D+ ESP32: now also USBJUMP1.5 (Pin_5)
- net D+ STM32: now also USBJUMP1.1 (Pin_1)
- net D-: now also D1.3 (I/O_2); no longer D1.1 (I/O_1)
- net D- ESP32: now also USBJUMP1.7 (Pin_7)
- net D- STM32: now also USBJUMP1.3 (Pin_3)
- net DATA+OUT: now also USBJUMP1.2 (Pin_2), USBJUMP1.6 (Pin_6)
- net DATA-OUT: now also USBJUMP1.4 (Pin_4), USBJUMP1.8 (Pin_8)
- net GND: now also LIDAR1.2, SWD1.4, TOF1.4, TOF2.4, TOF3.4, J4.3, J4.4, J5.13 (MP1), J5.14 (MP2), J5.6, J5.8
- net GND_CONTROLLED-: now also J5.12
- net HP+: now also J5.1
- net HP-: now also J5.2
- net NRST: now also SWD1.3
- net PWM_LiDAR: now also LIDAR1.1
- net RX_LiDAR: now also LIDAR1.3
- net SCL_OLED1: now also J5.9
- net SCL_TOF1: now also TOF1.2
- net SCL_TOF2: now also TOF2.2
- net SCL_TOF3: now also TOF3.2
- net SDA_OLED1: now also J5.10
- net SDA_TOF1: now also TOF1.3
- net SDA_TOF2: now also TOF2.3
- net SDA_TOF3: now also TOF3.3
- net SWCLK: now also SWD1.2
- net SWDIO: now also SWD1.1
- new net BTN_POWER_A: J4.1
- new net BTN_POWER_B: J4.2
- new net RX_SUP: J5.3
- new net TX_SUP: J5.4
Other:
- note added: "POWER SWITCH"
- moved on the sheet: H1, H2, H3, J3

Commit message: update
Changed lines of the file:
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@@
+	(wire
+		(pts
+			(xy 91.44 55.88) (xy 101.6 55.88)
+		)
+		(stroke
+			(width 0)
+			(type default)
+		)
+	)
 	(wire
 		(pts
@@
 		)
 		(stroke
-			(width 0)
-			(type default)
-		)
-	)
-	(wire
-		(pts
-			(xy 101.6 55.88) (xy 91.44 55.88)
-		)
-		(stroke

Commit message: up
Connections:
- net +5V: no longer J5.7
- new net 4.5V: J5.7
Changed lines of the file:
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@@
+		)
+	)
+	(global_label "4.5V"
+		(shape input)
+		(at 73.66 151.13 0)
+		(fields_autoplaced yes)
+		(effects
+			(font
+				(size 1.27 1.27)
+			)
+			(justify left)
+		)
+		(property "Intersheetrefs" "${INTERSHEET_REFS}"
+			(at 80.7576 151.13 0)
+			(effects
+				(font
+					(size 1.27 1.27)
+				)
+				(justify left)
+				(hide yes)
+			)
 		)
 	)
@@
 					(unit 1)
 				)
-			)
-		)
-	)
-	(symbol
-		(lib_id "power:+5V")
-		(at 73.66 151.13 270)
-		(unit 1)
-		(exclude_from_sim no)
-		(in_bom yes)
-		(on_board yes)
-		(dnp no)
-		(property "Reference" "#PWR068"
-			(at 69.85 151.13 0)
-			(effects
-				(font
-					(size 1.27 1.27)
-				)
-				(hide yes)
-			)
-		)
-		(property "Value" "+5V"
-			(at 77.47 151.1301 90)
-			(effects
-				(font
-					(size 1.27 1.27)
-				)
-				(justify left)
-			)
-		)
-		(property "Footprint" ""
-			(at 73.66 151.13 0)
-			(effects
-				(font
-					(size 1.27 1.27)
-				)
-				(hide yes)
-			)
-		)
-		(property "Datasheet" ""
-			(at 73.66 151.13 0)
-			(effects
-				(font
-					(size 1.27 1.27)
-				)
-				(hide yes)
-			)
-		)
-		(property "Description" "Power symbol creates a global label with name \"+5V\""
-			(at 73.66 151.13 0)
-			(effects
-				(font
-					(size 1.27 1.27)
-				)
-				(hide yes)
-			)
-		)
-		(pin "1"
-		)
-		(instances
-			(project "PCB_PAPI"
-				(path "/64301b3d-8a16-47d9-a9c6-0068257932ba/3b0227fd-8888-44e2-94a5-1880f3393fd0"
-					(reference "#PWR068")
-					(unit 1)
-				)

Commit message: up
Parts:
- J4: footprint SM02BGHSTBLFSN -> samacsys:SM02BGHSTBLFSN
- J5: footprint SM12BSRSSTBLFSN -> samacsys:SM12BSRSSTBLFSN
- R7, R8: footprint Resistor_SMD:R_0201_0603Metric -> samacsys:R_0201_custom
Changed lines of the file:
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@@
 			)
 		)
-		(property "Footprint" "SM02BGHSTBLFSN"
+		(property "Footprint" "samacsys:SM02BGHSTBLFSN"
 			(at 67.31 322.25 0)
 			(effects
@@
 			)
 		)
-		(property "Footprint" "SM12BSRSSTBLFSN"
+		(property "Footprint" "samacsys:SM12BSRSSTBLFSN"
 			(at 69.85 230.81 0)
 			(effects
@@
 			)
 		)
-		(property "Footprint" "Resistor_SMD:R_0201_0603Metric"
+		(property "Footprint" "samacsys:R_0201_custom"
 			(at 93.98 49.53 0)
 			(effects
@@
 			)
 		)
-		(property "Footprint" "Resistor_SMD:R_0201_0603Metric"
+		(property "Footprint" "samacsys:R_0201_custom"
 			(at 93.98 46.99 0)
 			(effects
