File: HARDWARE/PCB_PAPI/PCB_PAPI.kicad_pcb (KiCad board)
At the start: 2 copper layers, 50 x 43.3 mm, 116 parts, among them IC1 LMR51625YFDDCR, IC2 LDO40LPU33RY, IC3 LDO40LPU33RY, IC4 ESP32-C6FH4, IC5 ADXL343BCCZ-RL, IC6 MAX98357AETE+, IC7 W25Q128JVPIQ_TR, J1 USB4110-GF-A, J2 636101111001, J3 XT30PW-M, Q1 STR2N2VH5, Q3 SQS401EN-T1_BE3, U1 STM32H743VIHx, Y1 CSTNE8M00GH5C000R0, Y2 LFXTAL069527REEL

Commit message: up
Parts:
- added H1: MountingHole_Pad, MountingHole:MountingHole_2.5mm_Pad_Via, F.Cu at (127.1, 86.0)
- added H2: MountingHole_Pad, MountingHole:MountingHole_2.5mm_Pad_Via, F.Cu at (95.9, 104.0)
- added H3: MountingHole_Pad, MountingHole:MountingHole_2.5mm_Pad_Via, F.Cu at (127.1, 122.5)
- C10, C11, C12, C13, C14, C15, C16, C17, C18, C19, C2, C20, C3, C31, C33, C34, C35, C36, C37, C4, C6, C7, C8, IC1, L1, Q1, R11, R12, R13, R14, R15, R16, R21, R26, R27: moved to B.Cu
- Q3: moved to F.Cu
- moved R15 95.2 mm to (133.9, 114.8), turned to 150 degrees
- moved R16 93.6 mm to (132.4, 114.0), turned to 150 degrees
- moved Q1 91.0 mm to (134.2, 112.1), turned to 60 degrees
- moved R34 88.7 mm to (130.1, 109.5), turned to 180 degrees
- moved R17 79.8 mm to (117.8, 98.9)
- moved R13 79.2 mm to (115.2, 102.6), turned to -90 degrees
- moved C17 78.7 mm to (115.2, 104.1), turned to 90 degrees
- moved R12 78.4 mm to (114.9, 108.5)
- moved R14 76.3 mm to (115.2, 107.4), turned to -90 degrees
- moved R11 76.0 mm to (112.5, 108.5)
- moved IC1 75.6 mm to (113.0, 106.0), turned to 90 degrees
- moved C28 70.9 mm to (134.3, 101.0), turned to 90 degrees
- moved C30 70.3 mm to (133.6, 103.1)
- moved C19 69.5 mm to (114.0, 97.5), turned to 90 degrees
- moved R18 69.4 mm to (109.6, 118.8), turned to 180 degrees
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Connections:
- ACCESSORIES1 pad 1: unconnected-(ACCESSORIES1-Pad1) -> /CONNECTOR/HP+
- ACCESSORIES1 pad 2: unconnected-(ACCESSORIES1-Pad2) -> /CONNECTOR/HP-
- ESC1 pad 1: unconnected-(ESC1-Pad1) -> GND
- ESC1 pad 2: unconnected-(ESC1-Pad2) -> GND
- ESC1 pad 3: unconnected-(ESC1-Pad3) -> GND
- ESC1 pad 4: unconnected-(ESC1-Pad4) -> /CONNECTOR/GPIO_Mot1
- ESC1 pad 5: unconnected-(ESC1-Pad5) -> /CONNECTOR/TX_Mot1
- ESC1 pad 6: unconnected-(ESC1-Pad6) -> /CONNECTOR/RX_Mot1
- ESC1 pad 7: unconnected-(ESC1-Pad7) -> VBAT+
- ESC1 pad 8: unconnected-(ESC1-Pad8) -> VBAT+
- ESC2 pad 1: unconnected-(ESC2-Pad1) -> GND
- ESC2 pad 2: unconnected-(ESC2-Pad2) -> GND
- ESC2 pad 3: unconnected-(ESC2-Pad3) -> GND
- ESC2 pad 4: unconnected-(ESC2-Pad4) -> /CONNECTOR/GPIO_Mot2
- ESC2 pad 5: unconnected-(ESC2-Pad5) -> /CONNECTOR/TX_Mot2
- ESC2 pad 6: unconnected-(ESC2-Pad6) -> /CONNECTOR/RX_Mot2
- ESC2 pad 7: unconnected-(ESC2-Pad7) -> VBAT+
- ESC2 pad 8: unconnected-(ESC2-Pad8) -> VBAT+
- ESC3 pad 1: unconnected-(ESC3-Pad1) -> GND
- ESC3 pad 2: unconnected-(ESC3-Pad2) -> GND
- ESC3 pad 3: unconnected-(ESC3-Pad3) -> GND
- ESC3 pad 4: unconnected-(ESC3-Pad4) -> /CONNECTOR/GPIO_Mot3
- ESC3 pad 5: unconnected-(ESC3-Pad5) -> /CONNECTOR/TX_Mot3
- ESC3 pad 6: unconnected-(ESC3-Pad6) -> /CONNECTOR/RX_Mot3
- ESC3 pad 7: unconnected-(ESC3-Pad7) -> VBAT+
- ESC3 pad 8: unconnected-(ESC3-Pad8) -> VBAT+
- J1 pad A6: Net-(J1-D+-PadA6) -> /CONNECTOR/D+
- J1 pad A7: Net-(J1-D--PadA7) -> /CONNECTOR/D-
- J1 pad B6: Net-(J1-D+-PadA6) -> /CONNECTOR/D+
- J1 pad B7: Net-(J1-D--PadA7) -> /CONNECTOR/D-
- R10 pad 1: Net-(J1-D+-PadA6) -> /CONNECTOR/D+
- R9 pad 1: Net-(J1-D--PadA7) -> /CONNECTOR/D-

Commit message: updfate
Parts:
- removed ACCESSORIES1: SM10B-SRSS-TB_LF__SN_, samacsys:SM10B-SRSS-TB
- removed H1, H2: MountingHole_Pad, MountingHole:MountingHole_2.5mm_Pad_Via
- added H3: MountingHole_Pad, MountingHole:MountingHole_2.5mm_Pad_Via, F.Cu at (139.5, 101.2)
- added H3: MountingHole_Pad, MountingHole:MountingHole_2.5mm_Pad_Via, F.Cu at (108.0, 83.0)
- added J4: SM02B-GHS-TB_LF__SN_, samacsys:SM02BGHSTBLFSN, B.Cu at (144.8, 92.3)
- added J5: SM12B-SRSS-TB_LF__SN_, samacsys:SM12BSRSSTBLFSN, F.Cu at (145.3, 92.3)
- LIDAR1, TOF1, TOF2, TOF3: footprint Connector_JST:JST_GH_SM04B-GHS-TB_1x04-1MP_P1.25mm_Horizontal -> Connector_JST:JST_GH_BM04B-GHS-TBT_1x04-1MP_P1.25mm_Vertical
- R34: moved to B.Cu
- moved H3 59.0 mm to (139.5, 64.8)
- moved R16 32.5 mm to (147.3, 85.2), turned to 60 degrees
- moved R15 31.1 mm to (146.5, 86.4), turned to 60 degrees
- moved Q1 28.3 mm to (148.7, 87.8), turned to -30 degrees
- moved R9 25.9 mm to (131.1, 70.3)
- moved Y2 24.8 mm to (143.4, 85.6)
- moved C38 24.8 mm to (144.8, 85.7)
- moved C18 24.8 mm to (124.3, 76.1)
- moved C23 24.7 mm to (127.1, 76.0)
- moved C31 24.7 mm to (143.8, 80.7)
- moved C33 24.7 mm to (144.7, 84.0)
- moved C45 24.7 mm to (137.5, 97.1)
- moved R18 24.7 mm to (121.9, 97.4)
- moved R27 24.7 mm to (130.8, 92.4)
- moved S1 24.7 mm to (125.2, 89.1)
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Connections:
- net /POWER SUPPLY/POWERSWITCHA renamed /BTN_A
- net /STM32/BOOT0 renamed Net-(S1-COM_1)
- net /STM32/Tx8 renamed /STM32/Tx8_LIDAR
- C9 pad 2: /STM32/NRST -> /NRST
- D1 pad 1: /CONNECTOR/D- -> /CONNECTOR/D+
- D1 pad 3: /CONNECTOR/D+ -> /CONNECTOR/D-
- ESC1 pad 4: /CONNECTOR/GPIO_Mot1 -> /GPIO_MOT1
- ESC1 pad 5: /CONNECTOR/TX_Mot1 -> /TX_MOT1
- ESC1 pad 6: /CONNECTOR/RX_Mot1 -> /RX_MOT1
- ESC2 pad 4: /CONNECTOR/GPIO_Mot2 -> /GPIO_MOT2
- ESC2 pad 5: /CONNECTOR/TX_Mot2 -> /TX_MOT2
- ESC2 pad 6: /CONNECTOR/RX_Mot2 -> /RX_MOT2
- ESC3 pad 4: /CONNECTOR/GPIO_Mot3 -> /GPIO_MOT3
- ESC3 pad 5: /CONNECTOR/TX_Mot3 -> /TX_MOT3
- ESC3 pad 6: /CONNECTOR/RX_Mot3 -> /RX_MOT3
- IC4 pad 16: /ESP32/D-ESP32 -> /D-ESP32
- IC4 pad 17: /ESP32/D+ESP32 -> /D+ESP32
- IC4 pad 21: /ESP32/ESP32_TX -> /ESP32_TX
- IC4 pad 22: /ESP32/ESP32_RX -> /ESP32_RX
- IC5 pad 12: /ACCESOIRES/XYZ_MISO -> /ACCEL_MISO
- IC5 pad 13: /ACCESOIRES/XYZ_MOSI -> /ACCEL_MOSI
- IC5 pad 7: /ACCESOIRES/XYZ_CS -> /ACCEL_CS
- IC6 pad 1: /ACCESOIRES/DATA_OUT -> /SAI_SD
- IC6 pad 10: /ACCESOIRES/HP- -> /HP-
- IC6 pad 14: /ACCESOIRES/FRAME_CLOCK -> /SAI_FS
- IC6 pad 16: /ACCESOIRES/BIT_CLOCK -> /SAI_CLK
- IC6 pad 9: /ACCESOIRES/HP+ -> /HP+
- IC7 pad 1: /ACCESOIRES/FLASH_CS -> /FLASH_CS
- IC7 pad 2: /ACCESOIRES/FLASH_MISO -> /FLASH_MISO
- IC7 pad 5: /ACCESOIRES/FLASH_MOSI -> /FLASH_MOSI
- IC7 pad 6: /ACCESOIRES/FLASH_SCK -> /FLASH_CLK
- LIDAR1 pad 1: unconnected-(LIDAR1-Pad1) -> /LIDAR_PWM
- LIDAR1 pad 2: unconnected-(LIDAR1-Pad2) -> GND
- LIDAR1 pad 3: unconnected-(LIDAR1-Pad3) -> /RX_LIDAR
- LIDAR1 pad 4: unconnected-(LIDAR1-Pad4) -> +5V
- Q1 pad 3: /POWER SUPPLY/GND_CONTROLLED -> /GND_CONTROLLED
- R15 pad 1: /POWER SUPPLY/GND_CONTROL_PIN -> /GND_CONTROl_GPIO
- R25 pad 1: /ACCESOIRES/XYZ_SCLK -> /ACCEL_CLK
- R26 pad 2: /ACCESOIRES/XYZ_INT2 -> /ACCEL_INT2
- R27 pad 2: /ACCESOIRES/XYZ_INT1 -> /ACCEL_INT1
- R28 pad 2: /ACCESOIRES/XYZ_CS -> /ACCEL_CS
- R29 pad 1: /ACCESOIRES/FLASH_CS -> /FLASH_CS
- R30 pad 1: /ACCESOIRES/AMPLI_GPIO -> /AMPLI_SD_MODE
- R34 pad 1: /POWER SUPPLY/POWERSWITCHB -> /BTN_B
- SWD1 pad 1: unconnected-(SWD1-Pad1) -> /SWDIO
- SWD1 pad 2: unconnected-(SWD1-Pad2) -> /SWCLK
- SWD1 pad 3: unconnected-(SWD1-Pad3) -> /NRST
- SWD1 pad 4: unconnected-(SWD1-Pad4) -> GND
- TOF1 pad 1: unconnected-(TOF1-Pad1) -> +3.3V
- TOF1 pad 2: unconnected-(TOF1-Pad2) -> /SCL_TOF1
- TOF1 pad 3: unconnected-(TOF1-Pad3) -> /SDA_TOF1
- TOF1 pad 4: unconnected-(TOF1-Pad4) -> GND
- TOF2 pad 1: unconnected-(TOF2-Pad1) -> +3.3V
- TOF2 pad 2: unconnected-(TOF2-Pad2) -> /SCL_TOF2
- TOF2 pad 3: unconnected-(TOF2-Pad3) -> /SDA_TOF2
- TOF2 pad 4: unconnected-(TOF2-Pad4) -> GND
- TOF3 pad 1: unconnected-(TOF3-Pad1) -> +3.3V
- TOF3 pad 2: unconnected-(TOF3-Pad2) -> /SCL_TOF3
- TOF3 pad 3: unconnected-(TOF3-Pad3) -> /SDA_TOF3
- TOF3 pad 4: unconnected-(TOF3-Pad4) -> GND
- U1 pad A10: /STM32/SWDIO -> /SWDIO
- U1 pad A3: unconnected-(U1-PE2-PadA3) -> /ACCEL_CLK
- U1 pad A4: /STM32/Tx4 -> /SDA_TOF2
- U1 pad A5: /STM32/I2C1_SDA -> /LIDAR_PWM
- U1 pad A6: unconnected-(U1-PB4-PadA6) -> /FLASH_MISO
- U1 pad A7: unconnected-(U1-PB3-PadA7) -> /FLASH_CLK
- U1 pad A8: /STM32/BUZZER_TIM -> /FLASH_CS
- U1 pad A9: /STM32/SWCLK -> /SWCLK
- U1 pad B10: /STM32/D+ -> /D+STM32
- U1 pad B3: /STM32/LED0 -> unconnected-(U1-PE3-PadB3)
- U1 pad B4: /STM32/Rx4 -> /SCL_TOF2
- U1 pad B5: /STM32/I2C1_SCL -> unconnected-(U1-PB6-PadB5)
- U1 pad B8: unconnected-(U1-PC11-PadB8) -> /STM32/ADC_VBAT
- U1 pad C10: /STM32/D- -> /D-STM32
- U1 pad C3: /STM32/LED1 -> unconnected-(U1-PE4-PadC3)
- U1 pad C5: unconnected-(U1-PB5-PadC5) -> /FLASH_MOSI
- U1 pad C9: /STM32/Tx1 -> unconnected-(U1-PA9-PadC9)
- U1 pad D10: /STM32/Rx1 -> /GPIO_MOT3
- U1 pad D3: unconnected-(U1-PE5-PadD3) -> /ACCEL_MISO
- U1 pad D4: /STM32/Rx8 -> /RX_LIDAR
- U1 pad D7: unconnected-(U1-PD4-PadD7) -> /SAI_FS
- U1 pad D8: unconnected-(U1-PD0-PadD8) -> /SAI_CLK
- U1 pad D9: /STM32/LED_TIM -> /SCL_TOF3
- U1 pad E1: /STM32/NRST -> /NRST
- U1 pad E10: /STM32/Rx6/ppm -> /RX_MOT3
- U1 pad E2: unconnected-(U1-PC2_C-PadE2) -> /ACCEL_INT2
- U1 pad E3: unconnected-(U1-PE6-PadE3) -> /ACCEL_MOSI
- U1 pad E8: unconnected-(U1-PD1-PadE8) -> /SAI_SD
- U1 pad E9: unconnected-(U1-PC9-PadE9) -> /SDA_TOF3
- U1 pad F1: /STM32/ADC_VBAT -> /ACCEL_INT1
- U1 pad F10: /STM32/Tx6 -> /TX_MOT3
- U1 pad F2: /STM32/ADC_EXT3_CURR2 -> /ACCEL_CS
- U1 pad G10: unconnected-(U1-PB15-PadG10) -> /RX_MOT1
- U1 pad G2: unconnected-(U1-PA0-PadG2) -> /TX_MOT2
- U1 pad G3: /STM32/ADC_EXT2_VB2 -> /AMPLI_SD_MODE
- U1 pad G5: /STM32/GYROEXTI -> unconnected-(U1-PB2-PadG5)
- U1 pad G9: unconnected-(U1-PD11-PadG9) -> /STM32/LED0
- U1 pad H10: unconnected-(U1-PB14-PadH10) -> /TX_MOT1
- U1 pad H2: unconnected-(U1-PA1-PadH2) -> /RX_MOT2
- U1 pad H5: /STM32/Rx7 -> /RX_SUP
- U1 pad H6: /STM32/IMU_CLK_EXTI -> unconnected-(U1-PE11-PadH6)
- U1 pad H7: unconnected-(U1-PE15-PadH7) -> /GND_CONTROl_GPIO
- U1 pad H9: unconnected-(U1-PD10-PadH9) -> /STM32/LED1
- U1 pad J10: unconnected-(U1-PD13-PadJ10) -> /SDA_TOF1
- U1 pad J5: /STM32/Tx7 -> /TX_SUP
- U1 pad J7: /STM32/I2C2_SCL -> /SCL_OLED
- U1 pad J9: /STM32/Rx3 -> /ESP32_RX
- U1 pad K10: unconnected-(U1-PD12-PadK10) -> /SCL_TOF1
- U1 pad K2: unconnected-(U1-PA3-PadK2) -> /GPIO_MOT2
- U1 pad K3: /STM32/ADC_CURR -> unconnected-(U1-PA7-PadK3)
- U1 pad K4: unconnected-(U1-PB1-PadK4) -> /LED_TIM
- U1 pad K7: /STM32/I2C1_SDA -> /SDA_OLED
- U1 pad K8: unconnected-(U1-PB12-PadK8) -> /GPIO_MOT1
- U1 pad K9: /STM32/Tx3 -> /ESP32_TX
- USBJUMP1 pad 1: unconnected-(USBJUMP1-Pin_1-Pad1) -> /D+STM32
- USBJUMP1 pad 2: unconnected-(USBJUMP1-Pin_2-Pad2) -> /CONNECTOR/DATA+OUT
- USBJUMP1 pad 3: unconnected-(USBJUMP1-Pin_3-Pad3) -> /D-STM32
- USBJUMP1 pad 4: unconnected-(USBJUMP1-Pin_4-Pad4) -> /CONNECTOR/DATA-OUT
- USBJUMP1 pad 5: unconnected-(USBJUMP1-Pin_5-Pad5) -> /D+ESP32
- USBJUMP1 pad 6: unconnected-(USBJUMP1-Pin_6-Pad6) -> /CONNECTOR/DATA+OUT
- USBJUMP1 pad 7: unconnected-(USBJUMP1-Pin_7-Pad7) -> /D-ESP32
- USBJUMP1 pad 8: unconnected-(USBJUMP1-Pin_8-Pad8) -> /CONNECTOR/DATA-OUT
Routing:
- added copper zone on In1.Cu, net GND
- added copper zone on In6.Cu, net GND
Other:
- copper layers 2 -> 8
- board text added: "Mounting hole R = 21 mm"

Commit message: update
Parts:
- moved C16 0.86 mm to (123.1, 86.8)
- moved C39 0.60 mm to (140.1, 87.6)
- moved C9 0.12 mm to (133.0, 89.9)
- moved R5 0.12 mm to (132.2, 89.9)
- moved C5 0.07 mm to (126.5, 91.7)
- moved R6 0.07 mm to (126.5, 91.0)
- moved D1 0.07 mm to (128.6, 70.9)
- moved C38 0.06 mm to (144.8, 85.6)
Routing:
- net /TX_MOT3: track 0.00 -> 27.6 mm, vias 0 -> 2
- net /SDA_TOF3: track 0.00 -> 26.5 mm, vias 0 -> 2
- net /SCL_TOF3: track 0.00 -> 25.3 mm, vias 0 -> 2
- net /GPIO_MOT3: track 0.00 -> 25.0 mm, vias 0 -> 2
- net /RX_MOT3: track 0.00 -> 24.9 mm, vias 0 -> 2
- net /RX_MOT1: track 0.00 -> 21.3 mm, vias 0 -> 2
- net /TX_MOT1: track 0.00 -> 18.4 mm, vias 0 -> 2
- net /GPIO_MOT1: track 0.00 -> 17.7 mm, vias 0 -> 2
- net /SCL_TOF1: track 0.00 -> 17.6 mm, vias 0 -> 2
- net /SDA_TOF1: track 0.00 -> 15.0 mm, vias 0 -> 2
- net /SCL_OLED: track 0.00 -> 13.4 mm
- net /SDA_OLED: track 0.00 -> 12.7 mm
- net /FLASH_MOSI: track 0.00 -> 10.5 mm
- net /ACCEL_CS: track 0.00 -> 10.4 mm
- net /LED_TIM: track 0.00 -> 10.1 mm
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- added copper zone on B.Cu, net +5V
- added copper zone on F.Cu, net +5V
- added copper zone on F.Cu, net /BAT+
- added copper zone on F.Cu, net 4.5V
- added copper zone on In3.Cu, net GND
- added copper zone on B.Cu, net Net-(IC1-SW)
- added copper zone on B.Cu, net VBAT+
- added copper zone on F.Cu, net VUSB

Commit message: up
Parts:
- moved L2 0.09 mm to (145.6, 80.5)
- moved C30 0.05 mm to (145.9, 81.8)
Connections:
- J5 pad 7: +5V -> 4.5V
Routing:
- net /NRST: track 3.85 -> 35.1 mm, vias 2 -> 3
- net /BTN_A: track 1.72 -> 30.0 mm
- net /RX_LIDAR: track 2.95 -> 27.1 mm
- net /LIDAR_PWM: track 4.96 -> 25.2 mm
- net /SCL_TOF2: track 3.45 -> 23.5 mm
- net /SWCLK: track 1.66 -> 21.5 mm
- net /SDA_TOF2: track 3.34 -> 23.0 mm
- net /SWDIO: track 1.84 -> 20.9 mm
- net /GPIO_MOT2: track 3.03 -> 21.4 mm
- net /TX_MOT2: track 2.60 -> 20.1 mm
- net /RX_MOT2: track 4.95 -> 22.3 mm
- net /SAI_SD: track 2.55 -> 18.9 mm
- net /SAI_CLK: track 1.53 -> 17.2 mm
- net /RX_SUP: track 0.00 -> 13.8 mm
- net /TX_SUP: track 0.00 -> 13.5 mm
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- added copper zone on B.Cu, net +3.3V
- added copper zone on F.Cu, net +3.3V
- added copper zone on In3.Cu, net +3.3V
- added copper zone on In3.Cu, net +5V
- added copper zone on F.Cu, net 3.3VSENSOR
- added copper zone on In3.Cu, net 4.5V
- added copper zone on B.Cu, net GND
- added copper zone on F.Cu, net GND
- added copper zone on In4.Cu, net GND
- added copper zone on F.Cu, net Net-(IC4-VDDA3P3_1)
- removed copper zone on In3.Cu, net GND
- removed copper zone on In6.Cu, net GND
Other:
- copper layers 8 -> 6

Commit message: up
Parts:
- added C46: 22u, Capacitor_SMD:C_0805_2012Metric, B.Cu at (118.1, 101.1)
- added C48: 22u, Capacitor_SMD:C_0805_2012Metric, B.Cu at (120.1, 101.1)
- added C49: 22u, Capacitor_SMD:C_0805_2012Metric, B.Cu at (122.1, 101.1)
- added C53: 22u, Capacitor_SMD:C_0805_2012Metric, B.Cu at (137.2, 70.9)
- added C54: 22u, Capacitor_SMD:C_0805_2012Metric, B.Cu at (135.4, 70.0)
- added C55: 22u, Capacitor_SMD:C_0805_2012Metric, B.Cu at (133.8, 69.0)
- added LED2: XZMDKCBDDG45S-9, samacsys:XZMDKCBDDG45S9, B.Cu at (118.7, 66.2)
- added R23: 10k, Resistor_SMD:R_0201_0603Metric, B.Cu at (122.7, 64.9)
- added R24: 10k, Resistor_SMD:R_0201_0603Metric, B.Cu at (119.9, 62.1)
- added R35: 10k, Resistor_SMD:R_0201_0603Metric, B.Cu at (114.2, 66.6)
- C1, C27, C3, C31, C34, C35, C37, C38, C40, C42, C47, C5, C9: footprint Capacitor_SMD:C_0201_0603Metric -> samacsys:C_0201_custom
- R12, R14, R16, R18, R2, R21, R25, R31, R34, R6, R7, R8: footprint Resistor_SMD:R_0201_0603Metric -> samacsys:R_0201_custom
Connections:
- U1 pad B6: unconnected-(U1-PD5-PadB6) -> /BLUE
- U1 pad B7: unconnected-(U1-PD2-PadB7) -> /GREEN
- U1 pad C7: unconnected-(U1-PD3-PadC7) -> /RED
Routing:
- net /GREEN: track 0.00 -> 43.5 mm, vias 0 -> 2
- net /RED: track 0.00 -> 40.6 mm, vias 0 -> 2
- net /BLUE: track 0.00 -> 35.9 mm, vias 0 -> 2
- net 4.5V: track 7.38 -> 1.98 mm, vias 14 -> 15
- net +3.3V: track 9.27 -> 4.82 mm, vias 36 -> 37
- net Net-(LED2-CATHODE_BLUE): track 0.00 -> 2.39 mm
- net /STM32/ADC_VBAT: track 15.7 -> 13.7 mm
- net Net-(LED2-CATHODE_GREEN): track 0.00 -> 1.91 mm
- net Net-(LED2-CATHODE_RED): track 0.00 -> 1.89 mm
- net GND: vias 137 -> 267

Commit message: update
Parts:
- added C50: 22u, Capacitor_SMD:C_0805_2012Metric, B.Cu at (112.2, 85.4)
- added C51: 22u, Capacitor_SMD:C_0805_2012Metric, B.Cu at (112.2, 83.4)
- added C52: 22u, Capacitor_SMD:C_0805_2012Metric, B.Cu at (112.2, 81.4)
- added G*** (x2): LOGO, LOGO, F.Cu at (118.8, 66.2)
- added G*** (x2): LOGO, LOGO, F.Cu at (118.3, 99.9)
- added LED3: XZMDKCBDDG45S-9, samacsys:XZMDKCBDDG45S9, B.Cu at (118.8, 100.0)
- added Q2: BSS138PW, samacsys:SOT65P210X110-3N, F.Cu at (112.7, 86.0)
- added Q4: BSS138PW, samacsys:SOT65P210X110-3N, F.Cu at (112.7, 80.6)
- added Q5: BSS138PW, samacsys:SOT65P210X110-3N, F.Cu at (112.7, 83.3)
- added R36: 1k, Resistor_SMD:R_0201_0603Metric, B.Cu at (119.8, 103.8)
- added R37: 1k, Resistor_SMD:R_0201_0603Metric, B.Cu at (114.9, 100.1)
- added R38: 1k, Resistor_SMD:R_0201_0603Metric, B.Cu at (122.2, 96.9)
- added R39: 100k, Resistor_SMD:R_0201_0603Metric, F.Cu at (114.7, 85.7)
- added R40: 100k, Resistor_SMD:R_0201_0603Metric, F.Cu at (114.7, 80.1)
- added R41: 100k, Resistor_SMD:R_0201_0603Metric, F.Cu at (114.7, 82.9)
- added R42: 100R, Resistor_SMD:R_0201_0603Metric, F.Cu at (114.7, 87.2)
- added R43: 100R, Resistor_SMD:R_0201_0603Metric, F.Cu at (114.7, 81.5)
- added R44: 100R, Resistor_SMD:R_0201_0603Metric, F.Cu at (114.7, 84.3)
- R23, R24, R35: value 10k -> 1k
- moved C46 9.65 mm to (124.2, 93.7), turned to 45 degrees
- moved C22 9.29 mm to (119.7, 91.8)
- moved C48 8.20 mm to (125.6, 95.0), turned to 45 degrees
- moved C49 6.77 mm to (127.0, 96.4), turned to 45 degrees
- moved IC3 6.66 mm to (122.1, 94.4), turned to -90 degrees
- moved LEDRED2 3.43 mm to (119.6, 93.9), turned to -90 degrees
- moved R18 2.96 mm to (119.7, 95.5), turned to 90 degrees
- moved C24 1.56 mm to (123.3, 98.6), turned to 90 degrees
- moved R29 0.31 mm to (128.7, 77.5)
- moved C47 0.22 mm to (126.6, 87.1)
- moved LEDGREEN1 0.05 mm to (134.1, 78.5)
Connections:
- R23 pad 1: /RED -> /ACCESOIRES/RED1
- R24 pad 1: /GREEN -> /ACCESOIRES/GREEN1
- R35 pad 2: /BLUE -> /ACCESOIRES/BLEU1
- U1 pad J9: /ESP32_RX -> /ESP32_TX
- U1 pad K9: /ESP32_TX -> /ESP32_RX
Routing:
- net /ACCESOIRES/BLEU1: track 0.00 -> 67.7 mm, vias 0 -> 4
- net /ACCESOIRES/RED1: track 0.00 -> 55.6 mm, vias 0 -> 4
- net /ACCESOIRES/GREEN1: track 0.00 -> 54.6 mm, vias 0 -> 4
- net /GREEN: track 43.5 -> 16.3 mm
- net /RED: track 40.6 -> 18.0 mm
- net /BLUE: track 35.9 -> 17.1 mm
- net +3.3V: track 4.82 -> 19.4 mm, vias 37 -> 38
- net Net-(LED3-CATHODE_RED): track 0.00 -> 6.61 mm
- net Net-(Q5-G): track 0.00 -> 2.82 mm
- net Net-(LED3-CATHODE_BLUE): track 0.00 -> 1.97 mm
- net Net-(LED3-CATHODE_GREEN): track 0.00 -> 1.96 mm
- net Net-(Q2-G): track 0.00 -> 1.94 mm
- net Net-(Q4-G): track 0.00 -> 1.92 mm
- net 3.3VSENSOR: track 0.00 -> 1.52 mm
- net 4.5V: track 1.98 -> 0.71 mm, vias 15 -> 13
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- added copper zone on In2.Cu, net GND
Other:
- board text added: "+"
- board text added: "-"
- board text added: "1"
- board text added: "1->STM32"
- board text added: "10-20v 3s max"
- board text added: "2"
- board text added: "2->ESP32"
- board text added: "3.3v"
- board text added: "3.3vACC"
- board text added: "AUX"
- board text added: "L0"
- board text added: "L1"
- board text added: "LIDAR"
- board text added: "MOTOR1"
- board text added: "MOTOR2"
- board text added: "MOTOR3"
- board text added: "PAF"
- board text added: "POWERBUTTON"
- board text added: "SWD"
- board text added: "TOF1"
- board text added: "TOF2"
- board text added: "TOF3"
- board text added: "USB"
- board text added: "V1.0"
