File: HARDWARE/PCB_PAPI/PCB_PAPI.kicad_sch (KiCad schematic)
At the start: 0 parts

Commit message: update
Other:
- sheet ACCESOIRES ports: added AMPLI_GPIO, BIT_CLOCK, DATA_OUT, FLASH_CS, FLASH_MISO, FLASH_MOSI, FLASH_SCK, FRAME_CLOCK, HP+, HP-, XYZ_CS, XYZ_INT1, XYZ_INT2, XYZ_MISO, XYZ_MOSI, XYZ_SCLK; removed BUZ-, BUZ_PIN_CONTROL
- sheet CONNECTOR ports: added BAT+, GND_CONTROLLED-, HP+, HP-, SCL_TOF1, SCL_TOF2, SCL_TOF3, SDA_TOF1, SDA_TOF2, SDA_TOF3; removed SCL_OLED2, SDA_OLED2
- sheet POWER SUPPLY ports: added BAT+, POWERSWITCHA, POWERSWITCHB; removed none

Commit message: updfate
Connections:
- no-connect marks 0 -> 1
Other:
- sheet CONNECTOR ports: added BTN_POWER_A, BTN_POWER_B, RX_SUP, TX_SUP; removed none
- sheet STM32 ports: added ACCEL_CLK_SPI4, ACCEL_CS_SPI4, ACCEL_INT1, ACCEL_INT2, ACCEL_MISO_SPI4, ACCEL_MOSI_SPI4, FLASH_CLK_SPI1, FLASH_CS_SPI1, FLASH_MISO_SPI1, FLASH_MOSI_SPI1, GPIO_COMMAND_GND, GPIO_MOTOR1, GPIO_MOTOR2, GPIO_MOTOR3, I2C1_SCL_TOF2, I2C1_SDA_TOF2, I2C2_SCL_OLED, I2C2_SDA_OLED, I2C3_SCL_TOF3, I2C3_SDA_TOF3, I2C4_SCL_TOF1, I2C4_SDA_TOF1, LED_TIM3_CH4, LIDAR_PWM_TIM4_CH2, NRST, Rx1_MOTOR1, Rx3_esp32, Rx4_MOTOR2, Rx6_MOTOR3, Rx7_SUP, Rx8_LIDAR, SAI3_FS, SAI3_SCK, SAI3_SD, SD_MODE_AMPLI, Tx1_MOTOR1, Tx3_esp32, Tx4_MOTOR2, Tx6_MOTOR3, Tx7_SUP, Tx8_LIDAR; removed ADC_CURR, ADC_EXT2_VB2, ADC_EXT3_CURR2, BOOT0, BUZZER_TIM, GYROEXTI, I2C1_SCL, I2C1_SDA, I2C2_SCL, IMU_CLK_EXTI, LED_TIM, Rx1, Rx3, Rx4, Rx6/ppm, Rx7, Rx8, Tx1, Tx3, Tx4, Tx6, Tx7, Tx8

Commit message: up
Other:
- sheet ACCESOIRES ports: added BLUE, GREEN, RED; removed none
- sheet STM32 ports: added PD2, PD3, PD5; removed none
Changed lines of the file:
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@@
+	(wire
+		(pts
+			(xy 435.61 190.5) (xy 438.15 190.5)
+		)
+		(stroke
+			(width 0)
+			(type default)
+		)
+	)
 	(wire
 		(pts
@@
 	(wire
 		(pts
+			(xy 435.61 198.12) (xy 438.15 198.12)
+		)
+		(stroke
+			(width 0)
+			(type default)
+		)
+	)
+	(wire
+		(pts
 			(xy 477.52 204.47) (xy 477.52 201.93)
 		)
@@
 		(pts
 			(xy 492.76 204.47) (xy 492.76 201.93)
+		)
+		(stroke
+			(width 0)
+			(type default)
+		)
+	)
+	(wire
+		(pts
+			(xy 435.61 194.31) (xy 438.15 194.31)
 		)
 		(stroke
@@
 		)
 	)
+	(label "RED"
+		(at 435.61 198.12 180)
+		(effects
+			(font
+				(size 1.27 1.27)
+			)
+			(justify right bottom)
+		)
+	)
 	(label "D-ESP32"
 		(at 167.64 248.92 90)
@@
 		)
 	)
+	(label "BLUE"
+		(at 73.66 213.36 270)
+		(effects
+			(font
+				(size 1.27 1.27)
+			)
+			(justify right bottom)
+		)
+	)
 	(label "ACCEL_MISO"
 		(at 142.24 49.53 0)
@@
 		)
 	)
+	(label "GREEN"
+		(at 435.61 194.31 180)
+		(effects
+			(font
+				(size 1.27 1.27)
+			)
+			(justify right bottom)
+		)
+	)
 	(label "BTN_A"
 		(at 436.88 63.5 180)
@@
 		)
 	)
+	(label "RED"
+		(at 68.58 213.36 270)
+		(effects
+			(font
+				(size 1.27 1.27)
+			)
+			(justify right bottom)
+		)
+	)
 	(label "ACCEL_MISO"
 		(at 435.61 175.26 180)
@@
 		)
 	)
+	(label "BLUE"
+		(at 435.61 190.5 180)
+		(effects
+			(font
+				(size 1.27 1.27)
+			)
+			(justify right bottom)
+		)
+	)
 	(label "ESP32_RX"
 		(at 91.44 31.75 90)
@@
 			)
 			(justify left bottom)
+		)
+	)
+	(label "GREEN"
+		(at 64.77 213.36 270)
+		(effects
+			(font
+				(size 1.27 1.27)
+			)
+			(justify right bottom)
 		)
 	)
@@
 			)
 		)
+		(pin "PD2" input
+			(at 64.77 213.36 270)
+			(effects
+				(font
+					(size 1.27 1.27)
+				)
+				(justify left)
+			)
+		)
+		(pin "PD3" input
+			(at 68.58 213.36 270)
+			(effects
+				(font
+					(size 1.27 1.27)
+				)
+				(justify left)
+			)
+		)
+		(pin "PD5" input
+			(at 73.66 213.36 270)
+			(effects
+				(font
+					(size 1.27 1.27)
+				)
+				(justify left)
+			)
+		)
 		(instances
 			(project "PCB_PAPI"
@@
 			(effects
 				(font
+					(size 1.27 1.27)
+				)
+				(justify left)
+			)
+		)
+		(pin "BLUE" input
+			(at 438.15 190.5 180)
+			(effects
+				(font
+					(size 1.27 1.27)
+				)
+				(justify left)
+			)
+		)
+		(pin "GREEN" input
+			(at 438.15 194.31 180)
+			(effects
+				(font
+					(size 1.27 1.27)
+				)
+				(justify left)
+			)
+		)
+		(pin "RED" input
+			(at 438.15 198.12 180)
+			(effects
+				(font

Commit message: update
Changed lines of the file:
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@@
-	(wire
-		(pts
-			(xy 91.44 31.75) (xy 91.44 35.56)
-		)
-		(stroke
-			(width 0)
-			(type default)
-		)
-	)
 	(wire
 		(pts
@@
 	(wire
 		(pts
+			(xy 95.25 33.02) (xy 95.25 35.56)
+		)
+		(stroke
+			(width 0)
+			(type default)
+		)
+	)
+	(wire
+		(pts
 			(xy 350.52 247.65) (xy 350.52 252.73)
 		)
@@
 	(wire
 		(pts
+			(xy 91.44 33.02) (xy 91.44 35.56)
+		)
+		(stroke
+			(width 0)
+			(type default)
+		)
+	)
+	(wire
+		(pts
 			(xy 477.52 204.47) (xy 477.52 201.93)
 		)
@@
 		(pts
 			(xy 142.24 120.65) (xy 138.43 120.65)
-		)
-		(stroke
-			(width 0)
-			(type default)
-		)
-	)
-	(wire
-		(pts
-			(xy 95.25 31.75) (xy 95.25 35.56)
 		)
 		(stroke
@@
 	)
 	(label "ESP32_TX"
-		(at 95.25 31.75 90)
+		(at 91.44 33.02 90)
 		(effects
 			(font
@@
 	)
 	(label "ESP32_RX"
-		(at 91.44 31.75 90)
-		(effects
-			(font
+		(at 95.25 33.02 90)
+		(effects
+			(font
