File: HARDWARE/PCB_PAPI/accesoires.kicad_sch (KiCad schematic)
At the start: 3 parts, among them Q2 STR2N2VH5

Commit message: PCB Principal
Parts:
- added C41, C42: 100n, symbol Device:C_Small
- added C43: C_Polarized_Small, symbol Device:C_Polarized_Small
- added IC5: ADXL343BCCZ-RL, ADXL343BCCZRL, symbol SamacSys_Parts:ADXL343BCCZ-RL
Connections:
- net GND: now also C42.1, C43.2, IC5.4 (GND_2), IC5.5 (GND_3)
- new net: C41.2, IC5.2 (GND_1)
- new net +5V: C41.1, C42.2, C43.1, IC5.1 (VDD_I/O), IC5.6 (VS)
- new net XYZ_CS: IC5.7 (~{CS})
- new net XYZ_INT1: IC5.8 (INT1)
- new net XYZ_INT2: IC5.9 (INT2)
- new net XYZ_SCLK: IC5.14 (SCL/SCLK)
- new net XYZ_SDIO: IC5.13 (SDA/SDI/SDIO)
- new net XYZ_SDO: IC5.12 (SDO/ALT_ADDRESS)
- no-connect marks 0 -> 2
Other:
- note added: "XYZ Accelero"

Commit message: update
Parts:
- removed Q2: STR2N2VH5, samacsys:SOT95P255X140-3N, symbol samacsys:STR2N2VH5
- removed R23: 100R, Resistor_SMD:R_0201_0603Metric, symbol Device:R_Small
- removed R24: 100k, Resistor_SMD:R_0201_0603Metric, symbol Device:R_Small
- added C44, C47: 100n, Capacitor_SMD:C_0201_0603Metric, symbol Device:C_Small
- added C45: 10u, Capacitor_SMD:C_0402_1005Metric, symbol Device:C_Small
- added IC6: MAX98357AETE+, samacsys:QFN50P300X300X80-17N, symbol samacsys:MAX98357AETE+
- added IC7: W25Q128JVPIQ_TR, samacsys:SON127P800X600X80-9N-D, symbol winbond:W25Q128JVPIQ_TR
- added R25, R26, R27: 22R, Resistor_SMD:R_0201_0603Metric, symbol Device:R_Small
- added R28, R29: 10k, Resistor_SMD:R_0201_0603Metric, symbol Device:R_Small
- added R30: 300k, Resistor_SMD:R_0201_0603Metric, symbol Device:R_Small
- added R31, R32: 0R, Resistor_SMD:R_0201_0603Metric, symbol Device:R_Small
- C41, C42: footprint (none) -> Capacitor_SMD:C_0201_0603Metric
- C43: value C_Polarized_Small -> 10u; footprint (none) -> Capacitor_Tantalum_SMD:CP_EIA-1608-08_AVX-J
- IC5: footprint ADXL343BCCZRL -> samacsys:ADXL343BCCZRL
Connections:
- net GND: now also C41.2, IC5.2 (GND_1), C44.2, C45.2, C47.2, IC6.11 (GND_2), IC6.15 (GND_3), IC6.17 (GND_4), IC6.3 (GND_1), IC7.4 (GND), IC7.9 (EP), R31.1
- net XYZ_CS: now also R28.2
- net XYZ_INT1: now also R27.2; no longer IC5.8 (INT1)
- net XYZ_INT2: now also R26.2; no longer IC5.9 (INT2)
- net XYZ_SCLK: now also R25.1; no longer IC5.14 (SCL/SCLK)
- net +5V renamed 3.3VSENSOR
- net 3.3VSENSOR: now also R28.1
- net XYZ_SDIO renamed XYZ_MOSI
- net XYZ_SDO renamed XYZ_MISO
- new net: IC6.2 (GAIN_SLOT), R31.2, R32.1
- new net: IC5.14 (SCL/SCLK), R25.2
- new net: IC5.8 (INT1), R27.1
- new net: IC5.9 (INT2), R26.1
- new net: IC6.4 (~{SD_MODE}), R30.2
- new net +3.3V: C47.1, IC7.3 (~{WP_(IO2)}), IC7.7 (~{HOLD_OR_RESET_(IO3)}), IC7.8 (VCC), R29.2
- new net 4.5V: C44.1, C45.1, IC6.7 (VDD_1), IC6.8 (VDD_2), R32.2
- new net AMPLI_GPIO: R30.1
- new net BIT_CLOCK: IC6.16 (BCLK)
- new net DATA_OUT: IC6.1 (DIN)
- new net FLASH_CS: IC7.1 (~{CS}), R29.1
- new net FLASH_MISO: IC7.2 (DO_(IO1))
- new net FLASH_MOSI: IC7.5 (DI_(IO0))
- new net FLASH_SCK: IC7.6 (CLK)
- new net FRAME_CLOCK: IC6.14 (LRCLK)
- new net HP+: IC6.9 (OUTP)
- new net HP-: IC6.10 (OUTN)
- no-connect marks 2 -> 6
Other:
- note added: "12dB"
- note added: "6dB"
- note added: "AMPLI"
- note added: "MEMOIRE SPI"
- note removed: "BUZZER"
- moved on the sheet: C41, C42, C43, IC5

Commit message: up
Parts:
- added LED2: XZMDKCBDDG45S-9, XZMDKCBDDG45S9, symbol samacsys:XZMDKCBDDG45S-9
- added R23, R24, R35: 10k, Resistor_SMD:R_0201_0603Metric, symbol Device:R_Small
- C42, C47: footprint Capacitor_SMD:C_0201_0603Metric -> samacsys:C_0201_custom
- R25, R31: footprint Resistor_SMD:R_0201_0603Metric -> samacsys:R_0201_custom
Connections:
- net +3.3V: now also LED2.2 (COMMON_ANODE)
- new net: LED2.1 (CATHODE_RED), R23.2
- new net: LED2.3 (CATHODE_BLUE), R35.1
- new net: LED2.4 (CATHODE_GREEN), R24.2
- new net BLUE: R35.2
- new net GREEN: R24.1
- new net RED: R23.1

Commit message: update
Parts:
- added LED3: XZMDKCBDDG45S-9, samacsys:XZMDKCBDDG45S9, symbol samacsys:XZMDKCBDDG45S-9
- added Q2, Q4, Q5: BSS138PW, samacsys:SOT65P210X110-3N, symbol samacsys:BSS138PW
- added R36, R37, R38: 1k, Resistor_SMD:R_0201_0603Metric, symbol Device:R_Small
- added R39, R40, R41: 100k, Resistor_SMD:R_0201_0603Metric, symbol Device:R_Small
- added R42, R43, R44: 100R, Resistor_SMD:R_0201_0603Metric, symbol Device:R_Small
- LED2: footprint XZMDKCBDDG45S9 -> samacsys:XZMDKCBDDG45S9
- R23, R24, R35: value 10k -> 1k
Connections:
- net +3.3V: now also LED3.2 (COMMON_ANODE)
- net BLUE: now also R42.2; no longer R35.2
- net GND: now also Q2.2 (S), Q4.2 (S), Q5.2 (S), R39.1, R40.1, R41.1
- net GREEN: now also R44.2; no longer R24.1
- net RED: now also R43.2; no longer R23.1
- new net: Q5.1 (G), R41.2, R44.1
- new net: Q2.1 (G), R39.2, R42.1
- new net: LED3.3 (CATHODE_BLUE), R36.1
- new net: LED3.1 (CATHODE_RED), R38.2
- new net: LED3.4 (CATHODE_GREEN), R37.2
- new net: Q4.1 (G), R40.2, R43.1
- new net BLEU1: Q2.3 (D), R35.2, R36.2
- new net GREEN1: Q5.3 (D), R24.1, R37.1
- new net RED1: Q4.3 (D), R23.1, R38.1
Other:
- note added: "a calculer"
- moved on the sheet: C41, C42, C43, C44, C45, C47, IC5, IC6, IC7, LED2, R23, R24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
