File: HARDWARE/PCB_PAPI/esp32.kicad_sch (KiCad schematic)
At the start: 27 parts, among them IC4 ESP32-C6FH4, J2 636101111001, Y2 LFXTAL069527REEL

Commit message: up
Parts:
- C27, C31, C34, C35, C37, C38, C40: footprint Capacitor_SMD:C_0201_0603Metric -> samacsys:C_0201_custom
- R21: footprint Resistor_SMD:R_0201_0603Metric -> samacsys:R_0201_custom
Changed lines of the file:
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@@
 			)
 		)
-		(property "Footprint" "Capacitor_SMD:C_0201_0603Metric"
+		(property "Footprint" "samacsys:C_0201_custom"
 			(at 248.92 133.35 0)
 			(effects
@@
 			)
 		)
-		(property "Footprint" "Capacitor_SMD:C_0201_0603Metric"
+		(property "Footprint" "samacsys:C_0201_custom"
 			(at 100.33 32.385 0)
 			(effects
@@
 			)
 		)
-		(property "Footprint" "Capacitor_SMD:C_0201_0603Metric"
+		(property "Footprint" "samacsys:C_0201_custom"
 			(at 170.815 95.25 0)
 			(effects
@@
 			)
 		)
-		(property "Footprint" "Resistor_SMD:R_0201_0603Metric"
+		(property "Footprint" "samacsys:R_0201_custom"
 			(at 217.17 83.82 0)
 			(effects
@@
 			)
 		)
-		(property "Footprint" "Capacitor_SMD:C_0201_0603Metric"
+		(property "Footprint" "samacsys:C_0201_custom"
 			(at 108.585 32.385 0)
 			(effects
@@
 			)
 		)
-		(property "Footprint" "Capacitor_SMD:C_0201_0603Metric"
+		(property "Footprint" "samacsys:C_0201_custom"
 			(at 85.725 100.965 0)
 			(effects
@@
 			)
 		)
-		(property "Footprint" "Capacitor_SMD:C_0201_0603Metric"
+		(property "Footprint" "samacsys:C_0201_custom"
 			(at 204.47 34.29 0)
 			(effects
@@
 			)
 		)
-		(property "Footprint" "Capacitor_SMD:C_0201_0603Metric"
+		(property "Footprint" "samacsys:C_0201_custom"
 			(at 260.35 34.29 0)
 			(effects

Commit message: update
Other:
- moved on the sheet: C25, C26, C28, C29, C31, C32, C33, C34, C35, C37, C39, L3
