File: HARDWARE/PCB_PAPI/stm32.kicad_sch (KiCad schematic)
At the start: 25 parts, among them U1 STM32H743VIHx, Y1 CSTNE8M00GH5C000R0

Commit message: updfate
Connections:
- net ADC_VBAT: now also U1.B8 (PC11); no longer U1.F1 (PC0)
- net LED0: now also U1.G9 (PD11); no longer U1.B3 (PE3)
- net LED1: now also U1.H9 (PD10); no longer U1.C3 (PE4)
- net ACCEL_CLK_SPI4: now reaches U1.A3 (PE2)
- net FLASH_MISO_SPI1: now reaches U1.A6 (PB4)
- net FLASH_CLK_SPI1: now reaches U1.A7 (PB3)
- net FLASH_MOSI_SPI1: now reaches U1.C5 (PB5)
- net ACCEL_MISO_SPI4: now reaches U1.D3 (PE5)
- net SAI3_FS: now reaches U1.D7 (PD4)
- net SAI3_SCK: now reaches U1.D8 (PD0)
- net ACCEL_INT2: now reaches U1.E2 (PC2_C)
- net ACCEL_MOSI_SPI4: now reaches U1.E3 (PE6)
- net SAI3_SD: now reaches U1.E8 (PD1)
- net I2C3_SDA_TOF3: now reaches U1.E9 (PC9)
- net Rx1_MOTOR1: now reaches U1.G10 (PB15)
- net Tx4_MOTOR2: now reaches U1.G2 (PA0)
- net Tx1_MOTOR1: now reaches U1.H10 (PB14)
- net Rx4_MOTOR2: now reaches U1.H2 (PA1)
- net GPIO_COMMAND_GND: now reaches U1.H7 (PE15)
- net I2C4_SDA_TOF1: now reaches U1.J10 (PD13)
- net I2C4_SCL_TOF1: now reaches U1.K10 (PD12)
- net GPIO_MOTOR2: now reaches U1.K2 (PA3)
- net LED_TIM3_CH4: now reaches U1.K4 (PB1)
- net GPIO_MOTOR1: now reaches U1.K8 (PB12)
- net ADC_CURR: no longer names the net of U1.K3 (PA7)
- net ADC_EXT2_VB2 renamed SD_MODE_AMPLI
- net ADC_EXT3_CURR2 renamed ACCEL_CS_SPI4
- net BOOT0: no longer names the net of C5.2, R6.1, S1.3 (COM_1), S1.4 (COM_2), U1.D5 (BOOT0)
- net BUZZER_TIM renamed FLASH_CS_SPI1
- net GYROEXTI: no longer names the net of U1.G5 (PB2)
- net I2C1_SCL: no longer names the net of U1.B5 (PB6)
- net I2C1_SDA renamed I2C2_SDA_OLED
- net I2C2_SDA_OLED: no longer U1.A5 (PB7)
- net I2C2_SCL renamed I2C2_SCL_OLED
- net IMU_CLK_EXTI: no longer names the net of U1.H6 (PE11)
- net LED_TIM renamed I2C3_SCL_TOF3
- net Rx1 renamed GPIO_MOTOR3
- net Rx3 renamed Rx3_esp32
- net Rx4 renamed I2C1_SCL_TOF2
- net Rx6/ppm renamed Rx6_MOTOR3
- net Rx7 renamed Rx7_SUP
- net Rx8 renamed Rx8_LIDAR
- net Tx1: no longer names the net of U1.C9 (PA9)
- net Tx3 renamed Tx3_esp32
- net Tx4 renamed I2C1_SDA_TOF2
- net Tx6 renamed Tx6_MOTOR3
- net Tx7 renamed Tx7_SUP
- net Tx8 renamed Tx8_LIDAR
- new net ACCEL_INT1: U1.F1 (PC0)
- new net LIDAR_PWM_TIM4_CH2: U1.A5 (PB7)
- no-connect marks 51 -> 34

Commit message: up
Parts:
- C1, C3, C5, C9: footprint Capacitor_SMD:C_0201_0603Metric -> samacsys:C_0201_custom
- R2, R6: footprint Resistor_SMD:R_0201_0603Metric -> samacsys:R_0201_custom
Connections:
- net PD5: now reaches U1.B6 (PD5)
- net PD2: now reaches U1.B7 (PD2)
- net PD3: now reaches U1.C7 (PD3)
- no-connect marks 34 -> 31
Changed lines of the file:
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@@
 	)
 	(no_connect
-		(at 273.05 138.43)
-	)
-	(no_connect
 		(at 318.77 110.49)
 	)
@@
 	)
 	(no_connect
-		(at 273.05 130.81)
-	)
-	(no_connect
 		(at 318.77 105.41)
 	)
@@
 	)
 	(no_connect
-		(at 273.05 133.35)
-	)
-	(no_connect
 		(at 273.05 118.11)
 	)
@@
 		)
 	)
+	(hierarchical_label "PD5"
+		(shape input)
+		(at 273.05 138.43 180)
+		(effects
+			(font
+				(size 1.27 1.27)
+			)
+			(justify right)
+		)
+	)
 	(hierarchical_label "ACCEL_MISO_SPI4"
 		(shape input)
@@
 		)
 	)
+	(hierarchical_label "PD3"
+		(shape input)
+		(at 273.05 133.35 180)
+		(effects
+			(font
+				(size 1.27 1.27)
+			)
+			(justify right)
+		)
+	)
 	(hierarchical_label "Rx7_SUP"
 		(shape input)
@@
 		)
 	)
+	(hierarchical_label "PD2"
+		(shape input)
+		(at 273.05 130.81 180)
+		(effects
+			(font
+				(size 1.27 1.27)
+			)
+			(justify right)
+		)
+	)
 	(hierarchical_label "ACCEL_MOSI_SPI4"
 		(shape input)
@@
 			)
 		)
-		(property "Footprint" "Capacitor_SMD:C_0201_0603Metric"
+		(property "Footprint" "samacsys:C_0201_custom"
 			(at 232.41 44.45 0)
 			(effects
@@
 			)
 		)
-		(property "Footprint" "Resistor_SMD:R_0201_0603Metric"
+		(property "Footprint" "samacsys:R_0201_custom"
 			(at 234.95 77.47 0)
 			(effects
@@
 			)
 		)
-		(property "Footprint" "Capacitor_SMD:C_0201_0603Metric"
+		(property "Footprint" "samacsys:C_0201_custom"
 			(at 45.72 157.48 0)
 			(effects
@@
 			)
 		)
-		(property "Footprint" "Capacitor_SMD:C_0201_0603Metric"
+		(property "Footprint" "samacsys:C_0201_custom"
 			(at 245.11 77.47 0)
 			(effects
@@
 			)
 		)
-		(property "Footprint" "Resistor_SMD:R_0201_0603Metric"
+		(property "Footprint" "samacsys:R_0201_custom"
 			(at 38.1 157.48 0)
 			(effects
@@
 			)
 		)
-		(property "Footprint" "Capacitor_SMD:C_0201_0603Metric"
+		(property "Footprint" "samacsys:C_0201_custom"
 			(at 266.7 62.23 0)
 			(effects

Commit message: update
Changed lines of the file:
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@@
-	)
-	(label "HSE_IN"
-		(at 86.36 60.96 180)
-		(effects
-			(font
-				(size 1.27 1.27)
-			)
-			(justify right bottom)
-		)
 	)
 	(label "HSE_IN"
