File: HARDWARE/PCB_PAPI/PWR.kicad_sch (KiCad schematic)
At the start: 27 parts, among them IC1 LMR51625YFDDCR, IC2 LDO40LPU33RY, IC3 LDO40LPU33RY, Q1 STR2N2VH5

Commit message: update
Parts:
- added Q3: SQS401EN-T1_BE3, samacsys:SQS401ENT1_BE3, symbol samacsys:SQS401EN-T1_BE3
- added R33: 100k, Resistor_SMD:R_0201_0603Metric, symbol Device:R_Small
- added R34: 1k, Resistor_SMD:R_0201_0603Metric, symbol Device:R_Small
Connections:
- net GND: now also R34.2
- net VBAT+: now also Q3.10 (D_6), Q3.11 (D_7), Q3.5 (D_1), Q3.6 (D_2), Q3.7 (D_3), Q3.8 (D_4), Q3.9 (D_5)
- new net BAT+: Q3.1 (S_1), Q3.2 (S_2), Q3.3 (S_3), R33.1
- new net POWERSWITCHA: Q3.4 (G), R33.2
- new net POWERSWITCHB: R34.1

Commit message: up
Parts:
- added C46, C48, C49, C50, C51, C52, C53, C54, C55: 22u, Capacitor_SMD:C_0805_2012Metric, symbol Device:C_Small
- R12, R14, R16, R18, R34: footprint Resistor_SMD:R_0201_0603Metric -> samacsys:R_0201_custom
Connections:
- net GND: now also C46.2, C48.2, C49.2, C50.2, C51.2, C52.2, C53.2, C54.2, C55.2
- net VBAT+: now also C46.1, C48.1, C49.1, C50.1, C51.1, C52.1, C53.1, C54.1, C55.1

Commit message: update
Other:
- note added: "A verifier ref"
Changed lines of the file:
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@@
 		)
 	)
+	(text "A verifier ref\n"
+		(exclude_from_sim no)
+		(at 142.494 44.704 0)
+		(effects
+			(font
+				(size 1.27 1.27)
+			)
+		)
+	)
 	(text "RED WURTH 150040RS73240"
 		(exclude_from_sim no)
@@
 	)
 	(junction
+		(at 128.27 76.2)
+		(diameter 0)
+		(color 0 0 0 0)
+	)
+	(junction
 		(at 72.39 46.99)
 		(diameter 0)
@@
 	(wire
 		(pts
+			(xy 128.27 76.2) (xy 121.92 76.2)
+		)
+		(stroke
+			(width 0)
+			(type default)
+		)
+	)
+	(wire
+		(pts
 			(xy 96.52 46.99) (xy 96.52 52.07)
 		)
@@
 	(wire
 		(pts
-			(xy 139.7 76.2) (xy 121.92 76.2)
+			(xy 139.7 76.2) (xy 128.27 76.2)
 		)
 		(stroke
@@
 					(unit 1)
 				)
+			)
+		)
+	)
+	(symbol
+		(lib_id "power:PWR_FLAG")
+		(at 128.27 76.2 180)
+		(unit 1)
+		(exclude_from_sim no)
+		(in_bom yes)
+		(on_board yes)
+		(dnp no)
+		(fields_autoplaced yes)
+		(property "Reference" "#FLG05"
+			(at 128.27 78.105 0)
+			(effects
+				(font
+					(size 1.27 1.27)
+				)
+				(hide yes)
+			)
+		)
+		(property "Value" "PWR_FLAG"
+			(at 128.27 81.28 0)
+			(effects
+				(font
+					(size 1.27 1.27)
+				)
+			)
+		)
+		(property "Footprint" ""
+			(at 128.27 76.2 0)
+			(effects
+				(font
+					(size 1.27 1.27)
+				)
+				(hide yes)
+			)
+		)
+		(property "Datasheet" "~"
+			(at 128.27 76.2 0)
+			(effects
+				(font
+					(size 1.27 1.27)
+				)
+				(hide yes)
+			)
+		)
+		(property "Description" "Special symbol for telling ERC where power comes from"
+			(at 128.27 76.2 0)
+			(effects
+				(font
+					(size 1.27 1.27)
+				)
+				(hide yes)
+			)
+		)
+		(pin "1"
+		)
+		(instances
+			(project "PCB_PAPI"
+				(path "/64301b3d-8a16-47d9-a9c6-0068257932ba/847f55ac-306c-4b7a-8ec1-939febc79176"
+					(reference "#FLG05")
+					(unit 1)
+				)

Commit message: up pcb principal
Other:
- note removed: "A verifier ref"
Changed lines of the file:
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@@
-		)
-	)
-	(text "A verifier ref\n"
-		(exclude_from_sim no)
-		(at 142.494 44.704 0)
-		(effects
-			(font
-				(size 1.27 1.27)
-			)
 		)
 	)
