File: HARDWARE/ELECTRONIQUE/PCB_PAPI/accesoires.kicad_sch (KiCad schematic)
At the start: 34 parts, among them IC5 ADXL343BCCZ-RL, IC6 MAX98357AETE+, IC7 W25Q128JVPIQ_TR, Q2 BSS138PW, Q4 BSS138PW, Q5 BSS138PW

Commit message: up
Parts:
- removed LED2, LED3: XZMDKCBDDG45S-9, samacsys:XZMDKCBDDG45S9, symbol samacsys:XZMDKCBDDG45S-9
- added LED4, LED5: IN-P32TRRRGB, symbol samacsys:IN-P32TRRRGB
Connections:
- net +3.3V: now also LED4.4 (COM_A), LED5.4 (COM_A)
- net at R23.2: now also LED4.3 (K_RED)
- net at R35.1: now also LED4.1 (K_BLUE)
- net at R24.2: now also LED4.2 (K_GREEN)
- net at R36.1: now also LED5.1 (K_BLUE)
- net at R38.2: now also LED5.3 (K_RED)
- net at R37.2: now also LED5.2 (K_GREEN)
Other:
- note added: "ATTENTION EMPRINTE"
- moved on the sheet: R23, R24, R35, R36, R37, R38
