File: HARDWARE/ELECTRONIQUE/FOC_CONTROLLER/FOC_CONTROLLER_V1/FOC_CONTROLLER_V1.kicad_sch (KiCad schematic)
At the start: 53 parts, among them IC1 STSPIN32G0A2, J1 SM06B-GHS-TB_LF__SN_, J2 SM06B-GHS-TB_LF__SN_

Commit message: u
Other:
- note added: "3Imaxphase=1/Rshunt*((0.255*(3R46+R)/R46)-RVref/R46)"
- note added: "Avec R46=18k et R=2.2k et enfin Rshunt=50mohm on a 3Imaxphase=7.86A et donc ImaxPhase=2.62A"
- note added: "En considerant Rshuntafet=R et Rpullup=R46"
Changed lines of the file:
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@@
+		)
+	)
+	(text "En considerant Rshuntafet=R et Rpullup=R46"
+		(exclude_from_sim no)
+		(at 366.014 181.356 0)
+		(effects
+			(font
+				(size 1.27 1.27)
+			)
+		)
+	)
+	(text "3Imaxphase=1/Rshunt*((0.255*(3R46+R)/R46)-RVref/R46)\n"
+		(exclude_from_sim no)
+		(at 365.252 185.42 0)
+		(effects
+			(font
+				(size 1.27 1.27)
+			)
+		)
+	)
+	(text "Avec R46=18k et R=2.2k et enfin Rshunt=50mohm on a 3Imaxphase=7.86A et donc ImaxPhase=2.62A"
+		(exclude_from_sim no)
+		(at 355.346 188.468 0)
+		(effects
+			(font
+				(size 1.27 1.27)
+			)
 		)
 	)
