File: HARDWARE/ELECTRONIQUE/FOC_CONTROLLER/FOC_CONTROLLER_V1/U.kicad_sch (KiCad schematic)
At the start: 18 parts, among them Q1 DMT6018LDR-7

Commit message: up
Other:
- note added: "On veut Rth+==Rth- mais aussi que pour IMAX=3A avec Rshunt=50mohm on ait G=10 et donc tension aille de 0v a 3.3v environs"
- note added: "Rth+=R//R//R10"
- note added: "Rth-=R13//R9"
- note added: "VOUT=((R13+R9)/R9)*(R/(2R10+R))*SHUNTP+((R13+R9)/R9)*(R10/(2R10+R))*VREF"
- note added: "Vop3p=(IN+*(R/2R10+R))+(Vref*(R10/2R10+R)"
- note added: "avec R=R11=R12"

Commit message: u
Parts:
- D2, D3, R4, R7: now not fitted
- R43: value 3k -> 2.2k
Changed lines of the file:
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@@
 			)
 		)
-		(property "Value" "3k"
+		(property "Value" "2.2k"
 			(at 176.53 67.31 90)
 			(effects
@@
 		(in_bom yes)
 		(on_board yes)
-		(dnp no)
+		(dnp yes)
 		(fields_autoplaced yes)
 		(property "Reference" "R4"
@@
 		(in_bom yes)
 		(on_board yes)
-		(dnp no)
+		(dnp yes)
 		(fields_autoplaced yes)
 		(property "Reference" "D2"
@@
 		(in_bom yes)
 		(on_board yes)
-		(dnp no)
+		(dnp yes)
 		(fields_autoplaced yes)
 		(property "Reference" "D3"
@@
 		(in_bom yes)
 		(on_board yes)
-		(dnp no)
+		(dnp yes)
 		(fields_autoplaced yes)
 		(property "Reference" "R7"
