File: HARDWARE/ELECTRONIQUE/FOC_CONTROLLER/FOC_CONTROLLER_V1/FOC_CONTROLLER_V1.kicad_pcb (KiCad board)
At the start: 8 copper layers, 34.4 x 34.9 mm, 121 parts, among them IC1 STSPIN32G0A2, IC2 MA330GQ-Z, J1 SM06B-GHS-TB_LF__SN_, J2 SM06B-GHS-TB_LF__SN_, Q1 DMT6018LDR-7, Q2 DMT6018LDR-7, Q3 DMT6018LDR-7

Commit message: u
Parts:
- R43, R44, R45: value 3k -> 2.2k
Changed lines of the file:
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@@
 		(sheetname "/U/")
 		(sheetfile "U.kicad_sch")
-		(attr smd)
+		(attr smd dnp)
 		(fp_circle
 			(center -0.935 0)
@@
 		(sheetname "/W/")
 		(sheetfile "U.kicad_sch")
-		(attr smd)
+		(attr smd dnp)
 		(fp_line
 			(start -0.88 0.35)
@@
 		(sheetname "/U/")
 		(sheetfile "U.kicad_sch")
-		(attr smd)
+		(attr smd dnp)
 		(fp_circle
 			(center -0.935 0)
@@
 		(sheetname "/V/")
 		(sheetfile "U.kicad_sch")
-		(attr smd)
+		(attr smd dnp)
 		(fp_circle
 			(center -0.935 0)
@@
 		(sheetname "/V/")
 		(sheetfile "U.kicad_sch")
-		(attr smd)
+		(attr smd dnp)
 		(fp_line
 			(start -0.88 0.35)
@@
 		(sheetname "/W/")
 		(sheetfile "U.kicad_sch")
-		(attr smd)
+		(attr smd dnp)
 		(fp_circle
 			(center -0.935 0)
@@
 		(sheetname "/W/")
 		(sheetfile "U.kicad_sch")
-		(attr smd)
+		(attr smd dnp)
 		(fp_line
 			(start -0.88 0.35)
@@
 		(sheetname "/U/")
 		(sheetfile "U.kicad_sch")
-		(attr smd)
+		(attr smd dnp)
 		(fp_line
 			(start 0.88 -0.35)
@@
 		(sheetname "/V/")
 		(sheetfile "U.kicad_sch")
-		(attr smd)
+		(attr smd dnp)
 		(fp_line
 			(start -0.88 0.35)
@@
 		(sheetname "/W/")
 		(sheetfile "U.kicad_sch")
-		(attr smd)
+		(attr smd dnp)
 		(fp_circle
 			(center -0.935 0)
@@
 		(sheetname "/V/")
 		(sheetfile "U.kicad_sch")
-		(attr smd)
+		(attr smd dnp)
 		(fp_circle
 			(center -0.935 0)
@@
 		(sheetname "/U/")
 		(sheetfile "U.kicad_sch")
-		(attr smd)
+		(attr smd dnp)
 		(fp_line
 			(start 0.88 -0.35)
@@
 			)
 		)
-		(property "Value" "3k"
+		(property "Value" "2.2k"
 			(at 0 -1.05 0)
 			(layer "B.Fab")
@@
 			)
 		)
-		(property "Value" "3k"
+		(property "Value" "2.2k"
 			(at 0 -1.05 0)
 			(layer "B.Fab")
@@
 			)
 		)
-		(property "Value" "3k"
+		(property "Value" "2.2k"
 			(at 0 -1.05 0)
 			(layer "B.Fab")

Commit message: up
Parts:
- removed the G*** at (88.9, 106.5)
- removed the G*** at (87.3, 101.5)
- removed the G*** at (114.2, 101.5)
- removed the G*** at (107.5, 111.5)
- removed the G*** at (111.5, 106.5)
- removed the G*** at (94.2, 111.5)
- removed the G*** at (100.0, 113.3)
- added G***: LOGO, LOGO, F.Cu at (93.2, 111.1)
