File: HARDWARE/ELECTRONIQUE/PCB_Mouse/PCB_Mouse.kicad_sch (KiCad schematic)
At the start: 20 parts, among them IC1 STM32G431CBU6, U1 PMW3360, U2 TLV74318PDBVR

Commit message: up
Parts:
- removed IC1: STM32G431CBU6, QFN50P700X700X65-49N-D, symbol SamacSys_Parts:STM32G431CBU6
- removed JP1: SolderJumper_3_Open, Jumper:SolderJumper-3_P1.3mm_Open_RoundedPad1.0x1.5mm_NumberLabels, symbol Jumper:SolderJumper_3_Open
- removed TP1: V_{IO}, TestPoint:TestPoint_Pad_D1.0mm, symbol Connector:TestPoint
- removed TP2: V_{DD}, TestPoint:TestPoint_Pad_D1.0mm, symbol Connector:TestPoint
- removed TP3: GND, TestPoint:TestPoint_Pad_D1.0mm, symbol Connector:TestPoint
- removed U2: TLV74318PDBVR, Package_TO_SOT_SMD:SOT-23-5, symbol PMW3360_PCB:TLV74318PDBVR
- added C10, C14, C8: 1u, Capacitor_SMD:C_0402_1005Metric, symbol Device:C_Small
- added C11: 4.7u, Capacitor_SMD:C_0402_1005Metric, symbol Device:C_Small
- added C12, C13: 16p, Capacitor_SMD:C_0402_1005Metric, symbol Device:C_Small
- added C15, C16, C17, C9: 100n, Capacitor_SMD:C_0402_1005Metric, symbol Device:C_Small
- added C6: 0.1u, Capacitor_SMD:C_0402_1005Metric, symbol Device:C_Small
- added C7: 10n, Capacitor_SMD:C_0402_1005Metric, symbol Device:C_Small
- added D3: LED, LED_SMD:LED_0402_1005Metric, symbol Device:LED
- added IC1, IC2: LDLN025M33R, samacsys:SOT95P280X145-5N, symbol samacsys:LDLN025M33R
- added J1, J2: SM04B-GHS-TB_LF__SN_, samacsys:SM04B-GHS-TB, symbol samacsys:SM04B-GHS-TB_LF__SN_
- added R20: 1.1k, Resistor_SMD:R_0402_1005Metric, symbol Device:R_Small
- added R5: 10k, Resistor_SMD:R_0402_1005Metric, symbol Device:R
- added SW1: RSTBTN, samacsys:KXT341LHS, symbol Switch:SW_Push
- added U2: STM32G431CBUx, Package_DFN_QFN:QFN-48-1EP_7x7mm_P0.5mm_EP5.6x5.6mm, symbol MCU_ST_STM32G4:STM32G431CBUx
- added Y1: Crystal_GND24_Small, samacsys:LFXTAL069527REEL, symbol Device:Crystal_GND24_Small
- C2: footprint Capacitor_SMD:C_0603_1608Metric_Pad1.08x0.95mm_HandSolder -> Capacitor_SMD:C_0402_1005Metric
- C3, C4: value 1uF -> 1u; footprint Capacitor_SMD:C_0603_1608Metric_Pad1.08x0.95mm_HandSolder -> Capacitor_SMD:C_0402_1005Metric
- C5: value 22nF -> 1u; footprint Capacitor_SMD:C_0603_1608Metric_Pad1.08x0.95mm_HandSolder -> Capacitor_SMD:C_0402_1005Metric; LCSC C21122 -> (none); Mfr. # CL10B223KB8NNNC -> (none); now fitted
- R1, R2, R3: footprint Resistor_SMD:R_0603_1608Metric_Pad0.98x0.95mm_HandSolder -> Resistor_SMD:R_0402_1005Metric
- R4: value 28k -> 0R; footprint Resistor_SMD:R_0603_1608Metric_Pad0.98x0.95mm_HandSolder -> Resistor_SMD:R_0402_1005Metric; now fitted
- U1: footprint PMW3360_PCB:PMW3360DM-T2QU 16Pin -> samacsys:PMW3360
Connections:
- net V_{IN} is gone; now on net VDD: C3.1
- net CS: now also U2.12 (PA4)
- net GND: now also C10.1, C11.2, C12.2, C13.1, C14.2, C15.1, C16.1, C17.1, C6.1, C7.1, C8.1, C9.1, IC1.2 (GND), IC2.2 (GND), J1.1, J2.1, R20.1, SW1.1, U2.49 (VSS), Y1.2, Y1.4
- net MISO: now also U2.14 (PA6)
- net MOSI: now also U2.15 (PA7)
- net RESET: now also U2.43 (PB5)
- net SCLK: now also R5.2, U2.13 (PA5); no longer U1.10 (SCLK)
- net SWCLK: now also J1.4, U2.37 (PA14)
- net SWDIO: now also J1.3, U2.36 (PA13)
- net VDD: now also C14.1, IC1.1 (IN), IC1.3 (EN), IC2.1 (IN), IC2.3 (EN), J2.4; no longer C4.1, R3.1, R4.1, U1.4 (VDD)
- net +1V8: now reaches C5.1
- net +1V8: now also R3.1, U1.4 (VDD), IC2.5 (OUT); no longer R4.2
- net MOTION: no longer names the net of U1.9 (MOTION)
- net MOTION: now also R4.1
- net V_{IO} renamed +3.3V
- net +3.3V: now also C4.1, C10.2, C11.1, C15.2, C16.2, C17.2, C7.2, C8.2, C9.2, IC1.5 (OUT), U2.1 (VBAT), U2.20 (VREF+), U2.21 (VDDA), U2.23 (VDD), U2.35 (VDD), U2.48 (VDD)
- new net: C13.2, U2.5 (PF0), Y1.1
- new net: C12.1, U2.6 (PF1), Y1.3
- new net: R5.1, U1.10 (SCLK)
- new net: D3.2 (A), U2.27 (PB14)
- new net: D3.1 (K), R20.2
- new net NRST: C6.2, J1.2, SW1.2, U2.7 (PG10)
- new net SENSOR_INT: R4.2, U2.16 (PC4)
- new net USART1_RX: J2.3, U2.45 (PB7)
- new net USART1_TX: J2.2, U2.44 (PB6)
- no-connect marks 0 -> 28
Other:
- note added: "CONTROLEUR PRINCIPAL"
- note removed: "LDO selection: a) TLV74318PDBVR (Fixed 1.8V output): * C3 and C4: 1uF * C5 and R4: don't install b) RT9193-18GB (Fixed 1.8V output): * C3 and C4: 1uF * C5: 22nF or larger ceramic capacitor * R4: don't install c) TPS73601DBV: * C3: 1uF * C4: 4.7uF * C5: 56.2kΩ * R4: 28kΩ"
- note removed: "Operating voltage range: * VIN: Depends on config * VIO: VDD ~ 3.6V * VDD: 1.8 ~ 2.1V"
- note removed: "Power"
- note removed: "Test Points"
- note removed: "V_{IO} Selection"
- note removed: "Voltage-Level config: a) 3.3V: * VIN: connect to 3.3V, 3.6V max * JP1: [1-2 3], VIO=VIN b) 1.8V with LDO: * VIN: (VDD + 0.2V) ~ 5.5V * JP1: [1 2-3], VIO=VDD c) 1.8V without LDO: * VIN: connect to 1.8V, 2.1V max * JP1: [1-2-3], VIO=VDD=VIN * U2, R4, C3~5 can be omitted as well"
- moved on the sheet: C1, C2, R1, R2, R3, U1
