File: HARDWARE/ELECTRONIQUE/PCB_PAPI_V2/PCB_PAPI.kicad_sch (KiCad schematic)
At the start: 0 parts

Commit message: up
Other:
- sheet ACCESOIRES ports: added none; removed AMPLI_GPIO, BIT_CLOCK, DATA_OUT, FRAME_CLOCK, HP+, HP-
- sheet ESP32 ports: added HP+, HP-; removed none
Changed lines of the file:
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@@
-	(wire
-		(pts
-			(xy 496.57 204.47) (xy 496.57 201.93)
-		)
-		(stroke
-			(width 0)
-			(type default)
-		)
-	)
 	(wire
 		(pts
@@
 	(wire
 		(pts
-			(xy 435.61 167.64) (xy 438.15 167.64)
+			(xy 434.34 198.12) (xy 436.88 198.12)
 		)
 		(stroke
@@
 	(wire
 		(pts
-			(xy 435.61 163.83) (xy 438.15 163.83)
+			(xy 434.34 194.31) (xy 436.88 194.31)
 		)
 		(stroke
@@
 	(wire
 		(pts
-			(xy 435.61 175.26) (xy 438.15 175.26)
+			(xy 434.34 205.74) (xy 436.88 205.74)
 		)
 		(stroke
@@
 	(wire
 		(pts
-			(xy 435.61 179.07) (xy 438.15 179.07)
+			(xy 434.34 209.55) (xy 436.88 209.55)
 		)
 		(stroke
@@
 	(wire
 		(pts
-			(xy 435.61 171.45) (xy 438.15 171.45)
+			(xy 434.34 201.93) (xy 436.88 201.93)
 		)
 		(stroke
@@
 	(wire
 		(pts
-			(xy 469.9 204.47) (xy 469.9 201.93)
-		)
-		(stroke
-			(width 0)
-			(type default)
-		)
-	)
-	(wire
-		(pts
 			(xy 278.13 248.92) (xy 278.13 252.73)
 		)
@@
 	(wire
 		(pts
+			(xy 435.61 147.32) (xy 438.15 147.32)
+		)
+		(stroke
+			(width 0)
+			(type default)
+		)
+	)
+	(wire
+		(pts
 			(xy 142.24 124.46) (xy 138.43 124.46)
 		)
@@
 	(wire
 		(pts
-			(xy 473.71 204.47) (xy 473.71 201.93)
-		)
-		(stroke
-			(width 0)
-			(type default)
-		)
-	)
-	(wire
-		(pts
 			(xy 434.34 134.62) (xy 438.15 134.62)
 		)
@@
 	(wire
 		(pts
-			(xy 477.52 204.47) (xy 477.52 201.93)
-		)
-		(stroke
-			(width 0)
-			(type default)
-		)
-	)
-	(wire
-		(pts
 			(xy 438.15 303.53) (xy 434.34 303.53)
 		)
@@
 	(wire
 		(pts
-			(xy 435.61 182.88) (xy 438.15 182.88)
-		)
-		(stroke
-			(width 0)
-			(type default)
-		)
-	)
-	(wire
-		(pts
-			(xy 481.33 204.47) (xy 481.33 201.93)
+			(xy 434.34 213.36) (xy 436.88 213.36)
 		)
 		(stroke
@@
 	(wire
 		(pts
-			(xy 492.76 204.47) (xy 492.76 201.93)
-		)
-		(stroke
-			(width 0)
-			(type default)
-		)
-	)
-	(wire
-		(pts
 			(xy 434.34 121.92) (xy 438.15 121.92)
 		)
@@
 		(pts
 			(xy 142.24 140.97) (xy 138.43 140.97)
+		)
+		(stroke
+			(width 0)
+			(type default)
+		)
+	)
+	(wire
+		(pts
+			(xy 435.61 151.13) (xy 438.15 151.13)
 		)
 		(stroke
@@
 	)
 	(label "ACCEL_INT2"
-		(at 435.61 171.45 180)
+		(at 434.34 201.93 180)
 		(effects
 			(font
@@
 	)
 	(label "ACCEL_INT1"
-		(at 435.61 167.64 180)
+		(at 434.34 198.12 180)
 		(effects
 			(font
@@
 		)
 	)
-	(label "AMPLI_SD_MODE"
-		(at 469.9 204.47 270)
-		(effects
-			(font
-				(size 1.27 1.27)
-			)
-			(justify right bottom)
-		)
-	)
 	(label "GND_CONTROLLED"
 		(at 435.61 83.82 180)
@@
 		)
 	)
-	(label "SAI_FS"
-		(at 481.33 204.47 270)
-		(effects
-			(font
-				(size 1.27 1.27)
-			)
-			(justify right bottom)
-		)
-	)
 	(label "RX_MOT1"
 		(at 182.88 248.92 90)
@@
 		)
 	)
+	(label "HP+"
+		(at 435.61 147.32 180)
+		(effects
+			(font
+				(size 1.27 1.27)
+			)
+			(justify right bottom)
+		)
+	)
 	(label "SCL_OLED"
 		(at 140.97 165.1 0)
@@
 	)
 	(label "ACCEL_CS"
-		(at 435.61 163.83 180)
+		(at 434.34 194.31 180)
 		(effects
 			(font
@@
 		)
 	)
-	(label "HP+"
-		(at 492.76 204.47 270)
-		(effects
-			(font
-				(size 1.27 1.27)
-			)
-			(justify right bottom)
-		)
-	)
 	(label "GPIO_MOT2"
 		(at 142.24 115.57 0)
@@
 		)
 	)
-	(label "SAI_CLK"
-		(at 473.71 204.47 270)
-		(effects
-			(font
-				(size 1.27 1.27)
-			)
-			(justify right bottom)
-		)
-	)
 	(label "SWCLK"
 		(at 57.15 31.75 90)
@@
 		)
 	)
-	(label "HP-"
-		(at 496.57 204.47 270)
-		(effects
-			(font
-				(size 1.27 1.27)
-			)
-			(justify right bottom)
-		)
-	)
 	(label "GPIO_MOT2"
 		(at 199.39 248.92 90)
@@
 	)
 	(label "ACCEL_MOSI"
-		(at 435.61 179.07 180)
+		(at 434.34 209.55 180)
 		(effects
 			(font
@@
 	)
 	(label "ACCEL_CLK"
-		(at 435.61 182.88 180)
+		(at 434.34 213.36 180)
 		(effects
 			(font
@@
 		)
 	)
-	(label "SAI_SD"
-		(at 477.52 204.47 270)
-		(effects
-			(font
-				(size 1.27 1.27)
-			)
-			(justify right bottom)
-		)
-	)
 	(label "TX_MOT1"
 		(at 140.97 97.79 0)
@@
 	)
 	(label "ACCEL_MISO"
-		(at 435.61 175.26 180)
+		(at 434.34 205.74 180)
 		(effects
 			(font
@@
 			)
 			(justify left bottom)
+		)
+	)
+	(label "HP-"
+		(at 435.61 151.13 180)
+		(effects
+			(font
+				(size 1.27 1.27)
+			)
+			(justify right bottom)
 		)
 	)
@@
 	)
 	(sheet
-		(at 438.15 158.75)
+		(at 436.88 189.23)
 		(size 110.49 43.18)
 		(exclude_from_sim no)
@@
 		)
 		(property "Sheetname" "ACCESOIRES"
-			(at 438.15 158.0384 0)
+			(at 436.88 188.5184 0)
 			(effects
 				(font
@@
 		)
 		(property "Sheetfile" "accesoires.kicad_sch"
-			(at 438.15 202.5146 0)
+			(at 436.88 232.9946 0)
 			(effects
 				(font
@@
 			)
 		)
-		(pin "AMPLI_GPIO" input
-			(at 469.9 201.93 270)
+		(pin "XYZ_CS" input
+			(at 436.88 194.31 180)
 			(effects
 				(font
@@
 			)
 		)
-		(pin "BIT_CLOCK" input
-			(at 473.71 201.93 270)
+		(pin "XYZ_INT1" input
+			(at 436.88 198.12 180)
 			(effects
 				(font
@@
 			)
 		)
-		(pin "DATA_OUT" input
-			(at 477.52 201.93 270)
+		(pin "XYZ_INT2" input
+			(at 436.88 201.93 180)
 			(effects
 				(font
@@
 			)
 		)
-		(pin "FRAME_CLOCK" input
-			(at 481.33 201.93 270)
+		(pin "XYZ_MISO" input
+			(at 436.88 205.74 180)
 			(effects
 				(font
@@
 			)
 		)
-		(pin "HP+" input
-			(at 492.76 201.93 270)
+		(pin "XYZ_MOSI" input
+			(at 436.88 209.55 180)
 			(effects
 				(font
@@
 			)
 		)
-		(pin "HP-" input
-			(at 496.57 201.93 270)
+		(pin "XYZ_SCLK" input
+			(at 436.88 213.36 180)
 			(effects
 				(font
@@
 			)
 		)
-		(pin "XYZ_CS" input
-			(at 438.15 163.83 180)
-			(effects
-				(font
-					(size 1.27 1.27)
-				)
-				(justify left)
-			)
-		)
-		(pin "XYZ_INT1" input
-			(at 438.15 167.64 180)
-			(effects
-				(font
-					(size 1.27 1.27)
-				)
-				(justify left)
-			)
-		)
-		(pin "XYZ_INT2" input
-			(at 438.15 171.45 180)
-			(effects
-				(font
-					(size 1.27 1.27)
-				)
-				(justify left)
-			)
-		)
-		(pin "XYZ_MISO" input
-			(at 438.15 175.26 180)
-			(effects
-				(font
-					(size 1.27 1.27)
-				)
-				(justify left)
-			)
-		)
-		(pin "XYZ_MOSI" input
-			(at 438.15 179.07 180)
-			(effects
-				(font
-					(size 1.27 1.27)
-				)
-				(justify left)
-			)
-		)
-		(pin "XYZ_SCLK" input
-			(at 438.15 182.88 180)
-			(effects
-				(font
-					(size 1.27 1.27)
-				)
-				(justify left)
-			)
-		)
 		(pin "LED_TOM_JERRY_RGB" input
-			(at 438.15 191.77 180)
+			(at 436.88 222.25 180)
 			(effects
 				(font
@@
 	(sheet
 		(at 438.15 105.41)
-		(size 109.22 43.18)
+		(size 109.22 74.93)
 		(exclude_from_sim no)
 		(in_bom yes)
@@
 		)
 		(property "Sheetfile" "esp32.kicad_sch"
-			(at 438.15 149.1746 0)
+			(at 438.15 180.9246 0)
 			(effects
 				(font
@@
 			(effects
 				(font
+					(size 1.27 1.27)
+				)
+				(justify left)
+			)
+		)
+		(pin "HP+" input
+			(at 438.15 147.32 180)
+			(effects
+				(font
+					(size 1.27 1.27)
+				)
+				(justify left)
+			)
+		)
+		(pin "HP-" input
+			(at 438.15 151.13 180)
+			(effects
+				(font

Commit message: up
Other:
- sheet CONNECTOR ports: added MOUSE_CLK, MOUSE_CS, MOUSE_INT, MOUSE_MISO, MOUSE_MOSI; removed none
- sheet STM32 ports: added MOUSE_CLK_SPI1, MOUSE_CS_SPI1, MOUSE_MISO_SPI1, MOUSE_MOSI_SPI1; removed SAI3_FS, SAI3_SCK, SAI3_SD, SD_MODE_AMPLI
Changed lines of the file:
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@@
-	(wire
-		(pts
-			(xy 102.87 217.17) (xy 102.87 213.36)
-		)
-		(stroke
-			(width 0)
-			(type default)
-		)
-	)
 	(wire
 		(pts
@@
 	(wire
 		(pts
-			(xy 93.98 217.17) (xy 93.98 213.36)
-		)
-		(stroke
-			(width 0)
-			(type default)
-		)
-	)
-	(wire
-		(pts
 			(xy 223.52 248.92) (xy 223.52 252.73)
 		)
@@
 	(wire
 		(pts
+			(xy 434.34 222.25) (xy 436.88 222.25)
+		)
+		(stroke
+			(width 0)
+			(type default)
+		)
+	)
+	(wire
+		(pts
 			(xy 434.34 209.55) (xy 436.88 209.55)
 		)
@@
 	(wire
 		(pts
-			(xy 90.17 217.17) (xy 90.17 213.36)
-		)
-		(stroke
-			(width 0)
-			(type default)
-		)
-	)
-	(wire
-		(pts
 			(xy 436.88 78.74) (xy 439.42 78.74)
 		)
@@
 		(pts
 			(xy 435.61 83.82) (xy 439.42 83.82)
-		)
-		(stroke
-			(width 0)
-			(type default)
-		)
-	)
-	(wire
-		(pts
-			(xy 99.06 217.17) (xy 99.06 213.36)
 		)
 		(stroke
@@
 		)
 	)
-	(label "AMPLI_SD_MODE"
-		(at 102.87 217.17 270)
-		(effects
-			(font
-				(size 1.27 1.27)
-			)
-			(justify right bottom)
-		)
-	)
 	(label "RX_SUP"
 		(at 142.24 205.74 0)
@@
 		)
 	)
+	(label "RGB_TOM_JERRY"
+		(at 434.34 222.25 180)
+		(effects
+			(font
+				(size 1.27 1.27)
+			)
+			(justify right bottom)
+		)
+	)
 	(label "GPIO_MOT2"
 		(at 199.39 248.92 90)
@@
 		)
 	)
-	(label "SAI_SD"
-		(at 99.06 217.17 270)
-		(effects
-			(font
-				(size 1.27 1.27)
-			)
-			(justify right bottom)
-		)
-	)
 	(label "SDA_TOF2"
 		(at 142.24 127 0)
@@
 		)
 	)
-	(label "SAI_CLK"
-		(at 93.98 217.17 270)
-		(effects
-			(font
-				(size 1.27 1.27)
-			)
-			(justify right bottom)
-		)
-	)
-	(label "SAI_FS"
-		(at 90.17 217.17 270)
-		(effects
-			(font
-				(size 1.27 1.27)
-			)
-			(justify right bottom)
-		)
-	)
 	(label "LED_TIM"
 		(at 350.52 247.65 90)
@@
 			)
 			(justify left bottom)
+		)
+	)
+	(label "RGB_TOM_JERRY"
+		(at 97.79 222.25 180)
+		(effects
+			(font
+				(size 1.27 1.27)
+			)
+			(justify right bottom)
 		)
 	)
@@
 			)
 		)
-		(pin "SAI3_FS" input
-			(at 90.17 213.36 270)
-			(effects
-				(font
-					(size 1.27 1.27)
-				)
-				(justify left)
-			)
-		)
-		(pin "SAI3_SCK" input
-			(at 93.98 213.36 270)
-			(effects
-				(font
-					(size 1.27 1.27)
-				)
-				(justify left)
-			)
-		)
-		(pin "SAI3_SD" input
-			(at 99.06 213.36 270)
-			(effects
-				(font
-					(size 1.27 1.27)
-				)
-				(justify left)
-			)
-		)
-		(pin "SD_MODE_AMPLI" input
-			(at 102.87 213.36 270)
-			(effects
-				(font
-					(size 1.27 1.27)
-				)
-				(justify left)
-			)
-		)
 		(pin "SWCLK" input
 			(at 57.15 35.56 90)
@@
 				)
 				(justify right)
+			)
+		)
+		(pin "MOUSE_CLK_SPI1" input
+			(at 71.12 213.36 270)
+			(effects
+				(font
+					(size 1.27 1.27)
+				)
+				(justify left)
+			)
+		)
+		(pin "MOUSE_CS_SPI1" input
+			(at 74.93 213.36 270)
+			(effects
+				(font
+					(size 1.27 1.27)
+				)
+				(justify left)
+			)
+		)
+		(pin "MOUSE_MISO_SPI1" input
+			(at 78.74 213.36 270)
+			(effects
+				(font
+					(size 1.27 1.27)
+				)
+				(justify left)
+			)
+		)
+		(pin "MOUSE_MOSI_SPI1" input
+			(at 83.82 213.36 270)
+			(effects
+				(font
+					(size 1.27 1.27)
+				)
+				(justify left)
 			)
 		)
@@
 			)
 		)
+		(pin "MOUSE_CLK" input
+			(at 139.7 279.4 180)
+			(effects
+				(font
+					(size 1.27 1.27)
+				)
+				(justify left)
+			)
+		)
+		(pin "MOUSE_CS" input
+			(at 139.7 283.21 180)
+			(effects
+				(font
+					(size 1.27 1.27)
+				)
+				(justify left)
+			)
+		)
+		(pin "MOUSE_INT" input
+			(at 139.7 287.02 180)
+			(effects
+				(font
+					(size 1.27 1.27)
+				)
+				(justify left)
+			)
+		)
+		(pin "MOUSE_MISO" input
+			(at 139.7 275.59 180)
+			(effects
+				(font
+					(size 1.27 1.27)
+				)
+				(justify left)
+			)
+		)
+		(pin "MOUSE_MOSI" input
+			(at 139.7 271.78 180)
+			(effects
+				(font
+					(size 1.27 1.27)
+				)
+				(justify left)
+			)
+		)

Commit message: up
Other:
- sheet STM32 ports: added MOUSE_INT, TOM_JERRY_RGB; removed none
Changed lines of the file:
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@@
+	(wire
+		(pts
+			(xy 83.82 217.17) (xy 83.82 213.36)
+		)
+		(stroke
+			(width 0)
+			(type default)
+		)
+	)
 	(wire
 		(pts
@@
 	(wire
 		(pts
+			(xy 138.43 287.02) (xy 139.7 287.02)
+		)
+		(stroke
+			(width 0)
+			(type default)
+		)
+	)
+	(wire
+		(pts
 			(xy 140.97 95.25) (xy 138.43 95.25)
 		)
@@
 	(wire
 		(pts
+			(xy 66.04 217.17) (xy 66.04 213.36)
+		)
+		(stroke
+			(width 0)
+			(type default)
+		)
+	)
+	(wire
+		(pts
 			(xy 434.34 209.55) (xy 436.88 209.55)
 		)
@@
 	(wire
 		(pts
+			(xy 138.43 271.78) (xy 139.7 271.78)
+		)
+		(stroke
+			(width 0)
+			(type default)
+		)
+	)
+	(wire
+		(pts
 			(xy 160.02 248.92) (xy 160.02 252.73)
 		)
@@
 	(wire
 		(pts
+			(xy 71.12 217.17) (xy 71.12 213.36)
+		)
+		(stroke
+			(width 0)
+			(type default)
+		)
+	)
+	(wire
+		(pts
 			(xy 308.61 248.92) (xy 308.61 252.73)
 		)
@@
 	(wire
 		(pts
+			(xy 138.43 275.59) (xy 139.7 275.59)
+		)
+		(stroke
+			(width 0)
+			(type default)
+		)
+	)
+	(wire
+		(pts
 			(xy 142.24 210.82) (xy 138.43 210.82)
 		)
@@
 	(wire
 		(pts
+			(xy 138.43 283.21) (xy 139.7 283.21)
+		)
+		(stroke
+			(width 0)
+			(type default)
+		)
+	)
+	(wire
+		(pts
 			(xy 186.69 248.92) (xy 186.69 252.73)
 		)
@@
 	(wire
 		(pts
+			(xy 93.98 217.17) (xy 93.98 213.36)
+		)
+		(stroke
+			(width 0)
+			(type default)
+		)
+	)
+	(wire
+		(pts
 			(xy 142.24 146.05) (xy 138.43 146.05)
 		)
@@
 	(wire
 		(pts
+			(xy 138.43 279.4) (xy 139.7 279.4)
+		)
+		(stroke
+			(width 0)
+			(type default)
+		)
+	)
+	(wire
+		(pts
 			(xy 142.24 102.87) (xy 138.43 102.87)
 		)
@@
 	(wire
 		(pts
+			(xy 74.93 217.17) (xy 74.93 213.36)
+		)
+		(stroke
+			(width 0)
+			(type default)
+		)
+	)
+	(wire
+		(pts
 			(xy 142.24 140.97) (xy 138.43 140.97)
+		)
+		(stroke
+			(width 0)
+			(type default)
+		)
+	)
+	(wire
+		(pts
+			(xy 78.74 217.17) (xy 78.74 213.36)
 		)
 		(stroke
@@
 		)
 	)
+	(label "MOUSE_MISO"
+		(at 138.43 275.59 180)
+		(effects
+			(font
+				(size 1.27 1.27)
+			)
+			(justify right bottom)
+		)
+	)
+	(label "MOUSE_MOSI"
+		(at 138.43 271.78 180)
+		(effects
+			(font
+				(size 1.27 1.27)
+			)
+			(justify right bottom)
+		)
+	)
 	(label "ACCEL_INT2"
 		(at 142.24 60.96 0)
@@
 		)
 	)
+	(label "MOUSE_CS"
+		(at 74.93 217.17 270)
+		(effects
+			(font
+				(size 1.27 1.27)
+			)
+			(justify right bottom)
+		)
+	)
 	(label "RX_LIDAR"
 		(at 142.24 187.96 0)
@@
 		)
 	)
+	(label "MOUSE_CLK"
+		(at 138.43 279.4 180)
+		(effects
+			(font
+				(size 1.27 1.27)
+			)
+			(justify right bottom)
+		)
+	)
 	(label "D-ESP32"
 		(at 167.64 248.92 90)
@@
 		)
 	)
+	(label "MOUSE_CLK"
+		(at 71.12 217.17 270)
+		(effects
+			(font
+				(size 1.27 1.27)
+			)
+			(justify right bottom)
+		)
+	)
 	(label "RX_MOT3"
 		(at 223.52 248.92 90)
@@
 		)
 	)
+	(label "MOUSE_INT"
+		(at 138.43 287.02 180)
+		(effects
+			(font
+				(size 1.27 1.27)
+			)
+			(justify right bottom)
+		)
+	)
 	(label "ACCEL_INT1"
 		(at 142.24 57.15 0)
@@
 		)
 	)
+	(label "MOUSE_CS"
+		(at 138.43 283.21 180)
+		(effects
+			(font
+				(size 1.27 1.27)
+			)
+			(justify right bottom)
+		)
+	)
 	(label "TX_MOT1"
 		(at 140.97 97.79 0)
@@
 		)
 	)
+	(label "MOUSE_MOSI"
+		(at 83.82 217.17 270)
+		(effects
+			(font
+				(size 1.27 1.27)
+			)
+			(justify right bottom)
+		)
+	)
 	(label "SDA_TOF1"
 		(at 142.24 105.41 0)
@@
 		)
 	)
+	(label "MOUSE_MISO"
+		(at 78.74 217.17 270)
+		(effects
+			(font
+				(size 1.27 1.27)
+			)
+			(justify right bottom)
+		)
+	)
 	(label "RX_MOT2"
 		(at 142.24 118.11 0)
@@
 		)
 	)
+	(label "MOUSE_INT"
+		(at 66.04 217.17 270)
+		(effects
+			(font
+				(size 1.27 1.27)
+			)
+			(justify right bottom)
+		)
+	)
 	(label "SCL_TOF2"
 		(at 142.24 124.46 0)
@@
 	)
 	(label "RGB_TOM_JERRY"
-		(at 97.79 222.25 180)
+		(at 93.98 217.17 270)
 		(effects
 			(font
@@
 			(effects
 				(font
+					(size 1.27 1.27)
+				)
+				(justify left)
+			)
+		)
+		(pin "TOM_JERRY_RGB" input
+			(at 93.98 213.36 270)
+			(effects
+				(font
+					(size 1.27 1.27)
+				)
+				(justify left)
+			)
+		)
+		(pin "MOUSE_INT" input
+			(at 66.04 213.36 270)
+			(effects
+				(font

Commit message: up
Other:
- sheet CONNECTOR ports: added none; removed GND_CONTROLLED-
- sheet POWER SUPPLY ports: added none; removed GND_CONTROLLED, GND_CONTROL_PIN
- sheet STM32 ports: added none; removed GPIO_COMMAND_GND
Changed lines of the file:
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@@
-	(wire
-		(pts
-			(xy 346.71 247.65) (xy 346.71 252.73)
-		)
-		(stroke
-			(width 0)
-			(type default)
-		)
-	)
 	(wire
 		(pts
@@
 	(wire
 		(pts
-			(xy 436.88 78.74) (xy 439.42 78.74)
-		)
-		(stroke
-			(width 0)
-			(type default)
-		)
-	)
-	(wire
-		(pts
 			(xy 142.24 187.96) (xy 138.43 187.96)
 		)
@@
 	(wire
 		(pts
-			(xy 435.61 83.82) (xy 439.42 83.82)
-		)
-		(stroke
-			(width 0)
-			(type default)
-		)
-	)
-	(wire
-		(pts
 			(xy 438.15 298.45) (xy 434.34 298.45)
 		)
@@
 		(pts
 			(xy 179.07 248.92) (xy 179.07 252.73)
-		)
-		(stroke
-			(width 0)
-			(type default)
-		)
-	)
-	(wire
-		(pts
-			(xy 142.24 200.66) (xy 138.43 200.66)
 		)
 		(stroke
@@
 		)
 	)
-	(label "GND_CONTROLLED"
-		(at 435.61 83.82 180)
-		(effects
-			(font
-				(size 1.27 1.27)
-			)
-			(justify right bottom)
-		)
-	)
 	(label "ACCEL_MOSI"
 		(at 142.24 53.34 0)
@@
 		)
 	)
-	(label "GND_CONTROl_GPIO"
-		(at 436.88 78.74 180)
-		(effects
-			(font
-				(size 1.27 1.27)
-			)
-			(justify right bottom)
-		)
-	)
 	(label "D+STM32"
 		(at 74.93 31.75 90)
@@
 		)
 	)
-	(label "GND_CONTROLLED"
-		(at 346.71 247.65 90)
-		(effects
-			(font
-				(size 1.27 1.27)
-			)
-			(justify left bottom)
-		)
-	)
 	(label "ACCEL_CS"
 		(at 142.24 41.91 0)
@@
 			)
 			(justify right bottom)
-		)
-	)
-	(label "GND_CONTROl_GPIO"
-		(at 142.24 200.66 0)
-		(effects
-			(font
-				(size 1.27 1.27)
-			)
-			(justify left bottom)
 		)
 	)
@@
 			)
 		)
-		(pin "GPIO_COMMAND_GND" input
-			(at 138.43 200.66 0)
-			(effects
-				(font
-					(size 1.27 1.27)
-				)
-				(justify right)
-			)
-		)
 		(pin "GPIO_MOTOR1" input
 			(at 138.43 92.71 0)
@@
 			)
 		)
-		(pin "GND_CONTROLLED-" input
-			(at 346.71 252.73 90)
-			(effects
-				(font
-					(size 1.27 1.27)
-				)
-				(justify right)
-			)
-		)
 		(pin "GPIO_Mot1" input
 			(at 179.07 252.73 90)
@@
 			)
 		)
-		(pin "GND_CONTROLLED" input
-			(at 439.42 83.82 180)
-			(effects
-				(font
-					(size 1.27 1.27)
-				)
-				(justify left)
-			)
-		)
-		(pin "GND_CONTROL_PIN" input
-			(at 439.42 78.74 180)
-			(effects
-				(font
-					(size 1.27 1.27)
-				)
-				(justify left)
-			)
-		)
