File: HARDWARE/ELECTRONIQUE/PCB_PAPI_V2/stm32.kicad_sch (KiCad schematic)
At the start: 25 parts, among them U1 STM32H743VIHx, Y1 CSTNE8M00GH5C000R0

Commit message: up
Connections:
- net FLASH_CLK_SPI1 renamed MOUSE_CLK_SPI1
- net FLASH_CS_SPI1 renamed MOUSE_CS_SPI1
- net FLASH_MISO_SPI1 renamed MOUSE_MISO_SPI1
- net FLASH_MOSI_SPI1 renamed MOUSE_MOSI_SPI1
- net SAI3_FS: no longer names the net of U1.D7 (PD4)
- net SAI3_SCK: no longer names the net of U1.D8 (PD0)
- net SAI3_SD: no longer names the net of U1.E8 (PD1)
- net SD_MODE_AMPLI: no longer names the net of U1.G3 (PA4)
- no-connect marks 34 -> 38

Commit message: up
Connections:
- net ADC_VBAT: now also U1.B1 (PC15); no longer U1.B8 (PC11)
- net MOUSE_INT: now reaches U1.A2 (PC13)
- net TOM_JERRY_RGB: now reaches U1.B5 (PB6)
- no-connect marks 38 -> 36
Changed lines of the file:
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@@
-	)
-	(no_connect
-		(at 318.77 186.69)
 	)
 	(no_connect
@@
 	)
 	(no_connect
+		(at 318.77 176.53)
+	)
+	(no_connect
 		(at 273.05 118.11)
 	)
@@
 	)
 	(no_connect
-		(at 318.77 120.65)
-	)
-	(no_connect
 		(at 318.77 135.89)
 	)
@@
 	)
 	(no_connect
-		(at 318.77 181.61)
-	)
-	(no_connect
 		(at 273.05 90.17)
 	)
@@
 	(wire
 		(pts
+			(xy 321.31 186.69) (xy 318.77 186.69)
+		)
+		(stroke
+			(width 0)
+			(type default)
+		)
+	)
+	(wire
+		(pts
 			(xy 266.7 171.45) (xy 266.7 179.07)
 		)
@@
 		(pts
 			(xy 245.11 72.39) (xy 245.11 74.93)
-		)
-		(stroke
-			(width 0)
-			(type default)
-		)
-	)
-	(wire
-		(pts
-			(xy 321.31 176.53) (xy 318.77 176.53)
 		)
 		(stroke
@@
 	)
 	(label "ADC_VBAT"
-		(at 321.31 176.53 0)
+		(at 321.31 186.69 0)
 		(effects
 			(font
@@
 		)
 	)
+	(hierarchical_label "MOUSE_INT"
+		(shape input)
+		(at 318.77 181.61 0)
+		(effects
+			(font
+				(size 1.27 1.27)
+			)
+			(justify left)
+		)
+	)
 	(hierarchical_label "I2C3_SCL_TOF3"
 		(shape input)
@@
 		(effects
 			(font
+				(size 1.27 1.27)
+			)
+			(justify left)
+		)
+	)
+	(hierarchical_label "TOM_JERRY_RGB"
+		(shape input)
+		(at 318.77 120.65 0)
+		(effects
+			(font

Commit message: up
Connections:
- net TOM_JERRY_RGB: now also U1.C9 (PA9); no longer U1.B5 (PB6)
- net GPIO_COMMAND_GND: no longer names the net of U1.H7 (PE15)
- no-connect marks 36 -> 37
