File: HARDWARE/ELECTRONIQUE/PCB_PAPI_V2/PCB_PAPI.kicad_pcb (KiCad board)
At the start: 8 copper layers, 50 x 43.3 mm, 141 parts, among them IC1 LMR51625YFDDCR, IC2 LDO40LPU33RY, IC3 LDO40LPU33RY, IC4 ESP32-C6FH4, IC5 ADXL343BCCZ-RL, IC6 MAX98357AETE+, IC8 74HCT1G125GW-Q100H, J1 USB4110-GF-A, J2 636101111001, J3 XT30PW-M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

Commit message: up
Parts:
- removed C28, C30: 100n, Capacitor_SMD:C_0201_0603Metric
- removed C29, C32: TBD, Capacitor_SMD:C_0402_1005Metric
- removed C31, C37: 100n, samacsys:C_0201_custom
- removed C33, C36: 1u, Capacitor_SMD:C_0402_1005Metric
- removed C34, C35: 10n, samacsys:C_0201_custom
- removed H1, H2: MountingHole_Pad, MountingHole:MountingHole_2.5mm_Pad_Via
- removed IC4: ESP32-C6FH4, samacsys:QFN50P500X500X90-33N
- removed L2: 2nH, Inductor_SMD:L_0402_1005Metric
- removed L3: TBD, Inductor_SMD:L_0402_1005Metric
- removed REF**: QFN-56-1EP_7x7mm_P0.4mm_EP5.6x5.6mm, Package_DFN_QFN:QFN-56-1EP_7x7mm_P0.4mm_EP5.6x5.6mm
- removed S2: 435151014824, samacsys:435151014824
- added C23: 10u, Capacitor_SMD:C_0603_1608Metric, F.Cu at (180.8, 95.5)
- added C47: 10u, Capacitor_SMD:C_0402_1005Metric_Pad0.74x0.62mm_HandSolder, F.Cu at (159.3, 89.3)
- added C59: 10p, Capacitor_SMD:C_0201_0603Metric_Pad0.64x0.40mm_HandSolder, F.Cu at (168.7, 80.0)
- added C60: 1u, Capacitor_SMD:C_0402_1005Metric_Pad0.74x0.62mm_HandSolder, F.Cu at (159.3, 91.3)
- added C61: 100n, Capacitor_SMD:C_0201_0603Metric_Pad0.64x0.40mm_HandSolder, F.Cu at (168.7, 81.7)
- added C62: 1u, Capacitor_SMD:C_0402_1005Metric_Pad0.74x0.62mm_HandSolder, F.Cu at (159.3, 93.3)
- added C63: 100n, Capacitor_SMD:C_0201_0603Metric_Pad0.64x0.40mm_HandSolder, F.Cu at (168.7, 83.5)
- added C64: 10p, Capacitor_SMD:C_0201_0603Metric_Pad0.64x0.40mm_HandSolder, F.Cu at (168.7, 85.2)
- added C65: 10n, Capacitor_SMD:C_0201_0603Metric_Pad0.64x0.40mm_HandSolder, F.Cu at (171.5, 80.0)
- added C66: 100n, Capacitor_SMD:C_0201_0603Metric_Pad0.64x0.40mm_HandSolder, F.Cu at (171.5, 81.7)
- added C67: 100n, Capacitor_SMD:C_0201_0603Metric_Pad0.64x0.40mm_HandSolder, F.Cu at (171.5, 83.5)
- added C68: 100n, Capacitor_SMD:C_0201_0603Metric_Pad0.64x0.40mm_HandSolder, F.Cu at (171.5, 85.2)
- added C69: 1.56n, Capacitor_SMD:C_0402_1005Metric_Pad0.74x0.62mm_HandSolder, F.Cu at (159.3, 95.2)
- added C70: 1.56n, Capacitor_SMD:C_0402_1005Metric_Pad0.74x0.62mm_HandSolder, F.Cu at (159.3, 97.2)
- added C71: 100n, Capacitor_SMD:C_0201_0603Metric_Pad0.64x0.40mm_HandSolder, F.Cu at (174.3, 80.0)
- added L4: 2.2n, Inductor_SMD:L_0603_1608Metric, F.Cu at (172.2, 89.6)
- added L5: 2.7n, Inductor_SMD:L_0603_1608Metric, F.Cu at (172.2, 92.1)
- added R29: 100R, Resistor_SMD:R_0201_0603Metric_Pad0.64x0.40mm_HandSolder, F.Cu at (174.3, 81.7)
- added R35: 20k, Resistor_SMD:R_0201_0603Metric_Pad0.64x0.40mm_HandSolder, F.Cu at (174.3, 83.5)
- added R36: 20k, Resistor_SMD:R_0201_0603Metric_Pad0.64x0.40mm_HandSolder, F.Cu at (174.3, 85.2)
- added SW1: BOOTMODE, samacsys:KXT341LHS, F.Cu at (164.3, 91.0)
- added U5: ESP32-S3, Package_DFN_QFN:QFN-56-1EP_7x7mm_P0.4mm_EP4x4mm, F.Cu at (140.7, 81.4)
- added Y3: 40Mhz, samacsys:LFXTAL069527REEL, F.Cu at (171.7, 96.9)
- C21: value 1u -> 10u; footprint Capacitor_SMD:C_0402_1005Metric -> Capacitor_SMD:C_0603_1608Metric
- C25: value 10u -> 22u; footprint Capacitor_SMD:C_0402_1005Metric -> Capacitor_SMD:C_0603_1608Metric
- C26: value 1u -> 430pF; footprint Capacitor_SMD:C_0402_1005Metric -> Capacitor_SMD:C_0201_0603Metric
- C27: value 10n -> 22u; footprint samacsys:C_0201_custom -> Capacitor_SMD:C_0603_1608Metric
- IC2: value LDO40LPU33RY -> TPS82150SILR; footprint samacsys:SON95P300X300X90-7N-D -> samacsys2:TPS82130SILT
- R19: value 10k -> 100k
- R20: value 10k -> 309k
- R21: value 20R -> 100k; footprint samacsys:R_0201_custom -> Resistor_SMD:R_0201_0603Metric; moved to F.Cu
- moved R20 47.6 mm to (184.0, 98.6), turned to 0 degrees
- moved C27 47.6 mm to (180.8, 100.5), turned to 0 degrees
- moved R19 47.6 mm to (184.0, 96.8), turned to 0 degrees
- moved R21 43.4 mm to (184.0, 100.3), turned to 0 degrees
- moved C26 39.7 mm to (184.0, 95.1), turned to 0 degrees
- moved C25 37.2 mm to (180.8, 98.0), turned to 0 degrees
- moved LED1 36.6 mm to (175.0, 95.2), turned to 0 degrees
- moved Y2 29.7 mm to (171.7, 94.6), turned to 0 degrees
- moved C39 29.1 mm to (169.0, 91.0), turned to 0 degrees
- moved C40 27.8 mm to (169.0, 92.7), turned to 0 degrees
- moved R22 26.7 mm to (169.0, 94.5)
- moved C38 24.5 mm to (169.0, 89.2), turned to 0 degrees
- moved J2 17.6 mm to (163.4, 95.7), turned to 0 degrees
- moved C21 3.27 mm to (124.9, 76.6)
- moved IC2 1.57 mm to (128.2, 74.0), turned to 0 degrees
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Connections:
- net /ESP32/HSE_IN renamed HSE_IN
- C26 pad 1: +3.3V -> Net-(IC2-SS/TR)
- C27 pad 1: GND -> +3.3V
- C27 pad 2: /ESP32/BOOT1 -> GND
- IC2 pad 1: GND -> 4.5V
- IC2 pad 3: 4.5V -> GND
- IC2 pad 6: unconnected-(IC2-ADJ/NC-Pad6) -> Net-(IC2-FB)
- IC2 pad 7: GND -> Net-(IC2-PG)
- R19 pad 2: /ESP32/BOOT1 -> Net-(IC2-PG)
- R20 pad 2: /ESP32/BOOT0 -> Net-(IC2-FB)
- R21 pad 1: +3.3V -> Net-(IC2-FB)
- R21 pad 2: /ESP32/CHIP_PU -> GND
- R22 pad 1: /ESP32/HSE_OUT -> HSE_OUT
Routing:
- net /ESP32/BOOT1: track 7.67 -> 0.00 mm
- net /D+ESP32: track 6.84 -> 0.00 mm
- net /D-ESP32: track 6.59 -> 0.00 mm
- net /ESP32/LEDPWM: track 5.33 -> 0.00 mm
- net /ESP32_TX: track 3.77 -> 0.00 mm
- net HSE_IN: track 3.63 -> 0.00 mm
- net /ESP32_RX: track 2.88 -> 0.00 mm
- net /ESP32/CHIP_PU: track 2.70 -> 0.00 mm, vias 1 -> 0
- net Net-(IC4-ANT): track 2.42 -> 0.00 mm
- net Net-(C70-Pad1): track 2.34 -> 0.00 mm
- net Net-(IC4-VDDA3P3_1): track 2.30 -> 0.00 mm
- net /ESP32/HSE_OUT: track 1.83 -> 0.00 mm
- net Net-(Y2-CRYSTAL__1): track 1.70 -> 0.00 mm
- net /ESP32/BOOT0: track 1.66 -> 0.00 mm
- net +3.3V: track 2.59 -> 1.41 mm, vias 36 -> 25
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- removed copper zone on F.Cu, net Net-(IC4-VDDA3P3_1)

Commit message: up
Parts:
- removed the C23 at (126.7, 76.5)
- added C28: 4.7u, Capacitor_SMD:C_0402_1005Metric_Pad0.74x0.62mm_HandSolder, F.Cu at (181.9, 68.3)
- added C29: 100n, Capacitor_SMD:C_0201_0603Metric, F.Cu at (181.5, 63.0)
- added C30: 100n, Capacitor_SMD:C_0201_0603Metric_Pad0.64x0.40mm_HandSolder, F.Cu at (189.1, 68.3)
- added C44: 100n, Capacitor_SMD:C_0201_0603Metric, F.Cu at (181.5, 64.7)
- added C45: 10u, Capacitor_SMD:C_0402_1005Metric, F.Cu at (185.0, 68.3)
- added IC6: MAX98357AETE+, samacsys:QFN50P300X300X80-17N, F.Cu at (190.3, 64.7)
- added J4: 47309-2651, samacsys:473092651, F.Cu at (123.7, 82.9)
- added MK1: INMP441ACEZ-R7, INMP441:MIC_INMP441ACEZ-R7, F.Cu at (222.3, 88.2)
- added R29: 47k, Resistor_SMD:R_0201_0603Metric, F.Cu at (181.5, 66.5)
- added R30: 300k, Resistor_SMD:R_0201_0603Metric, F.Cu at (184.0, 63.0)
- added R31: 0R, samacsys:R_0201_custom, F.Cu at (184.0, 64.7)
- added R32: 0R, Resistor_SMD:R_0201_0603Metric, F.Cu at (184.0, 66.5)
- added R33: 300k, Resistor_SMD:R_0201_0603Metric, F.Cu at (186.4, 63.0)
- added R34: 10k, Resistor_SMD:R_0201_0603Metric, F.Cu at (186.4, 64.7)
- added R37: 20k, Resistor_SMD:R_0201_0603Metric_Pad0.64x0.40mm_HandSolder, F.Cu at (226.9, 86.0)
- added R38: 47k, Resistor_SMD:R_0201_0603Metric, F.Cu at (186.4, 66.5)
- J5: moved to B.Cu
- Q1, R15, R16: moved to F.Cu
- USBJUMP1: footprint Connector_PinHeader_1.00mm:PinHeader_2x04_P1.00mm_Vertical_SMD -> Connector_PinHeader_1.27mm:PinHeader_2x04_P1.27mm_Vertical_SMD
- moved U2 170.4 mm to (229.1, 65.4)
- moved U3 165.8 mm to (235.8, 65.4)
- moved R16 68.7 mm to (80.5, 101.5), turned to 120 degrees
- moved Q1 67.6 mm to (82.9, 103.5), turned to -60 degrees
- moved R15 66.8 mm to (81.3, 100.8), turned to 120 degrees
- moved R21 65.3 mm to (125.5, 71.4), turned to 90 degrees
- moved R20 65.1 mm to (124.8, 71.4), turned to -90 degrees
- moved R19 65.1 mm to (124.1, 71.4), turned to -90 degrees
- moved C26 65.1 mm to (123.4, 71.4), turned to 90 degrees
- moved C23 64.9 mm to (119.5, 74.1), turned to 180 degrees
- moved C27 57.7 mm to (129.1, 74.8)
- moved C25 57.2 mm to (129.1, 73.3)
- moved G*** 27.1 mm to (93.5, 81.9)
- moved C38 19.3 mm to (188.3, 87.7)
- moved C39 19.3 mm to (188.2, 89.4)
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Connections:
- net BOOT0 renamed Net-(U5-GPIO0)
- C40 pad 1: HSE_IN -> /ESP32/HSE_IN
- J5 pad 1: /HP+ -> /GND_CONTROLLED
- J5 pad 10: /SDA_OLED -> /RX_SUP
- J5 pad 11: +3.3V -> /HP-
- J5 pad 12: /GND_CONTROLLED -> /HP+
- J5 pad 2: /HP- -> +3.3V
- J5 pad 3: /RX_SUP -> /SDA_OLED
- J5 pad 4: /TX_SUP -> /SCL_OLED
- J5 pad 5: /LED_TIM -> GND
- J5 pad 6: GND -> 4.5V
- J5 pad 7: 4.5V -> GND
- J5 pad 8: GND -> /LED_TIM
- J5 pad 9: /SCL_OLED -> /TX_SUP
- R22 pad 1: HSE_OUT -> /ESP32/HSE_OUT
- U5 pad 10: unconnected-(U5-GPIO5-Pad10) -> /ESP32/mic_sck
- U5 pad 11: unconnected-(U5-GPIO6-Pad11) -> /ESP32/mic_data
- U5 pad 15: unconnected-(U5-GPIO10-Pad15) -> /ESP32/SD_FSPICS
- U5 pad 16: unconnected-(U5-GPIO11-Pad16) -> /ESP32/SD_FSPID
- U5 pad 17: unconnected-(U5-GPIO12-Pad17) -> /ESP32/SD_FSPICLK
- U5 pad 18: unconnected-(U5-GPIO13-Pad18) -> /ESP32/SD_FSPIQ
- U5 pad 23: unconnected-(U5-GPIO17-Pad23) -> /ESP32_TX
- U5 pad 24: unconnected-(U5-GPIO18-Pad24) -> /ESP32_RX
- U5 pad 29: VDD_SPI -> unconnected-(U5-VDD_SPI-Pad29)
- U5 pad 52: BOOT1 -> /ESP32/BOOT1
- U5 pad 53: HSE_IN -> /ESP32/HSE_IN
- U5 pad 54: HSE_OUT -> /ESP32/HSE_OUT
- U5 pad 9: unconnected-(U5-GPIO4-Pad9) -> /ESP32/mic_frame_sck
- Y2 pad 3: HSE_IN -> /ESP32/HSE_IN
Routing:
- net /TX_MOT1: track 46.9 -> 10.0 mm, vias 3 -> 0
- net /STM32/LED0: track 25.7 -> 0.00 mm, vias 1 -> 0
- net /RX_MOT1: track 22.6 -> 0.00 mm, vias 1 -> 0
- net /GPIO_MOT1: track 21.6 -> 0.00 mm, vias 1 -> 0
- net /TX_MOT3: track 20.6 -> 0.33 mm, vias 1 -> 0
- net /NRST: track 35.1 -> 16.2 mm, vias 3 -> 1
- net /RX_SUP: track 13.8 -> 0.00 mm, vias 2 -> 0
- net /TX_SUP: track 13.5 -> 0.00 mm, vias 2 -> 0
- net /GND_CONTROl_GPIO: track 13.5 -> 0.00 mm, vias 2 -> 0
- net /SCL_OLED: track 13.4 -> 0.00 mm
- net /SDA_OLED: track 12.7 -> 0.00 mm
- net /STM32/ADC_VBAT: track 12.3 -> 2.08 mm, vias 2 -> 1
- net /LED_TIM: track 10.1 -> 0.00 mm
- net /CONNECTOR/DATA-OUT: track 7.85 -> 0.00 mm
- net /SCL_TOF1: track 7.70 -> 0.00 mm, vias 1 -> 0
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
Commit message: up
Parts:
- removed the C47 at (178.5, 87.8)
- removed the C47 at (126.6, 87.1)
- removed C59, C64: 10p, Capacitor_SMD:C_0201_0603Metric_Pad0.64x0.40mm_HandSolder
- removed ESC2: SM08B-SRSS-TBLFSN, Connector_JST:JST_SHL_SM08B-SHLS-TF_1x08-1MP_P1.00mm_Horizontal
- removed the R29 at (193.5, 80.2)
- removed the R29 at (181.5, 66.5)
- removed Y3: 40Mhz, samacsys:LFXTAL069527REEL
- added C31: 100n, Capacitor_SMD:C_0201_0603Metric_Pad0.64x0.40mm_HandSolder, F.Cu at (137.4, 78.0)
- added C32: 1u, Capacitor_SMD:C_0402_1005Metric_Pad0.74x0.62mm_HandSolder, B.Cu at (137.4, 78.2)
- added C47: 10u, Capacitor_SMD:C_0402_1005Metric_Pad0.74x0.62mm_HandSolder, F.Cu at (152.4, 83.0)
- added H1: MountingHole_Pad, MountingHole:MountingHole_2.5mm_Pad_Via, F.Cu at (178.4, 54.1)
- added H2: MountingHole_Pad, MountingHole:MountingHole_2.5mm_Pad_Via, F.Cu at (178.4, 60.6)
- added J6: DF52-8S-0.8H_21_, samacsys2:DF528S08H21, F.Cu at (115.7, 82.3)
- added R29: 47k, Resistor_SMD:R_0201_0603Metric, F.Cu at (216.1, 88.7)
- added R39: 20k, Resistor_SMD:R_0201_0603Metric_Pad0.64x0.40mm_HandSolder, B.Cu at (142.0, 86.8)
- added R40: 22R, Resistor_SMD:R_0201_0603Metric, F.Cu at (211.8, 95.8)
- added R41: 0R, Resistor_SMD:R_0402_1005Metric_Pad0.72x0.64mm_HandSolder, B.Cu at (135.2, 78.2)
- added R42: 22R, Resistor_SMD:R_0201_0603Metric, F.Cu at (184.8, 109.7)
- C30, C56, C61, C68, C71, IC8, MK1, R23, R35, R36, R37, SW1, U2, U3: moved to B.Cu
- moved U2 116.2 mm to (113.3, 74.1), turned to -30 degrees
- moved U3 112.8 mm to (128.9, 101.3), turned to 90 degrees
- moved R16 112.7 mm to (192.8, 91.7), turned to 0 degrees
- moved R15 112.0 mm to (192.8, 90.0), turned to 0 degrees
- moved Q1 106.7 mm to (188.9, 91.4), turned to 0 degrees
- moved R37 84.2 mm to (142.7, 86.8), turned to 90 degrees
- moved R30 77.8 mm to (131.2, 120.1)
- moved R32 77.4 mm to (127.8, 119.7)
- moved R31 76.9 mm to (127.1, 116.4)
- moved IC6 74.8 mm to (136.8, 117.1)
- moved MK1 74.4 mm to (148.4, 79.8), turned to -150 degrees
- moved C44 73.3 mm to (131.6, 118.4)
- moved C45 72.0 mm to (131.8, 116.9)
- moved C68 51.0 mm to (139.8, 86.7)
- moved C71 49.5 mm to (144.4, 84.8)
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Connections:
- net /ACCESOIRES/LED_TOM_JERRY_RGB renamed /RGB_TOM_JERRY
- net /STM32/FLASH_CLK_SPI1 renamed /STM32/MOUSE_CLK_SPI1
- net /STM32/FLASH_CS_SPI1 renamed /STM32/MOUSE_CS_SPI1
- net /STM32/FLASH_MISO_SPI1 renamed /STM32/MOUSE_MISO_SPI1
- net /STM32/FLASH_MOSI_SPI1 renamed /STM32/MOUSE_MOSI_SPI1
- J4 pad 5: /ESP32/SD_FSPICLK -> Net-(J4-Pad5)
- U1 pad D7: /SAI_FS -> unconnected-(U1-PD4-PadD7)
- U1 pad D8: /SAI_CLK -> unconnected-(U1-PD0-PadD8)
- U1 pad E8: /SAI_SD -> unconnected-(U1-PD1-PadE8)
- U1 pad G3: /AMPLI_SD_MODE -> unconnected-(U1-PA4-PadG3)
- U5 pad 10: /ESP32/mic_sck -> /ESP32/max_gpio
- U5 pad 11: /ESP32/mic_data -> /ESP32/mic_frame_sck
- U5 pad 12: unconnected-(U5-GPIO7-Pad12) -> /ESP32/mic_data
- U5 pad 13: unconnected-(U5-GPIO8-Pad13) -> /ESP32/mic_sck
- U5 pad 22: unconnected-(U5-XTAL_32K_N-Pad22) -> /ESP32/LEDPWM
- U5 pad 29: unconnected-(U5-VDD_SPI-Pad29) -> Net-(U5-VDD_SPI)
- U5 pad 51: +3.3V -> Net-(U5-GPIO45)
- U5 pad 6: unconnected-(U5-GPIO1-Pad6) -> /ESP32/max_frame_clk
- U5 pad 7: unconnected-(U5-GPIO2-Pad7) -> /ESP32/max_bit_clk
- U5 pad 9: /ESP32/mic_frame_sck -> /ESP32/max_data
Routing:
- net /RX_MOT2: track 19.5 -> 0.00 mm
- net /SDA_TOF2: track 19.1 -> 0.00 mm
- net /SCL_TOF2: track 19.2 -> 0.67 mm
- net /GPIO_MOT2: track 17.0 -> 0.00 mm
- net /TX_MOT2: track 16.7 -> 0.00 mm
- net /STM32/LED1: track 12.8 -> 0.00 mm
- net /SDA_TOF1: track 11.4 -> 0.00 mm, vias 0 -> 1
- net /TX_MOT1: track 10.0 -> 0.00 mm, vias 0 -> 1
- net /D+ESP32: track 0.00 -> 8.01 mm
- net /NRST: track 16.2 -> 8.68 mm, vias 1 -> 2
- net /LIDAR_PWM: track 22.4 -> 15.0 mm, vias 1 -> 2
- net /RX_LIDAR: track 20.2 -> 12.9 mm, vias 1 -> 2
- net /D-ESP32: track 0.00 -> 6.93 mm
- net /ESP32/mic_frame_sck: track 0.00 -> 6.04 mm, vias 0 -> 1
- net /AMPLI_SD_MODE: track 5.27 -> 0.00 mm
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- added copper zone on In6.Cu, net GND
- removed copper zone on In2.Cu, net GND
- removed copper zone on In4.Cu, net GND
Other:
- board text removed: "POWERBUTTON"

Commit message: up
Parts:
- removed the C44 at (137.7, 96.3)
- removed the C45 at (137.5, 97.1)
- removed the IC6 at (136.5, 93.8)
- removed the R30 at (133.6, 94.6)
- removed the R31 at (133.6, 93.1)
- removed the R32 at (132.9, 93.1)
- removed U2, U3, U4: ~, samacsys:pin_header_smt_14pin
- added J7: ERF8-005-05.0-L-DV-K-TR, ERF8:SAMTEC_ERF8-005-05.0-L-DV-K-TR, B.Cu at (144.7, 73.9)
- added J8: ERF8-005-05.0-L-DV-K-TR, ERF8:SAMTEC_ERF8-005-05.0-L-DV-K-TR, B.Cu at (129.0, 101.2)
- added J9: ERF8-005-05.0-L-DV-K-TR, ERF8:SAMTEC_ERF8-005-05.0-L-DV-K-TR, B.Cu at (113.3, 73.9)
- added R45: 22R, Resistor_SMD:R_0201_0603Metric, F.Cu at (110.0, 87.4)
- C1, R1, R2: moved to F.Cu
- TOF1, TOF2, TOF3: footprint Connector_JST:JST_GH_BM04B-GHS-TBT_1x04-1MP_P1.25mm_Vertical -> samacsys:JST_GH_BM04B
- moved R38 98.5 mm to (120.1, 83.7)
- moved R34 97.9 mm to (120.1, 84.4)
- moved R29 96.4 mm to (120.1, 79.7)
- moved C28 93.9 mm to (119.1, 82.0), turned to 180 degrees
- moved R40 92.6 mm to (120.4, 80.8), turned to -90 degrees
- moved C29 92.1 mm to (119.4, 82.9), turned to 180 degrees
- moved R42 78.4 mm to (110.1, 86.0), turned to 180 degrees
- moved C39 53.7 mm to (148.2, 116.6)
- moved LED1 53.7 mm to (148.0, 114.2)
- moved R32 27.0 mm to (132.9, 93.1), turned to 90 degrees
- moved R15 26.5 mm to (166.3, 91.1)
- moved R16 26.5 mm to (166.3, 92.8)
- moved Q1 26.5 mm to (162.4, 92.5)
- moved R30 25.6 mm to (133.6, 94.6), turned to -90 degrees
- moved R31 24.2 mm to (133.6, 93.1), turned to -90 degrees
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Connections:
- J6 pad 2: /CONNECTOR/MOUSE_CS -> /MOUSE_CS
- J6 pad 5: /CONNECTOR/MOUSE_MISO -> /MOUSE_MISO
- J6 pad 7: /CONNECTOR/MOUSE_MOSI -> Net-(J6-Pad7)
- J6 pad 8: /CONNECTOR/MOUSE_INT -> /MOUSE_INT
- R42 pad 2: /CONNECTOR/MOUSE_CLK -> /MOUSE_CLK
- U1 pad A2: unconnected-(U1-PC13-PadA2) -> /MOUSE_INT
- U1 pad A6: /STM32/MOUSE_MISO_SPI1 -> /MOUSE_MISO
- U1 pad A7: /STM32/MOUSE_CLK_SPI1 -> /MOUSE_CLK
- U1 pad A8: /STM32/MOUSE_CS_SPI1 -> /MOUSE_CS
- U1 pad B1: unconnected-(U1-PC15-PadB1) -> /STM32/ADC_VBAT
- U1 pad B5: unconnected-(U1-PB6-PadB5) -> /RGB_TOM_JERRY
- U1 pad B8: /STM32/ADC_VBAT -> unconnected-(U1-PC11-PadB8)
- U1 pad C5: /STM32/MOUSE_MOSI_SPI1 -> /MOUSE_MOSI
Routing:
- net /ESP32/SD_FSPICS: track 0.67 -> 28.6 mm, vias 1 -> 2
- net /ESP32/SD_FSPIQ: track 0.61 -> 28.3 mm, vias 1 -> 2
- net /ESP32/SD_FSPICLK: track 0.66 -> 27.1 mm, vias 1 -> 2
- net /ESP32/SD_FSPID: track 0.60 -> 26.3 mm, vias 1 -> 2
- net /ESP32/max_gpio: track 0.73 -> 20.7 mm, vias 1 -> 2
- net /ESP32/max_data: track 0.72 -> 17.7 mm, vias 1 -> 2
- net /ESP32/max_bit_clk: track 0.68 -> 16.9 mm, vias 1 -> 2
- net /ESP32/max_frame_clk: track 0.74 -> 14.0 mm, vias 1 -> 2
- net /RX_LIDAR: track 12.9 -> 24.7 mm
- net /CONNECTOR/DATA-OUT: track 0.00 -> 9.98 mm
- net /MOUSE_CS: track 0.00 -> 9.87 mm, vias 0 -> 2
- net /LIDAR_PWM: track 15.0 -> 24.8 mm
- net /MOUSE_MISO: track 0.00 -> 9.17 mm, vias 0 -> 2
- net Net-(J6-Pad3): track 0.00 -> 8.20 mm
- net /D-STM32: track 0.00 -> 8.15 mm
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- added copper zone on F.Cu, net Net-(C66-Pad1)
- added copper zone on B.Cu, net Net-(U5-VDD_SPI)
- added copper zone on F.Cu, net Net-(U5-VDD_SPI)

Commit message: up
Parts:
- removed the G*** at (118.8, 66.2)
- removed the G*** at (118.3, 99.9)
- removed the G*** at (93.5, 81.9)
- removed the H3 at (139.5, 101.2)
- removed the H3 at (108.0, 83.0)
- removed Q1: STR2N2VH5, samacsys:SOT95P255X140-3N
- removed R15: 100R, Resistor_SMD:R_0201_0603Metric
- removed R16: 100k, samacsys:R_0201_custom
- SWD1: footprint Connector_JST:JST_GH_SM04B-GHS-TB_1x04-1MP_P1.25mm_Horizontal -> samacsys:JST_GH_BM04B
- moved H2 73.9 mm to (108.0, 83.0)
- moved H1 61.1 mm to (139.5, 101.2)
- moved C39 31.0 mm to (138.9, 87.0), turned to 180 degrees
- moved LED1 26.8 mm to (139.2, 88.9)
- moved R35 3.19 mm to (150.1, 84.2)
- moved R36 3.19 mm to (150.1, 85.0)
- moved C61 3.19 mm to (150.1, 83.5)
- moved R23 3.06 mm to (109.3, 80.2), turned to -30 degrees
- moved C30 0.93 mm to (151.5, 81.5)
- moved MK1 0.42 mm to (148.7, 80.2)
- moved C46 0.30 mm to (124.1, 93.4)
- moved C48 0.28 mm to (125.5, 94.8)
- moved C49 0.27 mm to (126.9, 96.2)
- moved C32 0.25 mm to (137.7, 78.2)
- moved R41 0.25 mm to (135.5, 78.2)
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Connections:
- J5 pad 1: /GND_CONTROLLED -> GND
- SWD1 pad 1: /SWDIO -> GND
- SWD1 pad 2: /SWCLK -> /NRST
- SWD1 pad 3: /NRST -> /SWCLK
- SWD1 pad 4: GND -> /SWDIO
- U1 pad B5: /RGB_TOM_JERRY -> unconnected-(U1-PB6-PadB5)
- U1 pad C9: unconnected-(U1-PA9-PadC9) -> /RGB_TOM_JERRY
- U1 pad H7: /GND_CONTROl_GPIO -> unconnected-(U1-PE15-PadH7)
Routing:
- net /TX_MOT3: track 0.00 -> 27.9 mm, vias 1 -> 2
- net /GPIO_MOT3: track 0.00 -> 26.6 mm, vias 1 -> 2
- net /RX_MOT3: track 0.00 -> 26.0 mm, vias 1 -> 2
- net /RGB_TOM_JERRY: track 0.00 -> 23.7 mm, vias 1 -> 2
- net /MOUSE_MOSI: track 0.00 -> 23.1 mm
- net /GPIO_MOT2: track 0.00 -> 22.8 mm, vias 1 -> 2
- net /TX_MOT2: track 0.00 -> 22.6 mm, vias 1 -> 2
- net /SDA_TOF3: track 0.57 -> 22.9 mm, vias 1 -> 2
- net /RX_MOT2: track 0.00 -> 21.7 mm, vias 1 -> 2
- net /MOUSE_MISO: track 9.17 -> 30.8 mm
- net /SCL_TOF3: track 0.00 -> 21.6 mm, vias 1 -> 2
- net /MOUSE_CS: track 9.87 -> 31.3 mm
- net /GPIO_MOT1: track 0.00 -> 21.2 mm, vias 1 -> 2
- net /MOUSE_CLK: track 0.00 -> 20.4 mm
- net /MOUSE_INT: track 7.59 -> 26.8 mm, vias 1 -> 2
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- added copper zone on In4.Cu, net GND

Commit message: up
Parts:
- removed MK1: INMP441ACEZ-R7, INMP441:MIC_INMP441ACEZ-R7
- added MK2: ICS-43434, Sensor_Audio:InvenSense_ICS-43434-6_3.5x2.65mm, B.Cu at (149.1, 79.9)
Connections:
- U5 pad 11: /ESP32/mic_frame_sck -> /ESP32/mic_sck
- U5 pad 13: /ESP32/mic_sck -> /ESP32/mic_frame_sck
Routing:
- net /ESP32/mic_sck: track 3.85 -> 10.8 mm
- net /ESP32/mic_frame_sck: track 6.47 -> 3.85 mm
- net /ESP32/mic_data: track 5.21 -> 3.00 mm
- net Net-(MK2-LR): track 2.08 -> 3.24 mm
- net /ESP32/max_gpio: track 21.1 -> 22.0 mm
- net GND: vias 385 -> 386

Commit message: pcb v2
Parts:
- added G***: LOGO, LOGO, F.Cu at (143.3, 96.8)
- added G***: LOGO, LOGO, F.Cu at (147.6, 79.6)
- added R15: 20k, Resistor_SMD:R_0201_0603Metric_Pad0.64x0.40mm_HandSolder, B.Cu at (147.2, 81.8)
Connections:
- U5 pad 8: unconnected-(U5-GPIO3-Pad8) -> Net-(U5-GPIO3)
Routing:
- net GND: track 0.53 -> 79.4 mm, vias 386 -> 440
- net Net-(U5-GPIO3): track 0.00 -> 3.83 mm, vias 0 -> 1
- net /ESP32/max_data: track 18.0 -> 18.7 mm
- net /GPIO_MOT1: track 21.2 -> 21.8 mm
- net Net-(U1-BOOT0): track 11.1 -> 11.5 mm, vias 2 -> 3
- net +3.3V: vias 29 -> 31
- added copper zone on In2.Cu, net GND
Other:
- board size 50 x 43.3 mm -> 50 x 48.6 mm
- board text added: "GPIO0"
- board text added: "GREEN LINE ON USER.ECO1 NEED TO BE V CUT SCORE"
- board text added: "MOUSE SENSOR"
- board text removed: "Mounting hole R = 21 mm"
