File: HARDWARE/ELECTRONIQUE/PCB_PAPI_V2/PCB_PAPI.kicad_pcb (KiCad board)
At the start: 8 copper layers, 50 x 48.6 mm, 155 parts, among them IC1 LMR51625YFDDCR, IC2 TPS82150SILR, IC3 LDO40LPU33RY, IC5 ADXL343BCCZ-RL, IC6 MAX98357AETE+, IC8 74HCT1G125GW-Q100H, J1 USB4110-GF-A, J2 636101111001, J3 XT30PW-M, J4 47309-2651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

Commit message: up
Parts:
- added REF**: BreakLine_5h_D0.5mm_P0.85mm, Panelization:BreakLine_5h_D0.5mm_P0.85mm, F.Cu at (123.0, 61.0)
- added REF**: BreakLine_5h_D0.5mm_P0.85mm, Panelization:BreakLine_5h_D0.5mm_P0.85mm, F.Cu at (118.8, 105.0)
- added REF**: BreakLine_2h_D0.5mm_P0.85mm, Panelization:BreakLine_2h_D0.5mm_P0.85mm, F.Cu at (138.8, 61.0)
- added REF**: BreakLine_5h_D0.5mm_P0.85mm, Panelization:BreakLine_5h_D0.5mm_P0.85mm, F.Cu at (135.8, 105.0)
- added REF**: BreakLine_2h_D0.5mm_P0.85mm, Panelization:BreakLine_2h_D0.5mm_P0.85mm, F.Cu at (140.5, 61.0)
- added REF**: BreakLine_5h_D0.5mm_P0.85mm, Panelization:BreakLine_5h_D0.5mm_P0.85mm, F.Cu at (131.6, 105.0)
- added REF**: BreakLine_5h_D0.5mm_P0.85mm, Panelization:BreakLine_5h_D0.5mm_P0.85mm, F.Cu at (118.8, 61.0)
- added REF**: BreakLine_5h_D0.5mm_P0.85mm, Panelization:BreakLine_5h_D0.5mm_P0.85mm, F.Cu at (135.8, 61.0)
- added REF**: BreakLine_2h_D0.5mm_P0.85mm, Panelization:BreakLine_2h_D0.5mm_P0.85mm, F.Cu at (140.5, 105.0)
- added REF**: BreakLine_5h_D0.5mm_P0.85mm, Panelization:BreakLine_5h_D0.5mm_P0.85mm, F.Cu at (127.3, 61.0)
- added REF**: BreakLine_5h_D0.5mm_P0.85mm, Panelization:BreakLine_5h_D0.5mm_P0.85mm, F.Cu at (131.6, 61.0)
- added REF**: BreakLine_5h_D0.5mm_P0.85mm, Panelization:BreakLine_5h_D0.5mm_P0.85mm, F.Cu at (127.3, 105.0)
- added REF**: BreakLine_5h_D0.5mm_P0.85mm, Panelization:BreakLine_5h_D0.5mm_P0.85mm, F.Cu at (123.1, 105.0)
- added REF**: BreakLine_2h_D0.5mm_P0.85mm, Panelization:BreakLine_2h_D0.5mm_P0.85mm, F.Cu at (138.8, 105.0)
Other:
- board text added: "V2.0"
- board text removed: "GREEN LINE ON USER.ECO1 NEED TO BE V CUT SCORE"
- board text removed: "V1.0"
