File: HARDWARE/ELECTRONIQUE/PCB_PAPI_V2/esp32.kicad_sch (KiCad schematic)
At the start: 26 parts, among them J2 636101111001, Y2 LFXTAL069527REEL

Commit message: up
Parts:
- removed C25: 10u, Capacitor_SMD:C_0402_1005Metric, symbol Device:C_Small
- removed C26, C33, C36: 1u, Capacitor_SMD:C_0402_1005Metric, symbol Device:C_Small
- removed C27, C34, C35: 10n, samacsys:C_0201_custom, symbol Device:C_Small
- removed C28, C30: 100n, Capacitor_SMD:C_0201_0603Metric, symbol Device:C_Small
- removed C29, C32: TBD, Capacitor_SMD:C_0402_1005Metric, symbol Device:C_Small
- removed C31, C37: 100n, samacsys:C_0201_custom, symbol Device:C_Small
- removed L2: 2nH, Inductor_SMD:L_0402_1005Metric, symbol Device:L_Small
- removed L3: TBD, Inductor_SMD:L_0402_1005Metric, symbol Device:L_Small
- removed R19, R20: 10k, Resistor_SMD:R_0201_0603Metric, symbol Device:R_Small
- removed R21: 20R, samacsys:R_0201_custom, symbol Device:R_Small
- removed S2: 435151014824, samacsys:435151014824, symbol samacsys:435151014824
- added C47: 10u, Capacitor_SMD:C_0402_1005Metric_Pad0.74x0.62mm_HandSolder, symbol Device:C_Small
- added C59, C64: 10p, Capacitor_SMD:C_0201_0603Metric_Pad0.64x0.40mm_HandSolder, symbol Device:C_Small
- added C60, C62: 1u, Capacitor_SMD:C_0402_1005Metric_Pad0.74x0.62mm_HandSolder, symbol Device:C_Small
- added C61, C63, C66, C67, C68, C71: 100n, Capacitor_SMD:C_0201_0603Metric_Pad0.64x0.40mm_HandSolder, symbol Device:C_Small
- added C65: 10n, Capacitor_SMD:C_0201_0603Metric_Pad0.64x0.40mm_HandSolder, symbol Device:C_Small
- added C69, C70: 1.56n, Capacitor_SMD:C_0402_1005Metric_Pad0.74x0.62mm_HandSolder, symbol Device:C_Small
- added L4: 2.2n, Inductor_SMD:L_0603_1608Metric, symbol Device:L_Small
- added L5: 2.7n, Inductor_SMD:L_0603_1608Metric, symbol Device:L_Small
- added R29: 100R, Resistor_SMD:R_0201_0603Metric_Pad0.64x0.40mm_HandSolder, symbol Device:R_Small
- added R35, R36: 20k, Resistor_SMD:R_0201_0603Metric_Pad0.64x0.40mm_HandSolder, symbol Device:R_Small
- added SW1: BOOTMODE, samacsys:KXT341LHS, symbol Switch:SW_Omron_B3FS
- added U5: ESP32-S3, Package_DFN_QFN:QFN-56-1EP_7x7mm_P0.4mm_EP4x4mm, symbol MCU_Espressif:ESP32-S3
- added Y3: 40Mhz, samacsys:LFXTAL069527REEL, symbol Device:Crystal_GND24
Connections:
- net +3.3V: now also C47.1, C60.1, C62.1, C63.1, C65.1, C67.2, C68.2, L4.1, R35.1, R36.1, U5.20 (VDD3P3_RTC), U5.46 (VDD3P3_CPU), U5.51 (GPIO45), U5.55 (VDDA), U5.56 (VDDA)
- net BOOT0: now also C61.2, R35.2, SW1.2, U5.5 (GPIO0)
- net BOOT1: now also U5.52 (GPIO46)
- net D+ESP32: now also U5.26 (GPIO20/USB_D+)
- net D-ESP32: now also U5.25 (GPIO19/USB_D-)
- net GND: now also C47.2, C59.2, C60.2, C61.1, C62.2, C63.2, C64.2, C65.2, C66.2, C67.1, C68.1, C69.2, C70.2, C71.1, SW1.1, U5.57 (GND), Y3.2, Y3.4
- net HSE_IN: now also C59.1, U5.53 (XTAL_N), Y3.1
- net HSE_OUT: now also R29.1, U5.54 (XTAL_P)
- net at J2.3: now also C70.1, L5.2
- new net: C64.1, R29.2, Y3.3
- new net: C66.1, L4.2, U5.2 (VDD3P3), U5.3 (VDD3P3)
- new net LNA_IN: C69.1, L5.1, U5.1 (LNA_IN)
- new net RESET: C71.2, R36.2, U5.4 (CHIP_PU)
- new net VDD_SPI: U5.29 (VDD_SPI)
- no-connect marks 4 -> 24
Other:
- note added: "35+j*0R and 2442Mhz"
- note added: "50R"
- note added: "SPI_VDD_SEL"
- moved on the sheet: C38, C39, C40, J2, LED1, R22, Y2

Commit message: up
Parts:
- removed C59, C64: 10p, Capacitor_SMD:C_0201_0603Metric_Pad0.64x0.40mm_HandSolder, symbol Device:C_Small
- removed Y3: 40Mhz, samacsys:LFXTAL069527REEL, symbol Device:Crystal_GND24
- added C28: 4.7u, Capacitor_SMD:C_0402_1005Metric_Pad0.74x0.62mm_HandSolder, symbol Device:C_Small
- added C29, C44: 100n, Capacitor_SMD:C_0201_0603Metric, symbol Device:C_Small
- added C30: 100n, Capacitor_SMD:C_0201_0603Metric_Pad0.64x0.40mm_HandSolder, symbol Device:C_Small
- added C45: 10u, Capacitor_SMD:C_0402_1005Metric, symbol Device:C_Small
- added IC6: MAX98357AETE+, samacsys:QFN50P300X300X80-17N, symbol samacsys:MAX98357AETE+
- added J4: 47309-2651, samacsys:473092651, symbol molex 47309-2651:47309-2651
- added MK1: INMP441ACEZ-R7, INMP441:MIC_INMP441ACEZ-R7, symbol INMP441:INMP441ACEZ-R7
- added R30, R33: 300k, Resistor_SMD:R_0201_0603Metric, symbol Device:R_Small
- added R31: 0R, samacsys:R_0201_custom, symbol Device:R_Small
- added R32: 0R, Resistor_SMD:R_0201_0603Metric, symbol Device:R_Small
- added R34: 10k, Resistor_SMD:R_0201_0603Metric, symbol Device:R_Small
- added R37: 20k, Resistor_SMD:R_0201_0603Metric_Pad0.64x0.40mm_HandSolder, symbol Device:R_Small
- added R38: 47k, Resistor_SMD:R_0201_0603Metric, symbol Device:R_Small
- R29: value 100R -> 47k; footprint Resistor_SMD:R_0201_0603Metric_Pad0.64x0.40mm_HandSolder -> Resistor_SMD:R_0201_0603Metric
Connections:
- net +3.3V: now also R29.1, C28.1, C29.1, C30.2, J4.4, MK1.7 (VDD), MK1.8 (CHIPEN), R34.1, R38.1
- net BOOT1: now also R37.2
- net ESP32_RX: now also U5.24 (GPIO18)
- net ESP32_TX: now also U5.23 (GPIO17)
- net GND: now also C28.2, C29.2, C30.1, C44.2, C45.2, IC6.11 (GND_2), IC6.15 (GND_3), IC6.17 (GND_4), IC6.3 (GND_1), J4.10 (G2), J4.11 (G3), J4.12 (G4), J4.6, J4.9 (G1), MK1.5 (GND), MK1.6 (GND), MK1.9 (GND), R31.1, R33.1, R37.1
- net HSE_OUT: no longer R29.1
- net SD_FSPIQ: now reaches R29.2
- net SD_FSPIQ: now also U5.18 (GPIO13), J4.7
- net mic_sck: now reaches U5.10 (GPIO5)
- net mic_sck: now also MK1.1 (SCK)
- net mic_data: now reaches U5.11 (GPIO6)
- net mic_data: now also MK1.2 (SD)
- net SD_FSPICS: now reaches U5.15 (GPIO10)
- net SD_FSPICS: now also J4.2, R34.2
- net SD_FSPID: now reaches U5.16 (GPIO11)
- net SD_FSPID: now also J4.3, R38.2
- net SD_FSPICLK: now reaches U5.17 (GPIO12)
- net SD_FSPICLK: now also J4.5
- net mic_frame_sck: now reaches U5.9 (GPIO4)
- net mic_frame_sck: now also MK1.3 (WS)
- net BOOT0: no longer names the net of C61.2, R35.2, SW1.2, U5.5 (GPIO0)
- net VDD_SPI: no longer names the net of U5.29 (VDD_SPI)
- new net: IC6.2 (GAIN_SLOT), R31.2, R32.1
- new net: IC6.4 (~{SD_MODE}), R30.2
- new net: MK1.4 (L/R), R33.2
- new net 4.5V: C44.1, C45.1, IC6.7 (VDD_1), IC6.8 (VDD_2), R32.2
- new net HP+: IC6.9 (OUTP)
- new net HP-: IC6.10 (OUTN)
- new net max_bit_clk: IC6.16 (BCLK)
- new net max_data: IC6.1 (DIN)
- new net max_frame_clk: IC6.14 (LRCLK)
- new net max_gpio: R30.1
- no-connect marks 24 -> 30
Other:
- note added: "12dB"
- note added: "6dB"
- note added: "AMPLI"
- note added: "MIC"
- note added: "SD_CARD"
- note added: "a calculer"
- moved on the sheet: C38, C39, C40, C47, C60, C61, C62, C63, C65, C66, C67, C68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

Commit message: up
Parts:
- added C31: 100n, Capacitor_SMD:C_0201_0603Metric_Pad0.64x0.40mm_HandSolder, symbol Device:C_Small
- added C32: 1u, Capacitor_SMD:C_0402_1005Metric_Pad0.74x0.62mm_HandSolder, symbol Device:C_Small
- added R39: 20k, Resistor_SMD:R_0201_0603Metric_Pad0.64x0.40mm_HandSolder, symbol Device:R_Small
- added R40: 22R, Resistor_SMD:R_0201_0603Metric, symbol Device:R_Small
- added R41: 0R, Resistor_SMD:R_0402_1005Metric_Pad0.72x0.64mm_HandSolder, symbol Device:R_Small
Connections:
- net +3.3V: now also R41.2; no longer U5.51 (GPIO45)
- net GND: now also C31.1, C32.2, R39.2
- net LEDPWM: now also U5.22 (XTAL_32K_N)
- net SD_FSPICLK: now also R40.1; no longer J4.5
- net max_bit_clk: now also U5.7 (GPIO2)
- net max_data: now also U5.9 (GPIO4)
- net max_frame_clk: now also U5.6 (GPIO1)
- net max_gpio: now also U5.10 (GPIO5)
- net mic_data: now also U5.12 (GPIO7); no longer U5.11 (GPIO6)
- net mic_frame_sck: now also U5.11 (GPIO6); no longer U5.9 (GPIO4)
- net mic_sck: now also U5.13 (GPIO8); no longer U5.10 (GPIO5)
- net at U5.29 (VDD_SPI): now also C31.2, C32.1, R41.1
- new net: J4.5, R40.2
- new net: R39.1, U5.51 (GPIO45)
- no-connect marks 30 -> 33
Other:
- moved on the sheet: C68

Commit message: up
Parts:
- removed MK1: INMP441ACEZ-R7, INMP441:MIC_INMP441ACEZ-R7, symbol INMP441:INMP441ACEZ-R7
- added MK2: ICS-43434, Sensor_Audio:InvenSense_ICS-43434-6_3.5x2.65mm, symbol Sensor_Audio:ICS-43434
Connections:
- net +3.3V: now also MK2.5 (VDD)
- net GND: now also MK2.3 (GND)
- net mic_data: now also MK2.6 (SD)
- net mic_frame_sck: now also U5.13 (GPIO8), MK2.1 (WS); no longer U5.11 (GPIO6)
- net mic_sck: now also U5.11 (GPIO6), MK2.4 (SCK); no longer U5.13 (GPIO8)
- net at R33.2: now also MK2.2 (LR)
Other:
- moved on the sheet: C30, C44, C45, IC6, R30, R31, R32, R33

Commit message: pcb v2
Parts:
- added R15: 20k, Resistor_SMD:R_0201_0603Metric_Pad0.64x0.40mm_HandSolder, symbol Device:R_Small
Connections:
- net +3.3V: now also R15.1
- net at U5.8 (GPIO3): now also R15.2
- no-connect marks 33 -> 32

Commit message: up
Parts:
- C38, C40: value 15p -> 3p
Other:
- note added: "830069527 40Mhz 15ppm 8pF load 1.6mmx1.2mm"
Changed lines of the file:
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@@
 		)
 	)
+	(text "830069527 40Mhz 15ppm 8pF load 1.6mmx1.2mm"
+		(exclude_from_sim no)
+		(at 218.948 20.32 0)
+		(effects
+			(font
+				(size 1.27 1.27)
+			)
+		)
+	)
 	(text "35+j*0R and 2442Mhz"
 		(exclude_from_sim no)
@@
 			)
 		)
-		(property "Value" "15p"
+		(property "Value" "3p"
 			(at 193.04 34.2962 0)
 			(effects
@@
 			)
 		)
-		(property "Value" "15p"
+		(property "Value" "3p"
 			(at 248.92 34.2962 0)
 			(effects
