File: HARDWARE/ELECTRONIQUE/FOC_CONTROLLER_V2/MOTEUR1.kicad_sch (KiCad schematic)
At the start: 41 parts, among them IC1 STSPIN32G0A2, J1 SM06B-GHS-TB_LF__SN_, J2 SM06B-GHS-TB_LF__SN_

Commit message: up
Other:
- moved on the sheet: C23, C24, C25, C26, C27, C31, C33, C34, C35, C36, J1, J2

Commit message: up
Parts:
- removed C30: 1nF, Capacitor_SMD:C_0201_0603Metric_Pad0.64x0.40mm_HandSolder, symbol Device:C_Small
- removed IC1: STSPIN32G0A2, samacsys:QFN50P700X700X105-49N-D, symbol samacsys:STSPIN32G0A2
- removed L2: 74438335220, samacsys:74438335220, symbol samacsys:74438335220
- removed R46: 18k, Resistor_SMD:R_0201_0603Metric_Pad0.64x0.40mm_HandSolder, symbol Device:R_Small
- added IC6: STSPIN32G4TR, QFN50P900X900X100-65N-D, symbol samacsys2:STSPIN32G4TR
- added J7: ERM8-005-XX.X-X-DV-TR, ERM8-005-XX.X-X-DV-TR:SAMTEC_ERM8-005-XX.X-X-DV-TR, symbol ERM8:ERM8-005-XX.X-X-DV-TR
- added L4: 74438335150, 74438335150, symbol samacsys2:74438335150
Connections:
- net +3.3V: now also L4.1
- net GND: now also IC6.32 (PGND)
- net HSU: now also IC6.43 (GHS1)
- net HSV: now also IC6.40 (GHS2)
- net HSW: now also IC6.37 (GHS3)
- net LSU: now also IC6.29 (GLS1)
- net LSV: now also IC6.30 (GLS2)
- net LSW: now also IC6.31 (GLS3)
- net OUTU: now also IC6.42 (OUT1)
- net OUTV: now also IC6.39 (OUT2)
- net OUTW: now also IC6.36 (OUT3)
- net SW: now also L4.2
- net at C3.1: now also IC6.38 (BOOT2)
- net at C4.1: now also IC6.35 (BOOT3)
- net at C2.1: now also IC6.41 (BOOT1)
- no-connect marks 1 -> 2
Other:
- moved on the sheet: C1, C10, C11, C12, C2, C3, C4, C5, C6, C7, C9, D1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
