File: HARDWARE/ELECTRONIQUE/FOC_CONTROLLER_V2/hall.kicad_sch (KiCad schematic)
At the start: 4 parts, among them IC1 MA330GQ-Z

Commit message: up
Parts:
- renumbered C10 to C25, IC1 to IC2, R37 to R7, R40 to R8
