File: HARDWARE/ELECTRONIQUE/PCB_BRUSHED/CONN.kicad_sch (KiCad schematic)
At the start: 4 parts, among them J1 ERM8-005-XX.X-X-DV-TR, J2 SM06B-GHS-TB_LF__SN_, J3 ERM8-005-XX.X-X-DV-TR, J4 ERM8-005-XX.X-X-DV-TR

Commit message: update
Parts:
- added C34: 100n, Capacitor_SMD:C_0201_0603Metric_Pad0.64x0.40mm_HandSolder, symbol Device:C_Small
- added R21: 1k, Resistor_SMD:R_0201_0603Metric_Pad0.64x0.40mm_HandSolder, symbol Device:R_Small
- renumbered J1 to J5, J2 to J6, J3 to J7, J4 to J8
Connections:
- net BTN: now also C34.1, R21.2
- net GND: now also J5.01, J5.02, J7.01, J7.02, J8.01, J8.02, C34.2, R21.1
- net VBAT+: now reaches J8.09
- net VBAT+: now also J5.09, J5.10, J7.09, J7.10, J8.10
- net EXTI_EXT: now reaches J5.03
- net EXTI_EXT: now also J5.04
- net UART_TX: now reaches J5.05
- net UART_TX: now also J5.06
- net UART_RX: now reaches J5.07
- net UART_RX: now also J5.08
- no-connect marks 0 -> 12
