File: HARDWARE/ELECTRONIQUE/PCB_BRUSHED/MOTOR1.kicad_sch (KiCad schematic)
At the start: 7 parts, among them IC2 DRV8871DDAR

Commit message: update
Parts:
- added J1: SM06B-GHS-TB_LF__SN_, samacsys:SM06B-GHS-TB, symbol samacsys:SM06B-GHS-TB_LF__SN_
- added J2: S6B-PH-SM4-TB_LF__SN_, samacsys2:S6B-PH-SM4-TB_LF__SN__3, symbol samacsys2:S6B-PH-SM4-TB_LF__SN_
- added R11, R15: 22R, Resistor_SMD:R_0201_0603Metric_Pad0.64x0.40mm_HandSolder, symbol Device:R_Small
- renumbered C27 to C28, C28 to C29, C29 to C30, R8 to R12, R9 to R13, R10 to R14
Connections:
- net GND: now also J1.1, J1.7, J1.8, J2.2
- net MOT1: now reaches IC2.6 (OUT1)
- net MOT1: now also J2.1
- net MOT2: now reaches IC2.8 (OUT2)
- net MOT2: now also J2.6
- new net: J1.5, R15.1
- new net: J1.3, R11.2
- new net +3.3V: J1.6, J2.5
- new net ENCODERA: J2.3
- new net ENCODERB: J2.4
- new net SPI_CLK: R11.1
- new net SPI_CS: J1.2
- new net SPI_MISO: J1.4
- new net SPI_MOSI: R15.2

Commit message: up
Parts:
- added C12: 22u, Capacitor_SMD:C_0805_2012Metric, symbol Device:C_Small
Connections:
- net GND: now also C12.2
- net VBAT+: now also C12.1
Changed lines of the file:
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@@
+	)
+	(junction
+		(at 167.64 60.96)
+		(diameter 0)
+		(color 0 0 0 0)
 	)
 	(junction
@@
 		(color 0 0 0 0)
 	)
+	(junction
+		(at 167.64 66.04)
+		(diameter 0)
+		(color 0 0 0 0)
+	)
 	(wire
 		(pts
@@
 	(wire
 		(pts
+			(xy 167.64 60.96) (xy 176.53 60.96)
+		)
+		(stroke
+			(width 0)
+			(type default)
+		)
+	)
+	(wire
+		(pts
 			(xy 144.78 54.61) (xy 144.78 60.96)
 		)
@@
 		(pts
 			(xy 76.2 158.75) (xy 90.17 158.75)
+		)
+		(stroke
+			(width 0)
+			(type default)
+		)
+	)
+	(wire
+		(pts
+			(xy 167.64 66.04) (xy 176.53 66.04)
 		)
 		(stroke
@@
 					(unit 1)
 				)
+			)
+		)
+	)
+	(symbol
+		(lib_id "Device:C_Small")
+		(at 176.53 63.5 0)
+		(unit 1)
+		(exclude_from_sim no)
+		(in_bom yes)
+		(on_board yes)
+		(dnp no)
+		(property "Reference" "C12"
+			(at 179.07 62.2362 0)
+			(effects
+				(font
+					(size 1.27 1.27)
+				)
+				(justify left)
+			)
+		)
+		(property "Value" "22u"
+			(at 179.07 64.7762 0)
+			(effects
+				(font
+					(size 1.27 1.27)
+				)
+				(justify left)
+			)
+		)
+		(property "Footprint" "Capacitor_SMD:C_0805_2012Metric"
+			(at 176.53 63.5 0)
+			(effects
+				(font
+					(size 1.27 1.27)
+				)
+				(hide yes)
+			)
+		)
+		(property "Datasheet" "~"
+			(at 176.53 63.5 0)
+			(effects
+				(font
+					(size 1.27 1.27)
+				)
+				(hide yes)
+			)
+		)
+		(property "Description" "GRM21BR61A476ME15"
+			(at 187.96 69.088 0)
+			(effects
+				(font
+					(size 1.27 1.27)
+				)
+				(hide yes)
+			)
+		)
+		(property "Manufacturer_Part_Number" "GRM21BR61E226ME4L"
+			(at 176.53 63.5 0)
+			(effects
+				(font
+					(size 1.27 1.27)
+				)
+				(hide yes)
+			)
+		)
+		(property "Mouser Part Number" "81-GRM21BR61E226ME4L"
+			(at 176.53 63.5 0)
+			(effects
+				(font
+					(size 1.27 1.27)
+				)
+				(hide yes)
+			)
+		)
+		(pin "1"
+		)
+		(pin "2"
+		)
+		(instances
+			(project "PCB_BRUSHED"
+				(path "/21624bb8-7220-4725-ab4f-34c4768aac8d/36b31599-fc9c-43df-a06c-d0549a8044da"
+					(reference "C13")
+					(unit 1)
+				)
+				(path "/21624bb8-7220-4725-ab4f-34c4768aac8d/572c8ccb-40d1-41ab-95fe-e81a18cac254"
+					(reference "C14")
+					(unit 1)
+				)
+				(path "/21624bb8-7220-4725-ab4f-34c4768aac8d/77eb2796-38d1-43a1-af17-d64a90a7dfbd"
+					(reference "C12")
+					(unit 1)
+				)

Commit message: up brushed
Connections:
- net GND: now also J2.7, J2.8
Changed lines of the file:
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@@
 		(pin "6"
+		)
+		(pin "7"
+		)
+		(pin "8"
 		)
 		(instances
@@
 					(unit 1)
 				)
+			)
+		)
+	)
+	(symbol
+		(lib_id "power:GND")
+		(at 162.56 115.57 0)
+		(unit 1)
+		(exclude_from_sim no)
+		(in_bom yes)
+		(on_board yes)
+		(dnp no)
+		(property "Reference" "#PWR016"
+			(at 162.56 121.92 0)
+			(effects
+				(font
+					(size 1.27 1.27)
+				)
+				(hide yes)
+			)
+		)
+		(property "Value" "GND"
+			(at 162.56 119.634 0)
+			(effects
+				(font
+					(size 1.27 1.27)
+				)
+			)
+		)
+		(property "Footprint" ""
+			(at 162.56 115.57 0)
+			(effects
+				(font
+					(size 1.27 1.27)
+				)
+				(hide yes)
+			)
+		)
+		(property "Datasheet" ""
+			(at 162.56 115.57 0)
+			(effects
+				(font
+					(size 1.27 1.27)
+				)
+				(hide yes)
+			)
+		)
+		(property "Description" "Power symbol creates a global label with name \"GND\" , ground"
+			(at 162.56 115.57 0)
+			(effects
+				(font
+					(size 1.27 1.27)
+				)
+				(hide yes)
+			)
+		)
+		(pin "1"
+		)
+		(instances
+			(project "PCB_BRUSHED"
+				(path "/21624bb8-7220-4725-ab4f-34c4768aac8d/36b31599-fc9c-43df-a06c-d0549a8044da"
+					(reference "#PWR017")
+					(unit 1)
+				)
+				(path "/21624bb8-7220-4725-ab4f-34c4768aac8d/572c8ccb-40d1-41ab-95fe-e81a18cac254"
+					(reference "#PWR054")
+					(unit 1)
+				)
+				(path "/21624bb8-7220-4725-ab4f-34c4768aac8d/77eb2796-38d1-43a1-af17-d64a90a7dfbd"
+					(reference "#PWR016")
+					(unit 1)
+				)
