File: HARDWARE/ELECTRONIQUE/PCB_BRUSHED/PCB_BRUSHED.kicad_pcb (KiCad board)
At the start: 8 copper layers, 50 x 43.3 mm, 297 parts, among them IC1 STSPIN32G4TR, IC2 MA330GQ-Z, IC3 STSPIN32G4TR, IC4 MA330GQ-Z, IC5 STSPIN32G4TR, IC6 MA330GQ-Z, J1 SM06B-GHS-TB_LF__SN_, J2 ERM8-005-XX.X-X-DV-TR, J3 SM06B-GHS-TB_LF__SN_, J4 SM06B-GHS-TB_LF__SN_, J5 ERM8-005-XX.X-X-DV-TR, J6 SM06B-GHS-TB_LF__SN_, J7 SM06B-GHS-TB_LF__SN_, J8 ERM8-005-XX.X-X-DV-TR, J9 SM06B-GHS-TB_LF__SN_, Q1 DMT6018LDR-7, Q2 DMT6018LDR-7, Q3 DMT6018LDR-7, Q4 DMT6018LDR-7, Q5 DMT6018LDR-7, Q6 DMT6018LDR-7, Q7 DMT6018LDR-7, Q8 DMT6018LDR-7, Q9 DMT6018LDR-7

Commit message: update
Parts:
- removed C100, C59, C63, C66, C93, C97: DNP, Capacitor_SMD:C_0201_0603Metric_Pad0.64x0.40mm_HandSolder
- removed C101, C53, C54, C55, C60, C64, C67, C87, C88, C89, C94, C98: 1u, Capacitor_SMD:C_0603_1608Metric
- removed C102, C61, C65, C68, C95, C99: 470p, Capacitor_SMD:C_0201_0603Metric_Pad0.64x0.40mm_HandSolder
- removed C38, C39, C40, C41, C42, C43, C44, C69, C70, C71, C72, C73, C74, C75, C76, C77, C78: 22u, Capacitor_SMD:C_0805_2012Metric
- removed C45, C47, C49, C52, C56, C57, C79, C81, C83, C86, C90, C91: 100n, Capacitor_SMD:C_0201_0603Metric_Pad0.64x0.40mm_HandSolder
- removed C46, C80: 47u, Capacitor_SMD:C_0805_2012Metric
- removed C48, C82: 10u, Capacitor_SMD:C_0603_1608Metric
- removed C50, C84: 220n, Capacitor_SMD:C_0603_1608Metric
- removed C51, C85: 4.7u, Capacitor_SMD:C_0402_1005Metric
- removed C58, C92: 10n, Capacitor_SMD:C_0201_0603Metric_Pad0.64x0.40mm_HandSolder
- removed C62, C96: 1u, Capacitor_SMD:C_0402_1005Metric
- removed D10, D18, D2: STPS0560Z, samacsys:STPS0560Z
- removed D11, D12, D13, D14, D15, D16, D19, D20, D21, D22, D23, D24, D3, D4, D5, D6, D7, D8: BAS16LP-7B, Diode_SMD:D_01005_0402Metric_Pad0.57x0.30mm_HandSolder
- removed D17, D9: LED, LED_SMD:LED_0402_1005Metric
- removed IC5: STSPIN32G4TR, samacsys2:QFN50P900X900X100-65N-D
- removed IC6: MA330GQ-Z, samacsys:QFN50P300X300X100-17N-D
- removed L1, L2, L3: 74438335150, samacsys2:74438335150
- removed Q1, Q2, Q3, Q4, Q5, Q6, Q7, Q8, Q9: DMT6018LDR-7, samacsys:DMT6018LDR7
- removed R100, R101, R114, R115, R126, R127, R27, R38, R39, R46, R56, R57, R70, R71, R82, R83, R90: 0R, Resistor_SMD:R_0201_0603Metric_Pad0.64x0.40mm_HandSolder
- removed R102, R109, R116, R121, R128, R28, R33, R40, R45, R51, R58, R65, R72, R77, R84, R89, R95: 1k, Resistor_SMD:R_0201_0603Metric_Pad0.64x0.40mm_HandSolder
- removed R103, R117, R129, R29, R41, R59, R73, R85: 7.5k, Resistor_SMD:R_0201_0603Metric_Pad0.64x0.40mm_HandSolder
- removed R104, R118, R130, R30, R42, R60, R74, R86: R_Shunt, samacsys:4wire_0603
- removed R105, R119, R131, R31, R43, R61, R75, R87: 220R, Resistor_SMD:R_0201_0603Metric_Pad0.64x0.40mm_HandSolder
- removed R106, R120, R132, R32, R44, R62, R76, R88: 2.2k, Resistor_SMD:R_0201_0603Metric_Pad0.64x0.40mm_HandSolder
- removed R107, R47, R50, R63, R91, R94: 10k, Resistor_SMD:R_0201_0603Metric_Pad0.64x0.40mm_HandSolder
- removed R108, R64: 100R, Resistor_SMD:R_0201_0603Metric_Pad0.64x0.40mm_HandSolder
- removed R110, R111, R122, R123, R34, R35, R48, R52, R53, R66, R67, R78, R79, R92, R96, R97: 15k, Resistor_SMD:R_0201_0603Metric_Pad0.64x0.40mm_HandSolder
- removed R112, R113, R124, R125, R36, R37, R54, R55, R68, R69, R80, R81, R98, R99: 120R, Resistor_SMD:R_0201_0603Metric_Pad0.64x0.40mm_HandSolder
- removed R49, R93: 100k, Resistor_SMD:R_0201_0603Metric_Pad0.64x0.40mm_HandSolder
- removed TP10, TP11, TP12, TP4, TP5, TP6, TP7, TP8, TP9: TestPoint, samacsys:hole_1.5mm
- added J10: S6B-PH-SM4-TB_LF__SN_, samacsys2:S6B-PH-SM4-TB_LF__SN__3, B.Cu at (118.0, 103.0)
- added LEDRED1: 150040RS73240, LED_SMD:LED_0402_1005Metric, F.Cu at (191.8, 86.5)
- added U1: STM32G431CBUx, Package_DFN_QFN:QFN-48-1EP_7x7mm_P0.5mm_EP5.6x5.6mm, F.Cu at (130.0, 96.0)
- added Y1: 830069528, samacsys:830069528, F.Cu at (199.5, 87.6)
- C1, C2: value 22u -> 10u; footprint Capacitor_SMD:C_0805_2012Metric -> Capacitor_SMD:C_0603_1608Metric
- C10, C35: value 22u -> 1u; footprint Capacitor_SMD:C_0805_2012Metric -> Capacitor_SMD:C_0402_1005Metric_Pad0.74x0.62mm_HandSolder
- C12: value 47u -> 22u
- C13, C15, C22: value 100n -> 22u; footprint Capacitor_SMD:C_0201_0603Metric_Pad0.64x0.40mm_HandSolder -> Capacitor_SMD:C_0805_2012Metric
- C14: value 10u -> 22u; footprint Capacitor_SMD:C_0603_1608Metric -> Capacitor_SMD:C_0805_2012Metric
- C16: value 220n -> 4.7u; footprint Capacitor_SMD:C_0603_1608Metric -> Capacitor_SMD:C_0402_1005Metric_Pad0.74x0.62mm_HandSolder
- C17: value 4.7u -> 100n; footprint Capacitor_SMD:C_0402_1005Metric -> Capacitor_SMD:C_0201_0603Metric_Pad0.64x0.40mm_HandSolder
- C19, C20, C27, C30, C33: value 1u -> 22u; footprint Capacitor_SMD:C_0603_1608Metric -> Capacitor_SMD:C_0805_2012Metric
- C21: value 1u -> 100n; footprint Capacitor_SMD:C_0603_1608Metric -> Capacitor_SMD:C_0201_0603Metric_Pad0.64x0.40mm_HandSolder
- C24: value 10n -> 22u; footprint Capacitor_SMD:C_0201_0603Metric_Pad0.64x0.40mm_HandSolder -> Capacitor_SMD:C_0805_2012Metric
- C25: value 1u -> 10n; footprint Capacitor_SMD:C_0402_1005Metric -> Capacitor_SMD:C_0201_0603Metric_Pad0.64x0.40mm_HandSolder
- C26: value DNP -> 1u; footprint Capacitor_SMD:C_0201_0603Metric_Pad0.64x0.40mm_HandSolder -> Capacitor_SMD:C_0402_1005Metric_Pad0.74x0.62mm_HandSolder
- C28, C31: value 470p -> 1u; footprint Capacitor_SMD:C_0201_0603Metric_Pad0.64x0.40mm_HandSolder -> Capacitor_SMD:C_0402_1005Metric_Pad0.74x0.62mm_HandSolder
- C29, C32: value DNP -> 22u; footprint Capacitor_SMD:C_0201_0603Metric_Pad0.64x0.40mm_HandSolder -> Capacitor_SMD:C_0805_2012Metric
- C3: value 22u -> 430pF; footprint Capacitor_SMD:C_0805_2012Metric -> Capacitor_SMD:C_0201_0603Metric_Pad0.64x0.40mm_HandSolder
- C34: value 470p -> 100n
- C4, C7, C8, C9: value 22u -> 100n; footprint Capacitor_SMD:C_0805_2012Metric -> Capacitor_SMD:C_0201_0603Metric_Pad0.64x0.40mm_HandSolder
- C5, C6: footprint Capacitor_SMD:C_0805_2012Metric -> Capacitor_SMD:C_0603_1608Metric
- IC1: value STSPIN32G4TR -> TPS82150SILR; footprint samacsys2:QFN50P900X900X100-65N-D -> samacsys2:TPS82130SILT; moved to B.Cu
- IC2, IC4: value MA330GQ-Z -> DRV8871DDAR; footprint samacsys:QFN50P300X300X100-17N-D -> samacsys2:SOIC127P600X170-9N; moved to B.Cu
- IC3: value STSPIN32G4TR -> DRV8871DDAR; footprint samacsys2:QFN50P900X900X100-65N-D -> samacsys2:SOIC127P600X170-9N; moved to B.Cu
- J2: value ERM8-005-XX.X-X-DV-TR -> S6B-PH-SM4-TB_LF__SN_; footprint ERM8:SAMTEC_ERM8-005-XX.X-X-DV-TR -> samacsys2:S6B-PH-SM4-TB_LF__SN__3; moved to B.Cu
- J4: value SM06B-GHS-TB_LF__SN_ -> S6B-PH-SM4-TB_LF__SN_; footprint samacsys:SM06B-GHS-TB -> samacsys2:S6B-PH-SM4-TB_LF__SN__3; moved to B.Cu
- J6: moved to B.Cu
- J7: value SM06B-GHS-TB_LF__SN_ -> ERM8-005-XX.X-X-DV-TR; footprint samacsys:SM06B-GHS-TB -> ERM8:SAMTEC_ERM8-005-XX.X-X-DV-TR
- R1: value 1k -> 15k
- R10, R11, R22, R23: value 15k -> 22R
- R12, R13, R24: value 120R -> 22R
- R14: value 0R -> 32k
- R15, R26: value 0R -> 22R
- R16: value 1k -> 22R
- R17: value 7.5k -> 22R
- R18: value R_Shunt -> 22R; footprint samacsys:4wire_0603 -> Resistor_SMD:R_0201_0603Metric_Pad0.64x0.40mm_HandSolder
- R19: value 220R -> 32k
- R2: value 0R -> 100k
- R20: value 2.2k -> 22R
- R25: value 120R -> 32k
- R3: value 10k -> 100k
- R4: value 15k -> 309k
- R6, R7: value 10k -> 1k
- R8: value 100R -> 10k
- TP1, TP2, TP3: footprint samacsys:m3test -> MountingHole:MountingHole_2.5mm_Pad_Via
- moved C36 210.2 mm to (236.3, 92.4)
- moved C37 210.2 mm to (236.3, 95.4)
- moved C35 209.9 mm to (235.7, 97.9)
- moved C29 177.9 mm to (236.3, 113.8)
- moved C22 177.7 mm to (236.7, 73.9)
- moved C30 176.9 mm to (236.3, 116.8)
- moved C24 174.8 mm to (236.7, 76.9)
- moved C15 173.2 mm to (232.3, 73.9)
- moved R22 170.2 mm to (229.3, 102.4)
- moved R23 170.2 mm to (229.3, 104.1)
- moved C13 168.7 mm to (227.8, 76.9)
- moved R24 167.6 mm to (229.3, 105.9)
- moved R25 167.6 mm to (229.3, 107.6)
- moved R26 167.6 mm to (229.3, 109.4)
- moved C12 163.6 mm to (227.8, 73.9)
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Connections:
- C10 pad 1: VBAT+ -> GND
- C10 pad 2: GND -> +3.3V
- C11 pad 1: +3.3V -> GND
- C11 pad 2: GND -> +3.3V
- C12 pad 1: +3.3V -> VBAT+
- C13 pad 1: /MOTEUR1/NRST -> VBAT+
- C14 pad 1: GND -> VBAT+
- C14 pad 2: /MOTEUR1/REG12 -> GND
- C15 pad 1: /MOTEUR1/REG12 -> VBAT+
- C16 pad 1: GND -> +3.3V
- C16 pad 2: VBAT+ -> GND
- C17 pad 1: +3.3V -> GND
- C17 pad 2: GND -> Net-(Y1-CRYSTAL_2)
- C18 pad 1: +3.3V -> GND
- C18 pad 2: GND -> +3.3V
- C19 pad 1: Net-(IC1-BOOT1) -> VBAT+
- C19 pad 2: /MOTEUR1/OUTU -> GND
- C20 pad 1: Net-(IC1-BOOT2) -> VBAT+
- C20 pad 2: /MOTEUR1/OUTV -> GND
- C21 pad 1: Net-(IC1-BOOT3) -> GND
- C21 pad 2: /MOTEUR1/OUTW -> +3.3V
- C22 pad 1: /MOTEUR1/BTN -> VBAT+
- C23 pad 1: Net-(C23-Pad1) -> GND
- C23 pad 2: GND -> +3.3V
- C24 pad 1: Net-(C24-Pad1) -> VBAT+
- C25 pad 1: +3.3V -> GND
- C25 pad 2: GND -> +3.3V
- C26 pad 1: /MOTEUR1/OP1N -> GND
- C26 pad 2: /MOTEUR1/OP1O -> +3.3V
- C27 pad 1: GND -> VBAT+
- C27 pad 2: VBAT+ -> GND
- C28 pad 2: /MOTEUR1/ISNSW -> VBAT+
- C29 pad 1: /MOTEUR1/OP2N -> VBAT+
- C29 pad 2: /MOTEUR1/OP2O -> GND
- C3 pad 1: VBAT+ -> Net-(IC1-SS/TR)
- C30 pad 1: GND -> VBAT+
- C30 pad 2: VBAT+ -> GND
- C31 pad 2: /MOTEUR1/ISNSU -> VBAT+
- C32 pad 1: /MOTEUR1/OP3N -> VBAT+
- C32 pad 2: /MOTEUR1/OP3O -> GND
- C33 pad 1: GND -> VBAT+
- C33 pad 2: VBAT+ -> GND
- C34 pad 1: GND -> /EXT_BTN_EXTI10
- C34 pad 2: /MOTEUR1/ISNSV -> GND
- C35 pad 1: VBAT+ -> GND
- C35 pad 2: GND -> VBAT+
- C4 pad 1: VBAT+ -> /ADC2_IN5
- C5 pad 1: VBAT+ -> +3.3V
- C6 pad 1: VBAT+ -> +3.3V
- C7 pad 1: VBAT+ -> /NRST
- C8 pad 1: VBAT+ -> /ADC_VBAT
- C9 pad 1: VBAT+ -> GND
- C9 pad 2: GND -> /HSE_IN
- D1 pad 2: unconnected-(D1-A-Pad2) -> Net-(D1-A)
- IC1 pad 1: unconnected-(IC1-REG3V3/VDD-Pad1) -> VBAT+
- IC1 pad 2: unconnected-(IC1-VBAT-Pad2) -> VBAT+
- IC1 pad 3: unconnected-(IC1-PC13-Pad3) -> GND
- IC1 pad 4: unconnected-(IC1-PC14-Pad4) -> +3.3V
- IC1 pad 5: unconnected-(IC1-PC15-Pad5) -> +3.3V
- IC1 pad 6: unconnected-(IC1-PF0-Pad6) -> Net-(IC1-FB)
- IC1 pad 7: unconnected-(IC1-PF1-Pad7) -> Net-(IC1-PG)
- IC1 pad 8: unconnected-(IC1-PG10-Pad8) -> Net-(IC1-SS/TR)
- IC1 pad 9: unconnected-(IC1-PC0-Pad9) -> GND
- IC2 pad 1: unconnected-(IC2-V-Pad1) -> GND
- IC2 pad 2: unconnected-(IC2-A-Pad2) -> Net-(IC2-IN2)
- IC2 pad 3: unconnected-(IC2-Z-Pad3) -> Net-(IC2-IN1)
- IC2 pad 4: /MOTEUR1/SPI2_MOSI -> Net-(IC2-ILIM)
- IC2 pad 5: /MOTEUR1/SPI2_CS -> VBAT+
- IC2 pad 6: unconnected-(IC2-B-Pad6) -> /MOTOR2/MOT1
- IC2 pad 7: /MOTEUR1/SPI2_MISO -> GND
- IC2 pad 8: GND -> /MOTOR2/MOT2
- IC2 pad 9: unconnected-(IC2-W-Pad9) -> GND
- IC3 pad 1: unconnected-(IC3-REG3V3/VDD-Pad1) -> GND
- IC3 pad 2: unconnected-(IC3-VBAT-Pad2) -> Net-(IC3-IN2)
- IC3 pad 3: unconnected-(IC3-PC13-Pad3) -> Net-(IC3-IN1)
- IC3 pad 4: unconnected-(IC3-PC14-Pad4) -> Net-(IC3-ILIM)
- IC3 pad 5: unconnected-(IC3-PC15-Pad5) -> VBAT+
- IC3 pad 6: unconnected-(IC3-PF0-Pad6) -> /MOTOR1/MOT1
- IC3 pad 7: unconnected-(IC3-PF1-Pad7) -> GND
- IC3 pad 8: unconnected-(IC3-PG10-Pad8) -> /MOTOR1/MOT2
- IC3 pad 9: unconnected-(IC3-PC0-Pad9) -> GND
- IC4 pad 1: unconnected-(IC4-V-Pad1) -> GND
- IC4 pad 2: unconnected-(IC4-A-Pad2) -> Net-(IC4-IN2)
- IC4 pad 3: unconnected-(IC4-Z-Pad3) -> Net-(IC4-IN1)
- IC4 pad 4: /MOTEUR2/SPI2_MOSI -> Net-(IC4-ILIM)
- IC4 pad 5: /MOTEUR2/SPI2_CS -> VBAT+
- IC4 pad 6: unconnected-(IC4-B-Pad6) -> /MOTOR3/MOT1
- IC4 pad 7: /MOTEUR2/SPI2_MISO -> GND
- IC4 pad 8: GND -> /MOTOR3/MOT2
- IC4 pad 9: unconnected-(IC4-W-Pad9) -> GND
- J1 pad 1: VBAT+ -> GND
- J1 pad 2: VBAT+ -> /HALL2_CS
- J1 pad 3: /MOTEUR1/UART_RX -> Net-(J1-Pad3)
- J1 pad 4: /MOTEUR1/UART_TX -> /HALL2_MISO
- J1 pad 5: GND -> Net-(J1-Pad5)
- J1 pad 6: GND -> +3.3V
- J3 pad 1: /MOTEUR1/NRST -> GND
- J3 pad 2: /MOTEUR1/SWCLK -> /HALL1_CS
- J3 pad 3: /MOTEUR1/SWDIO -> Net-(J3-Pad3)
- J3 pad 4: +3.3V -> /HALL1_MISO
- J3 pad 5: GND -> Net-(J3-Pad5)
- J3 pad 6: /MOTEUR1/BTN -> +3.3V
- J4 pad 1: VBAT+ -> /MOTOR1/MOT1
- J4 pad 2: VBAT+ -> GND
- J4 pad 3: /MOTEUR2/UART_RX -> /MOT1_HALL_A/TIM2CH1
- J4 pad 4: /MOTEUR2/UART_TX -> /MOT1_HALL_B/TIM2CH2
- J4 pad 5: GND -> +3.3V
- J4 pad 6: GND -> /MOTOR1/MOT2
- J4 pad 7: GND -> (no net)
- J4 pad 8: GND -> (no net)
- J5 pad 01: unconnected-(J5-Pad01) -> GND
- J5 pad 02: unconnected-(J5-Pad02) -> GND
- J5 pad 03: unconnected-(J5-Pad03) -> /UART_EXTI
- J5 pad 04: unconnected-(J5-Pad04) -> /UART_EXTI
- J5 pad 05: unconnected-(J5-Pad05) -> /USART3_TX
- J5 pad 06: unconnected-(J5-Pad06) -> /USART3_TX
- J5 pad 07: unconnected-(J5-Pad07) -> /USART3_RX
- J5 pad 08: unconnected-(J5-Pad08) -> /USART3_RX
- J5 pad 09: unconnected-(J5-Pad09) -> VBAT+
- J5 pad 10: unconnected-(J5-Pad10) -> VBAT+
- J6 pad 1: /MOTEUR2/NRST -> /NRST
- J6 pad 2: /MOTEUR2/SWCLK -> /SWCLK
- J6 pad 3: /MOTEUR2/SWDIO -> /SWDIO
- J6 pad 6: /MOTEUR2/BTN -> /EXT_BTN_EXTI10
- J8 pad 01: unconnected-(J8-Pad01) -> GND
- J8 pad 02: unconnected-(J8-Pad02) -> GND
- J8 pad 09: unconnected-(J8-Pad09) -> VBAT+
- J8 pad 10: unconnected-(J8-Pad10) -> VBAT+
- J9 pad 1: /MOTEUR3/NRST -> GND
- J9 pad 2: /MOTEUR3/SWCLK -> /HALL3_CS
- J9 pad 3: /MOTEUR3/SWDIO -> Net-(J9-Pad3)
- J9 pad 4: +3.3V -> /HALL3_MISO
- J9 pad 5: GND -> Net-(J9-Pad5)
- J9 pad 6: /MOTEUR3/BTN -> +3.3V
- R1 pad 1: GND -> /ADC2_IN5
- R1 pad 2: Net-(D1-K) -> GND
- R10 pad 1: +3.3V -> Net-(Y1-CRYSTAL_2)
- R10 pad 2: /MOTEUR1/OP1P -> /HSE_OUT
- R11 pad 1: /MOTEUR1/OP1P -> /HALL2_CLK
- R11 pad 2: GND -> Net-(J1-Pad3)
- R12 pad 1: /MOTEUR1/HSU -> /MOT2_PWMA/TIM4CH1
- R12 pad 2: Net-(Q1-G1) -> Net-(IC2-IN2)
- R13 pad 1: /MOTEUR1/LSU -> /MOT2_PWMB/TIM4CH2
- R13 pad 2: Net-(Q1-G2) -> Net-(IC2-IN1)
- R14 pad 1: Net-(D3-A) -> Net-(IC2-ILIM)
- R14 pad 2: Net-(Q1-G1) -> GND
- R15 pad 1: Net-(D4-A) -> Net-(J1-Pad5)
- R15 pad 2: Net-(Q1-G2) -> /HALL2_MOSI
- R16 pad 1: /MOTEUR1/U/SHUNT- -> /HALL1_CLK
- R16 pad 2: /MOTEUR1/OP1N -> Net-(J3-Pad3)
- R17 pad 1: /MOTEUR1/OP1N -> /MOT1_PWMA/TIM3CH3
- R17 pad 2: /MOTEUR1/OP1O -> Net-(IC3-IN2)
- R18 pad 1: Net-(Q1-S2) -> /MOT1_PWMB/TIM3CH4
- R18 pad 2: /MOTEUR1/U/SHUNT+ -> Net-(IC3-IN1)
- R19 pad 1: /MOTEUR1/OP1O -> Net-(IC3-ILIM)
- R19 pad 2: /MOTEUR1/ISNSW -> GND
- R2 pad 1: unconnected-(R2-Pad1) -> +3.3V
- R2 pad 2: /MOTEUR1/NRST -> /ADC2_IN5
- R20 pad 1: /MOTEUR1/U/SHUNT+ -> Net-(J3-Pad5)
- R20 pad 2: /MOTEUR1/SHUNT+AFTER -> /HALL1_MOSI
- R21 pad 1: /MOTEUR1/V/SHUNT+ -> GND
- R21 pad 2: /MOTEUR1/OP2P -> /EXT_BTN_EXTI10
- R22 pad 1: +3.3V -> /HALL3_CLK
- R22 pad 2: /MOTEUR1/OP2P -> Net-(J9-Pad3)
- R23 pad 1: /MOTEUR1/OP2P -> /MOT3_PWMA/TIM3CH1
- R23 pad 2: GND -> Net-(IC4-IN2)
- R24 pad 1: /MOTEUR1/HSV -> /MOT3_PWMB/TIM3CH2
- R24 pad 2: Net-(Q2-G1) -> Net-(IC4-IN1)
- R25 pad 1: /MOTEUR1/LSV -> Net-(IC4-ILIM)
- R25 pad 2: Net-(Q2-G2) -> GND
- R26 pad 1: Net-(D5-A) -> Net-(J9-Pad5)
- R26 pad 2: Net-(Q2-G1) -> /HALL3_MOSI
- R3 pad 2: /MOTEUR1/BTN -> Net-(IC1-PG)
- R4 pad 1: Net-(C23-Pad1) -> +3.3V
- R4 pad 2: GND -> Net-(IC1-FB)
- R5 pad 1: +3.3V -> Net-(IC1-FB)
- R5 pad 2: Net-(C23-Pad1) -> GND
- R6 pad 2: Net-(C24-Pad1) -> Net-(LEDRED1-A)
- R7 pad 1: /MOTEUR1/SPI2_CS -> /ADC_VBAT
- R7 pad 2: +3.3V -> GND
- R8 pad 1: /MOTEUR1/SPI2_SCK -> VBAT+
- R8 pad 2: Net-(IC2-SCLK) -> /ADC_VBAT
- R9 pad 1: /MOTEUR1/U/SHUNT+ -> GND
- R9 pad 2: /MOTEUR1/OP1P -> Net-(D1-K)
Other:
- copper layers 8 -> 6

Commit message: up
Parts:
- removed C15, C19, C20, C22, C24, C27: 22u, Capacitor_SMD:C_0805_2012Metric
- C1, C10, C11, C16, C18, C2, C21, C23, C25, C26, C28, C3, C31, C35, C4, C5, C6, C7, R1, R14, R19, R2, R25, R3, R4, R5: moved to B.Cu
- moved C37 114.4 mm to (122.0, 91.4), turned to 60 degrees
- moved C36 112.6 mm to (123.7, 92.4), turned to 60 degrees
- moved R15 112.5 mm to (128.0, 81.8), turned to -90 degrees
- moved C35 111.8 mm to (124.0, 93.2), turned to -120 degrees
- moved R22 111.4 mm to (118.0, 103.0), turned to -150 degrees
- moved R26 110.5 mm to (118.9, 104.7), turned to 30 degrees
- moved C13 108.4 mm to (120.2, 90.4), turned to 60 degrees
- moved R11 107.9 mm to (130.0, 81.7), turned to 90 degrees
- moved R13 106.4 mm to (129.6, 90.0), turned to 150 degrees
- moved R12 105.7 mm to (130.0, 89.3), turned to 150 degrees
- moved R25 105.2 mm to (125.5, 90.3), turned to -120 degrees
- moved C28 103.8 mm to (135.5, 92.2), turned to 120 degrees
- moved C12 103.4 mm to (130.0, 107.3), turned to 180 degrees
- moved C29 102.3 mm to (136.3, 92.3), turned to -60 degrees
- moved C30 101.6 mm to (138.0, 91.3), turned to -60 degrees
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Routing:
- net /HALL3_CS: track 0.00 -> 18.0 mm
- net /HALL3_MISO: track 0.00 -> 16.7 mm
- net /HALL2_MISO: track 0.00 -> 15.9 mm
- net /HALL2_CS: track 0.00 -> 15.9 mm
- net /HALL1_CS: track 0.00 -> 15.6 mm
- net /HALL1_MISO: track 0.00 -> 14.0 mm
- net /HALL3_CLK: track 0.00 -> 13.9 mm
- net /HALL3_MOSI: track 0.00 -> 13.4 mm
- net /HALL2_CLK: track 0.00 -> 13.2 mm
- net /HALL2_MOSI: track 0.00 -> 13.1 mm
- net /HALL1_MOSI: track 0.00 -> 11.2 mm
- net /HALL1_CLK: track 0.00 -> 10.6 mm
- net +3.3V: track 0.00 -> 7.85 mm, vias 0 -> 4
- net /ADC2_IN5: track 0.00 -> 6.45 mm, vias 0 -> 1
- net /HSE_IN: track 0.00 -> 5.97 mm
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- added copper zone on B.Cu, net /MOTOR1/MOT1
- added copper zone on B.Cu, net /MOTOR1/MOT2
- added copper zone on B.Cu, net /MOTOR2/MOT1
- added copper zone on B.Cu, net /MOTOR2/MOT2
- added copper zone on B.Cu, net /MOTOR3/MOT1
- added copper zone on B.Cu, net /MOTOR3/MOT2

Commit message: up brushed
Parts:
- moved J6 5.39 mm to (146.4, 86.5)
- moved R5 1.23 mm to (131.3, 115.7), turned to 0 degrees
- moved R4 0.86 mm to (131.4, 115.0), turned to 180 degrees
Connections:
- J10 pad 7: (no net) -> GND
- J10 pad 8: (no net) -> GND
- J2 pad 7: (no net) -> GND
- J2 pad 8: (no net) -> GND
- J4 pad 7: (no net) -> GND
- J4 pad 8: (no net) -> GND
Routing:
- net /UART_EXTI: track 5.93 -> 33.5 mm, vias 2 -> 3
- net /SWCLK: track 1.41 -> 27.1 mm, vias 1 -> 2
- net /USART3_TX: track 5.72 -> 29.0 mm, vias 2 -> 3
- net /EXT_BTN_EXTI10: track 1.00 -> 24.2 mm, vias 1 -> 2
- net Net-(IC4-IN1): track 0.00 -> 22.5 mm, vias 1 -> 2
- net /SWDIO: track 0.86 -> 22.9 mm, vias 1 -> 2
- net /NRST: track 1.03 -> 22.2 mm, vias 1 -> 2
- net /USART3_RX: track 5.53 -> 25.6 mm, vias 2 -> 3
- net /ADC_VBAT: track 2.75 -> 17.4 mm, vias 1 -> 2
- net /MOT1_HALL_A/TIM2CH1: track 1.08 -> 15.5 mm
- net /MOT2_HALL_A/TIM1CH1: track 0.79 -> 15.2 mm
- net Net-(IC2-IN2): track 0.00 -> 13.6 mm, vias 0 -> 2
- net Net-(IC3-IN2): track 0.00 -> 13.3 mm, vias 0 -> 2
- net /MOT3_HALL_A/TIM8CH1: track 0.40 -> 13.6 mm
- net Net-(IC3-IN1): track 0.00 -> 12.9 mm, vias 0 -> 2
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- added copper zone on B.Cu, net +3.3V
- added copper zone on F.Cu, net +3.3V
- added copper zone on In3.Cu, net +3.3V
- added copper zone on B.Cu, net GND
- added copper zone on F.Cu, net GND
- added copper zone on In1.Cu, net GND
- added copper zone on In4.Cu, net GND
- added copper zone on B.Cu, net VBAT+
- added copper zone on F.Cu, net VBAT+

Commit message: update
Parts:
- added G***: LOGO, LOGO, F.Cu at (139.8, 97.2)
- added REF**: BreakLine_5h_D0.5mm_P0.85mm, Panelization:BreakLine_5h_D0.5mm_P0.85mm, F.Cu at (136.8, 118.0)
- added REF**: BreakLine_5h_D0.5mm_P0.85mm, Panelization:BreakLine_5h_D0.5mm_P0.85mm, F.Cu at (124.1, 118.0)
- added REF**: BreakLine_5h_D0.5mm_P0.85mm, Panelization:BreakLine_5h_D0.5mm_P0.85mm, F.Cu at (128.3, 74.0)
- added REF**: BreakLine_5h_D0.5mm_P0.85mm, Panelization:BreakLine_5h_D0.5mm_P0.85mm, F.Cu at (119.8, 74.0)
- added REF**: BreakLine_5h_D0.5mm_P0.85mm, Panelization:BreakLine_5h_D0.5mm_P0.85mm, F.Cu at (128.3, 118.0)
- added REF**: BreakLine_2h_D0.5mm_P0.85mm, Panelization:BreakLine_2h_D0.5mm_P0.85mm, F.Cu at (141.4, 74.0)
- added REF**: BreakLine_2h_D0.5mm_P0.85mm, Panelization:BreakLine_2h_D0.5mm_P0.85mm, F.Cu at (139.8, 118.0)
- added REF**: BreakLine_5h_D0.5mm_P0.85mm, Panelization:BreakLine_5h_D0.5mm_P0.85mm, F.Cu at (119.8, 118.0)
- added REF**: BreakLine_5h_D0.5mm_P0.85mm, Panelization:BreakLine_5h_D0.5mm_P0.85mm, F.Cu at (132.5, 74.0)
- added REF**: BreakLine_2h_D0.5mm_P0.85mm, Panelization:BreakLine_2h_D0.5mm_P0.85mm, F.Cu at (139.8, 74.0)
- added REF**: BreakLine_5h_D0.5mm_P0.85mm, Panelization:BreakLine_5h_D0.5mm_P0.85mm, F.Cu at (136.8, 74.0)
- added REF**: BreakLine_5h_D0.5mm_P0.85mm, Panelization:BreakLine_5h_D0.5mm_P0.85mm, F.Cu at (132.6, 118.0)
- added REF**: BreakLine_5h_D0.5mm_P0.85mm, Panelization:BreakLine_5h_D0.5mm_P0.85mm, F.Cu at (124.0, 74.0)
- added REF**: BreakLine_2h_D0.5mm_P0.85mm, Panelization:BreakLine_2h_D0.5mm_P0.85mm, F.Cu at (141.5, 118.0)
- C17, C9: value 100n -> 10p
Routing:
- net GND: vias 124 -> 348
Other:
- board size 50 x 43.3 mm -> 50 x 49.4 mm
- board text added: "HALL1"
- board text added: "HALL2"
- board text added: "HALL3"
- board text added: "L.ROMEO"
- board text added: "M.POMMERY"
- board text added: "MOTOR1"
- board text added: "MOTOR2"
- board text added: "MOTOR3"
