File: HARDWARE/ELECTRONIQUE/PCB_BRUSHED/PCB_BRUSHED.kicad_pcb (KiCad board)
At the start: 6 copper layers, 50 x 49.4 mm, 93 parts, among them IC1 TPS82150SILR, IC2 DRV8871DDAR, IC3 DRV8871DDAR, IC4 DRV8871DDAR, J1 SM06B-GHS-TB_LF__SN_, J10 S6B-PH-SM4-TB_LF__SN_, J2 S6B-PH-SM4-TB_LF__SN_, J3 SM06B-GHS-TB_LF__SN_, J4 S6B-PH-SM4-TB_LF__SN_, J5 ERM8-005-XX.X-X-DV-TR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

Commit message: up
Parts:
- C17, C9: value 10p -> 3p
Changed lines of the file:
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@@
 			)
 		)
-		(property "Value" "10p"
+		(property "Value" "3p"
 			(at 0 1.05 150)
 			(layer "F.Fab")
@@
 			)
 		)
-		(property "Value" "10p"
+		(property "Value" "3p"
 			(at 0 1.05 60)
 			(layer "F.Fab")
