File: HARDWARE/ELECTRONIQUE/PCB_BRUSHED/PCB_BRUSHED.kicad_sch (KiCad schematic)
At the start: 41 parts, among them IC1 TPS82150SILR, U1 STM32G431CBUx, Y1 Crystal_GND24_Small

Commit message: update
Parts:
- removed C10: 16p, Capacitor_SMD:C_0402_1005Metric_Pad0.74x0.62mm_HandSolder, symbol Device:C_Small
- removed Y1: Crystal_GND24_Small, crystalmulticomp:MCSJK7U1200101080B10, symbol Device:Crystal_GND24_Small
- added C17, C9: 100n, Capacitor_SMD:C_0201_0603Metric_Pad0.64x0.40mm_HandSolder, symbol Device:C_Small
- added R10: 22R, Resistor_SMD:R_0201_0603Metric_Pad0.64x0.40mm_HandSolder, symbol Device:R_Small
- added R7: 1k, Resistor_SMD:R_0201_0603Metric_Pad0.64x0.40mm_HandSolder, symbol Device:R_Small
- added R8: 10k, Resistor_SMD:R_0201_0603Metric_Pad0.64x0.40mm_HandSolder, symbol Device:R_Small
- added Y1: 830069528, samacsys:830069528, symbol samacsys:830069528
- C11, C7: footprint Capacitor_SMD:C_0402_1005Metric_Pad0.74x0.62mm_HandSolder -> Capacitor_SMD:C_0201_0603Metric_Pad0.64x0.40mm_HandSolder
- C18: renamed from C17; footprint Capacitor_SMD:C_0402_1005Metric_Pad0.74x0.62mm_HandSolder -> Capacitor_SMD:C_0201_0603Metric_Pad0.64x0.40mm_HandSolder
- C21: renamed from C20; footprint Capacitor_SMD:C_0402_1005Metric_Pad0.74x0.62mm_HandSolder -> Capacitor_SMD:C_0201_0603Metric_Pad0.64x0.40mm_HandSolder
- C23: renamed from C22; footprint Capacitor_SMD:C_0402_1005Metric_Pad0.74x0.62mm_HandSolder -> Capacitor_SMD:C_0201_0603Metric_Pad0.64x0.40mm_HandSolder
- C25: renamed from C24; footprint Capacitor_SMD:C_0402_1005Metric_Pad0.74x0.62mm_HandSolder -> Capacitor_SMD:C_0201_0603Metric_Pad0.64x0.40mm_HandSolder
- C3: footprint Capacitor_SMD:C_0201_0603Metric -> Capacitor_SMD:C_0201_0603Metric_Pad0.64x0.40mm_HandSolder
- C8: value 16p -> 100n; footprint Capacitor_SMD:C_0402_1005Metric_Pad0.74x0.62mm_HandSolder -> Capacitor_SMD:C_0201_0603Metric_Pad0.64x0.40mm_HandSolder
- R3: renamed from R2; footprint Resistor_SMD:R_0201_0603Metric -> Resistor_SMD:R_0201_0603Metric_Pad0.64x0.40mm_HandSolder
- R4, R5: footprint Resistor_SMD:R_0201_0603Metric -> Resistor_SMD:R_0201_0603Metric_Pad0.64x0.40mm_HandSolder
- R6: renamed from R7; footprint Resistor_SMD:R_0201_0603Metric -> Resistor_SMD:R_0201_0603Metric_Pad0.64x0.40mm_HandSolder
- TP1, TP2, TP3: footprint samacsys:m3test -> MountingHole:MountingHole_2.5mm_Pad_Via
- renumbered C9 to C10, C18 to C19, C19 to C20, C21 to C22, C23 to C24, C25 to C26, C26 to C27, C5 to C4, C4 to C5, R3 to R1, R6 to R2, R1 to R9
Connections:
- net GND: now also C17.1, C9.1, R7.2, Y1.2 (GND_1), Y1.4 (GND_2)
- net VBAT+: now also R8.1
- net HSE_IN: now reaches U1.5 (PF0)
- net HSE_IN: now also C9.2, Y1.1 (CRYSTAL_1)
- net ADC_VBAT: now reaches C8.1
- net ADC_VBAT: now also U1.4 (PC15), R7.1, R8.2; no longer U1.6 (PF1)
- net at D1.2 (A): now also U1.2 (PC13)
- net ADC2_IN5: now reaches C4.1, R1.1, R2.2
- net ADC2_IN5: now also U1.16 (PC4)
- net UART_EXTI: now reaches U1.19 (PB2)
- net EXT_BTN_EXTI10: now reaches U1.39 (PC10)
- net MOT1_HALL_C/TIM2CH3: no longer names the net of U1.10 (PA2)
- net MOT2_HALL_C/TIM1CH3: no longer names the net of U1.32 (PA10)
- net MOT3_HALL_C/TIM8CH3: no longer names the net of U1.47 (PB9)
- new net: C17.2, R10.1, Y1.3 (CRYSTAL_2)
- new net HSE_OUT: R10.2, U1.6 (PF1)
- no-connect marks 0 -> 6
Other:
- removed sheet HALL
- sheet CONN ports: added BTN, EXTI_EXT, NRST, SWCLK, SWDIO, UART_RX, UART_TX; removed none
- sheet MOTOR1 ports: added ENCODERA, ENCODERB, PWMMOT_1, PWMMOT_2, SPI_CLK, SPI_CS, SPI_MISO, SPI_MOSI; removed none
- sheet MOTOR2 ports: added ENCODERA, ENCODERB, PWMMOT_1, PWMMOT_2, SPI_CLK, SPI_CS, SPI_MISO, SPI_MOSI; removed none
- sheet MOTOR3 ports: added ENCODERA, ENCODERB, PWMMOT_1, PWMMOT_2, SPI_CLK, SPI_CS, SPI_MISO, SPI_MOSI; removed none
- moved on the sheet: C4, D1, R1, R2, R9

Commit message: up
Parts:
- removed C12, C13, C14, C15, C19, C20, C22, C24, C27: 22u, Capacitor_SMD:C_0805_2012Metric, symbol Device:C_Small
Other:
- note removed: "CONDO_VBAT"

Commit message: up brushed
Changed lines of the file:
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@@
 	)
 	(junction
+		(at 412.75 335.28)
+		(diameter 0)
+		(color 0 0 0 0)
+	)
+	(junction
 		(at 518.16 83.82)
 		(diameter 0)
@@
 	)
 	(junction
+		(at 354.33 363.22)
+		(diameter 0)
+		(color 0 0 0 0)
+	)
+	(junction
 		(at 509.27 54.61)
 		(diameter 0)
@@
 	(wire
 		(pts
-			(xy 408.94 335.28) (xy 414.02 335.28)
+			(xy 408.94 335.28) (xy 412.75 335.28)
 		)
 		(stroke
@@
 	(wire
 		(pts
+			(xy 412.75 335.28) (xy 414.02 335.28)
+		)
+		(stroke
+			(width 0)
+			(type default)
+		)
+	)
+	(wire
+		(pts
 			(xy 471.17 116.84) (xy 474.98 116.84)
 		)
@@
 	(wire
 		(pts
+			(xy 412.75 341.63) (xy 412.75 335.28)
+		)
+		(stroke
+			(width 0)
+			(type default)
+		)
+	)
+	(wire
+		(pts
 			(xy 351.79 358.14) (xy 354.33 358.14)
 		)
@@
 	(wire
 		(pts
+			(xy 354.33 364.49) (xy 354.33 363.22)
+		)
+		(stroke
+			(width 0)
+			(type default)
+		)
+	)
+	(wire
+		(pts
 			(xy 160.02 295.91) (xy 160.02 299.72)
 		)
@@
 	(wire
 		(pts
+			(xy 354.33 363.22) (xy 354.33 358.14)
+		)
+		(stroke
+			(width 0)
+			(type default)
+		)
+	)
+	(wire
+		(pts
 			(xy 115.57 110.49) (xy 111.76 110.49)
 		)
@@
 	(symbol
 		(lib_id "power:GND")
-		(at 354.33 358.14 0)
+		(at 354.33 364.49 0)
 		(unit 1)
 		(exclude_from_sim no)
@@
 		(fields_autoplaced yes)
 		(property "Reference" "#PWR01"
-			(at 354.33 364.49 0)
+			(at 354.33 370.84 0)
 			(effects
 				(font
@@
 		)
 		(property "Value" "GND"
-			(at 354.33 363.22 0)
+			(at 354.33 369.57 0)
 			(effects
 				(font
@@
 		)
 		(property "Footprint" ""
-			(at 354.33 358.14 0)
+			(at 354.33 364.49 0)
 			(effects
 				(font
@@
 		)
 		(property "Datasheet" ""
-			(at 354.33 358.14 0)
+			(at 354.33 364.49 0)
 			(effects
 				(font
@@
 		)
 		(property "Description" "Power symbol creates a global label with name \"GND\" , ground"
-			(at 354.33 358.14 0)
+			(at 354.33 364.49 0)
 			(effects
 				(font
@@
 	)
 	(symbol
+		(lib_id "power:PWR_FLAG")
+		(at 354.33 363.22 90)
+		(unit 1)
+		(exclude_from_sim no)
+		(in_bom yes)
+		(on_board yes)
+		(dnp no)
+		(fields_autoplaced yes)
+		(property "Reference" "#FLG01"
+			(at 352.425 363.22 0)
+			(effects
+				(font
+					(size 1.27 1.27)
+				)
+				(hide yes)
+			)
+		)
+		(property "Value" "PWR_FLAG"
+			(at 350.52 363.2199 90)
+			(effects
+				(font
+					(size 1.27 1.27)
+				)
+				(justify left)
+			)
+		)
+		(property "Footprint" ""
+			(at 354.33 363.22 0)
+			(effects
+				(font
+					(size 1.27 1.27)
+				)
+				(hide yes)
+			)
+		)
+		(property "Datasheet" "~"
+			(at 354.33 363.22 0)
+			(effects
+				(font
+					(size 1.27 1.27)
+				)
+				(hide yes)
+			)
+		)
+		(property "Description" "Special symbol for telling ERC where power comes from"
+			(at 354.33 363.22 0)
+			(effects
+				(font
+					(size 1.27 1.27)
+				)
+				(hide yes)
+			)
+		)
+		(pin "1"
+		)
+		(instances
+			(project ""
+				(path "/21624bb8-7220-4725-ab4f-34c4768aac8d"
+					(reference "#FLG01")
+					(unit 1)
+				)
+			)
+		)
+	)
+	(symbol
 		(lib_id "Device:C_Small")
 		(at 509.27 81.28 180)
@@
 					(unit 1)
 				)
+			)
+		)
+	)
+	(symbol
+		(lib_id "power:PWR_FLAG")
+		(at 412.75 341.63 180)
+		(unit 1)
+		(exclude_from_sim no)
+		(in_bom yes)
+		(on_board yes)
+		(dnp no)
+		(fields_autoplaced yes)
+		(property "Reference" "#FLG02"
+			(at 412.75 343.535 0)
+			(effects
+				(font
+					(size 1.27 1.27)
+				)
+				(hide yes)
+			)
+		)
+		(property "Value" "PWR_FLAG"
+			(at 412.75 346.71 0)
+			(effects
+				(font
+					(size 1.27 1.27)
+				)
+			)
+		)
+		(property "Footprint" ""
+			(at 412.75 341.63 0)
+			(effects
+				(font
+					(size 1.27 1.27)
+				)
+				(hide yes)
+			)
+		)
+		(property "Datasheet" "~"
+			(at 412.75 341.63 0)
+			(effects
+				(font
+					(size 1.27 1.27)
+				)
+				(hide yes)
+			)
+		)
+		(property "Description" "Special symbol for telling ERC where power comes from"
+			(at 412.75 341.63 0)
+			(effects
+				(font
+					(size 1.27 1.27)
+				)
+				(hide yes)
+			)
+		)
+		(pin "1"
+		)
+		(instances
+			(project "PCB_BRUSHED"
+				(path "/21624bb8-7220-4725-ab4f-34c4768aac8d"
+					(reference "#FLG02")
+					(unit 1)
+				)

Commit message: update
Parts:
- C17, C9: value 100n -> 10p
Changed lines of the file:
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@@
 			)
 		)
-		(property "Value" "100n"
+		(property "Value" "10p"
 			(at 451.612 57.15 90)
 			(effects
@@
 			)
 		)
-		(property "Value" "100n"
+		(property "Value" "10p"
 			(at 513.842 57.15 90)
 			(effects
@@
 		(dnp no)
 		(property "Reference" "C16"
-			(at 506.73 80.0162 0)
+			(at 498.602 78.994 0)
 			(effects
 				(font

Commit message: up
Parts:
- C17, C9: value 10p -> 3p
Other:
- note added: "830072539 24Mhz 1.6mmx1.2mm 8pF"
- note added: "j'ai mis du 10u 6.3v"
Changed lines of the file:
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@@
 		)
 	)
+	(text "830072539 24Mhz 1.6mmx1.2mm 8pF"
+		(exclude_from_sim no)
+		(at 481.584 40.64 0)
+		(effects
+			(font
+				(size 1.27 1.27)
+			)
+		)
+	)
+	(text "j'ai mis du 10u 6.3v\n"
+		(exclude_from_sim no)
+		(at 394.97 329.184 0)
+		(effects
+			(font
+				(size 1.27 1.27)
+			)
+		)
+	)
 	(text "MCU SIP\n"
 		(exclude_from_sim no)
@@
 			)
 		)
-		(property "Value" "10p"
+		(property "Value" "3p"
 			(at 451.612 57.15 90)
 			(effects
@@
 			)
 		)
-		(property "Value" "10p"
+		(property "Value" "3p"
 			(at 513.842 57.15 90)
 			(effects
